File: ESP32-WROOM-32E/ESP32-MB-1.0/_autosave-ESP32-MB-1.0.kicad_sch (KiCad schematic)
At the start: 46 parts, among them J1 Conn_01x19, J10 Conn_01x03_Pin, J11 Conn_01x03_Pin, J12 Conn_01x03_Pin, J13 Conn_01x03_Pin, J14 Conn_01x03_Pin, J15 Conn_01x03_Pin, J16 XT60-M, J17 Conn_01x04_Pin, J18 Conn_01x04_Pin, J19 Conn_01x04_Pin, J2 Conn_01x19, J20 Conn_01x04_Pin, J21 Conn_01x02_Pin, J22 XT60-M, J23 Conn_01x02_Pin, J24 Conn_01x02_Pin, J25 Conn_01x02_Pin, J26 Conn_01x02_Pin, J27 Conn_01x02_Pin, J28 Conn_01x02_Pin, J29 Conn_01x02_Pin, J3 Conn_01x19, J30 XT60-M, J4 Conn_01x11_Pin, J5 Conn_01x11_Pin, J6 XT60-M, J7 Conn_01x19, J8 Conn_01x03_Pin, J9 Conn_01x03_Pin, U1 IRLB3813PBF, U2 IRLB3813PBF, U3 IRLB3813PBF, U4 IRLB3813PBF, U5 IRLB3813PBF, U6 IRLB3813PBF, U7 IRLB3813PBF, U8 IRLB3813PBF

Commit message: １００×１００
Parts:
- added J31, J32: Conn_01x02_Pin, symbol Connector:Conn_01x02_Pin
Changed lines of the file:
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@@
+	)
+	(symbol
+		(lib_id "Connector:Conn_01x02_Pin")
+		(at 171.45 125.73 0)
+		(unit 1)
+		(exclude_from_sim no)
+		(in_bom yes)
+		(on_board yes)
+		(dnp no)
+		(fields_autoplaced yes)
+		(property "Reference" "J32"
+			(at 172.085 120.65 0)
+			(effects
+				(font
+					(size 1.27 1.27)
+				)
+			)
+		)
+		(property "Value" "Conn_01x02_Pin"
+			(at 172.085 123.19 0)
+			(effects
+				(font
+					(size 1.27 1.27)
+				)
+			)
+		)
+		(property "Footprint" ""
+			(at 171.45 125.73 0)
+			(effects
+				(font
+					(size 1.27 1.27)
+				)
+				(hide yes)
+			)
+		)
+		(property "Datasheet" "~"
+			(at 171.45 125.73 0)
+			(effects
+				(font
+					(size 1.27 1.27)
+				)
+				(hide yes)
+			)
+		)
+		(property "Description" "Generic connector, single row, 01x02, script generated"
+			(at 171.45 125.73 0)
+			(effects
+				(font
+					(size 1.27 1.27)
+				)
+				(hide yes)
+			)
+		)
+		(pin "1"
+		)
+		(pin "2"
+		)
+		(instances
+			(project ""
+				(path "/f192144f-1ca9-429a-9b75-464cafba9f58"
+					(reference "J32")
+					(unit 1)
+				)
+			)
+		)
 	)
 	(symbol
@@
 					(unit 1)
 				)
+			)
+		)
+	)
+	(symbol
+		(lib_id "Connector:Conn_01x02_Pin")
+		(at 170.18 105.41 0)
+		(unit 1)
+		(exclude_from_sim no)
+		(in_bom yes)
+		(on_board yes)
+		(dnp no)
+		(fields_autoplaced yes)
+		(property "Reference" "J31"
+			(at 170.815 100.33 0)
+			(effects
+				(font
+					(size 1.27 1.27)
+				)
+			)
+		)
+		(property "Value" "Conn_01x02_Pin"
+			(at 170.815 102.87 0)
+			(effects
+				(font
+					(size 1.27 1.27)
+				)
+			)
+		)
+		(property "Footprint" ""
+			(at 170.18 105.41 0)
+			(effects
+				(font
+					(size 1.27 1.27)
+				)
+				(hide yes)
+			)
+		)
+		(property "Datasheet" "~"
+			(at 170.18 105.41 0)
+			(effects
+				(font
+					(size 1.27 1.27)
+				)
+				(hide yes)
+			)
+		)
+		(property "Description" "Generic connector, single row, 01x02, script generated"
+			(at 170.18 105.41 0)
+			(effects
+				(font
+					(size 1.27 1.27)
+				)
+				(hide yes)
+			)
+		)
+		(pin "2"
+		)
+		(pin "1"
+		)
+		(instances
+			(project ""
+				(path "/f192144f-1ca9-429a-9b75-464cafba9f58"
+					(reference "J31")
+					(unit 1)
+				)
