File: ESP32-WROOM-32E/ESP32-MB-1.0/ESP32-MB-1.0.kicad_sch (KiCad schematic)
At the start: 46 parts, among them J1 Conn_01x19, J10 Conn_01x03_Pin, J11 Conn_01x03_Pin, J12 Conn_01x03_Pin, J13 Conn_01x03_Pin, J14 Conn_01x03_Pin, J15 Conn_01x03_Pin, J16 XT60-M, J17 Conn_01x04_Pin, J18 Conn_01x04_Pin, J19 Conn_01x04_Pin, J2 Conn_01x19, J20 Conn_01x04_Pin, J21 Conn_01x02_Pin, J22 XT60-M, J23 Conn_01x02_Pin, J24 Conn_01x02_Pin, J25 Conn_01x02_Pin, J26 Conn_01x02_Pin, J27 Conn_01x02_Pin, J28 Conn_01x02_Pin, J29 Conn_01x02_Pin, J3 Conn_01x19, J30 XT60-M, J4 Conn_01x11_Pin, J5 Conn_01x11_Pin, J6 XT60-M, J7 Conn_01x19, J8 Conn_01x03_Pin, J9 Conn_01x03_Pin, U1 IRLB3813PBF, U2 IRLB3813PBF, U3 IRLB3813PBF, U4 IRLB3813PBF, U5 IRLB3813PBF, U6 IRLB3813PBF, U7 IRLB3813PBF, U8 IRLB3813PBF

Commit message: モタドラ３つバージョンの自動配線前
Parts:
- added J31, J32, J34, J35, J36, J37, J38, J39: Conn_01x02_Pin, Connector_JST:JST_XH_B2B-XH-AM_1x02_P2.50mm_Vertical, symbol Connector:Conn_01x02_Pin
- added J33: Conn_01x11_Pin, Connector_PinHeader_2.54mm:PinHeader_1x11_P2.54mm_Vertical, symbol Connector:Conn_01x11_Pin
- added U9: MCP2562-E-P, Package_DIP:DIP-8_W7.62mm, symbol Interface_CAN_LIN:MCP2562-E-P
Connections:
- net 0_+3V3: now also U9.5 (Vio)
- net 0_+5V: now also U9.3 (VDD)
- net 0_GPIO4: now also U9.1 (TXD)
- net 0_GPIO5: now also U9.4 (RXD)
- net 1_GPIO12: now also R7.2
- net 1_GPIO13: now also R8.2
- net 1_GPIO16: now also J33.5 (Pin_5); no longer R7.2
- net 1_GPIO2: now also J33.9 (Pin_9); no longer R8.2
- net 1_GPIO4: now also J33.11 (Pin_11)
- net 1_GPIO5: now also J33.7 (Pin_7)
- net GND: now also J33.1 (Pin_1), J33.3 (Pin_3), U9.2 (VSS), U9.8 (STBY)
- new net: J31.1 (Pin_1), J32.1 (Pin_1), J34.1 (Pin_1), J35.1 (Pin_1), J36.1 (Pin_1), J37.1 (Pin_1), J38.1 (Pin_1), J39.1 (Pin_1), U9.7 (CANH)
- new net: J31.2 (Pin_2), U9.6 (CANL)

Commit message: ESP割り当て
Parts:
- removed J17, J18, J19, J20: Conn_01x04_Pin, Connector_JST:JST_XH_B4B-XH-AM_1x04_P2.50mm_Vertical, symbol Connector:Conn_01x04_Pin
Connections:
- net 1_GZPIO3 renamed 1_GPIO3

Commit message: 100になれなかったモタドラ4枚
Connections:
- net 0_GPIO11: now also J33.9 (Pin_9)
- net 0_GPIO21: now also J33.7 (Pin_7)
- net 0_GPIO22: now also J33.11 (Pin_11)
- net 0_GPIO23: now also J33.5 (Pin_5)
- net 1_GPIO16: no longer J33.5 (Pin_5)
- net 1_GPIO2: no longer J33.9 (Pin_9)
- net 1_GPIO4: no longer J33.11 (Pin_11)
- net 1_GPIO5: no longer J33.7 (Pin_7)

Commit message: １００×１００
Parts:
- added J17: Conn_01x11_Pin, Connector_PinHeader_2.54mm:PinHeader_1x11_P2.54mm_Vertical, symbol Connector:Conn_01x11_Pin
Connections:
- net 0_GPIO16: now also J17.7 (Pin_7)
- net 0_GPIO17: now also J17.11 (Pin_11)
- net 0_GPIO18: now also J17.5 (Pin_5)
- net 0_GPIO19: now also J17.9 (Pin_9)
- net GND: now also J17.1 (Pin_1), J17.3 (Pin_3)

Commit message: kakunin
Connections:
- net 1_GPIO12: no longer R7.2
- net 1_GPIO13: no longer R8.2
- net 1_GPIO16: now also R7.2
- net 1_GPIO2: now also R8.2
- net at J39.2 (Pin_2): now also J31.2 (Pin_2), J32.2 (Pin_2), J34.2 (Pin_2), J35.2 (Pin_2), J36.2 (Pin_2), J37.2 (Pin_2), J38.2 (Pin_2), U9.6 (CANL)
Other:
- moved on the sheet: J31, J32, J34, J35, J36, J37, J38, J39
