File: ESP32-WROOM-32E/ESP32-WROOM-32E-RRST/ESP32-WROOM-32E-RRST.kicad_pcb (KiCad board)
At the start: 2 copper layers, 115.8 x 100 mm, 76 parts, among them J1 USB_B_Micro, J10 Conn_01x02_Pin, J11 Conn_01x02_Pin, J12 Conn_01x02_Pin, J13 XT60-M, J14 Conn_01x02_Pin, J15 Conn_01x02_Pin, J16 Conn_01x02_Pin, J17 Conn_01x02_Pin, J18 XT60-M, J19 XT60-M, J2 XT60-M, J20 XT60-M, J21 Conn_01x02_Pin, J22 Conn_01x02_Pin, J23 Conn_01x02_Pin, J24 Conn_01x02_Pin, J25 Conn_01x02_Pin, J3 XT60-M, J4 Conn_01x11_Pin, J5 Conn_01x11_Pin, J6 Conn_01x04_Pin, J7 Conn_01x04_Pin, J8 Conn_01x04_Pin, J9 Conn_01x04_Pin, Q1 SS8050-G, Q2 SS8050-G, SW1 SW_Push, SW2 SW_Push, U10 ESP32-WROOM-32E, U11 AMS1117-3.3, U2 MCP2562-E-P, U9 CP2102N-A02-GQFN28

Commit message: 配線済み
Routing:
- net GND: track 230.7 -> 718.1 mm, vias 0 -> 7
- net VDD33: track 0.00 -> 347.7 mm, vias 0 -> 7
- net IO13: track 0.00 -> 297.6 mm, vias 0 -> 9
- net IO14: track 0.00 -> 297.4 mm, vias 0 -> 7
- net IO21: track 0.00 -> 282.1 mm, vias 0 -> 14
- net IO27: track 0.00 -> 260.8 mm, vias 0 -> 6
- net IO25: track 0.00 -> 251.4 mm, vias 0 -> 7
- net IO32: track 0.00 -> 248.2 mm, vias 0 -> 7
- net IO26: track 0.00 -> 247.8 mm, vias 0 -> 8
- net IO15: track 0.00 -> 244.3 mm, vias 0 -> 9
- net IO17: track 0.00 -> 228.2 mm, vias 0 -> 3
- net IO23: track 0.00 -> 226.7 mm, vias 0 -> 13
- net IO12: track 0.00 -> 225.7 mm, vias 0 -> 4
- net IO18: track 0.00 -> 210.4 mm, vias 0 -> 2
- net IO22: track 0.00 -> 207.0 mm, vias 0 -> 7
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
Commit message: シルクの追加と修正、お盆休み開始
Other:
- board text added: "(kicad_pcb (version 20241229) (generator "pcbnew") (generator_version "9.0") (layers (0 "F.Cu" signal) (2 "B.Cu" signal) (9 "F.Adhes" user "F.Adhesive") (11 "B.Adhes" user "B.Adhesive") (13 "F.Paste" user) (15 "B.Paste" user) (5 "F.SilkS" user "F.Silkscreen") (7 "B.SilkS" user "B.Silkscreen") (1 "F.Mask" user) (3 "B.Mask" user) (17 "Dwgs.User" user "User.Drawings") (19 "Cmts.User" user "User.Comm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"
- board text added: "02 04 05 12 13 14 15 16 17 18 19"
- board text added: "21 22 23 25 26 27 32 33 3V GND"
- board text added: "24V IN"
- board text added: "24V OUT"
- board text added: "24V OUT 24V OUT"
- board text added: "3V G A B"
- board text added: "CAN-BUS CAN-BUS"
- board text added: "CANL CANH"
- board text added: "ENC1"
- board text added: "ENC2"
- board text added: "ENC4"
- board text added: "ESP32-WROOM-32E"
- board text added: "GND +"
- board text added: "GPIO"
- board text added: "MCP2562-E-P"
- board text added: "S + GND"
- board text added: "SERVO POWER"
- board text added: "SV1"
- board text added: "SV2"
- board text added: "SV3"
- board text added: "SV4"
- board text added: "SV5"
- board text added: "SV6"
- board text added: "SV7"
- board text added: "TBD62003APG"
