File: MD旧/MD旧.kicad_pcb (KiCad board)
At the start: 2 copper layers, 42 parts, among them J1 Conn_01x04_Pin, J2 Conn_02x04_Odd_Even, J3 XT60-M, J4 XT60-M

Commit message: 配線できたよー
Parts:
- moved R7 10.2 mm to (167.6, 66.0), turned to 180 degrees
- moved R8 10.2 mm to (137.2, 121.9), turned to -90 degrees
- moved R9 10.2 mm to (119.4, 121.9), turned to -90 degrees
- moved R10 10.2 mm to (137.2, 106.7), turned to -90 degrees
- moved R11 10.2 mm to (119.4, 106.7), turned to -90 degrees
- moved R6 10.2 mm to (167.6, 61.0), turned to 180 degrees
- moved FET1 5.24 mm to (143.5, 124.5), turned to -90 degrees
- moved FET3 5.24 mm to (143.5, 109.2), turned to -90 degrees
- moved FET2 5.08 mm to (127.0, 124.5), turned to -90 degrees
- moved FET4 5.08 mm to (127.0, 109.2), turned to -90 degrees
Routing:
- net +2V5: track 0.00 -> 153.9 mm
- net MC: track 0.00 -> 110.3 mm
- net +12V: track 0.00 -> 108.7 mm
- net GATE1: track 0.00 -> 62.3 mm
- net +24V: track 0.00 -> 59.0 mm
- net DIGITAL: track 0.00 -> 55.8 mm
- net PWM_NOT: track 0.00 -> 52.6 mm
- net PWM1: track 0.00 -> 52.3 mm, vias 0 -> 2
- net Net-(FET1-G): track 0.00 -> 49.6 mm
- net GATE2: track 0.00 -> 43.5 mm, vias 0 -> 2
- net DIGITAL_NOT: track 0.00 -> 37.8 mm
- net Net-(FET2-G): track 0.00 -> 36.4 mm
- net PWM_IN: track 0.00 -> 28.0 mm
- net DIGITAL_IN: track 0.00 -> 27.7 mm
- net PWM2: track 0.00 -> 26.2 mm
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Other:
- board outline added: 69.8 x 92.7 mm

Commit message: MOUT1,2
Connections:
- C10 pad 2: MC -> MOUT1
- C11 pad 2: MC -> MOUT2
- FET1 pad 3: MC -> MOUT1
- FET2 pad 2: MC -> MOUT1
- FET3 pad 3: MC -> MOUT2
- FET4 pad 2: MC -> MOUT2
- IC3 pad 6: MC -> MOUT1
- IC4 pad 6: MC -> MOUT2
- R10 pad 2: MC -> MOUT2
- R8 pad 2: MC -> MOUT1
Routing:
- net MC: track 110.3 -> 0.00 mm
- net MOUT1: track 0.00 -> 86.6 mm
- net MOUT2: track 0.00 -> 83.3 mm, vias 0 -> 2

Commit message: 完成？
Parts:
- R1, R2, R3, R4, R5: value 200 -> 200Ω
- R6, R7: value 330 -> 330Ω
Routing:
- net GND2: track 0.00 -> 176.5 mm, vias 0 -> 5
- net +24V: track 59.0 -> 0.00 mm
- net GND1: track 0.00 -> 24.6 mm
- net MOUT1: track 86.6 -> 67.5 mm
- net MOUT2: vias 2 -> 0
- added copper zone on B.Cu, net +24V
- added copper zone on F.Cu, net GND2
- added copper zone on F.Cu, net MOUT1
- added copper zone on F.Cu, net MOUT2
Other:
- board text added: "24V 24V 24V"
- board text added: "D P GND1 5V"
- board text added: "G D S"
- board text added: "MOUT2 MOUT1"

Commit message: これで完成と言うことに勝手にしておきますねむい
Parts:
- D1: value LED -> PWM_IN
- D2: value LED -> 2.5V
- D3: value LED -> 12V
Other:
- board text added: "IN"
- board text added: "OUT"
Changed lines of the file:
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@@
 		(tags "IRLB3813PBF ")
 		(property "Reference" "REFG5V1"
-			(at 2.54 -3.81 0)
+			(at 2.54 -2.286 0)
 			(unlocked yes)
 			(layer "F.SilkS")
@@
 		(property "Reference" "D3"
 			(at 1.27 -3.96 0)
-			(layer "F.SilkS")
+			(layer "F.Fab")
 			(effects
 				(font
@@
 			)
 		)
-		(property "Value" "LED"
+		(property "Value" "12V"
 			(at 1.27 3.96 0)
-			(layer "F.Fab")
+			(layer "F.SilkS")
 			(effects
 				(font
@@
 		(property "Reference" "D2"
 			(at 1.27 -3.96 0)
-			(layer "F.SilkS")
+			(layer "F.Fab")
 			(effects
 				(font
@@
 			)
 		)
-		(property "Value" "LED"
+		(property "Value" "2.5V"
 			(at 1.27 3.96 0)
-			(layer "F.Fab")
+			(layer "F.SilkS")
 			(effects
 				(font
@@
 		(tags "IRLB3813PBF ")
 		(property "Reference" "REG12V1"
-			(at 2.54 2.54 0)
+			(at 2.54 -2.286 0)
 			(unlocked yes)
 			(layer "F.SilkS")
@@
 		(property "Reference" "D1"
 			(at 1.27 -3.96 0)
-			(layer "F.SilkS")
+			(layer "F.Fab")
 			(effects
 				(font
@@
 			)
 		)
-		(property "Value" "LED"
+		(property "Value" "PWM_IN"
 			(at 1.27 3.96 0)
-			(layer "F.Fab")
+			(layer "F.SilkS")
 			(effects
 				(font
@@
 		)
 		(property "Value" "0.1μF"
-			(at 2.5 3.75 0)
-			(layer "F.Fab")
+			(at 2.5 -3.556 0)
+			(layer "F.SilkS")
 			(effects
 				(font
@@
 		(tags "Through hole pin header THT 1x04 2.54mm single row")
 		(property "Reference" "J1"
-			(at 0 -2.38 90)
+			(at 0 3.81 180)
 			(layer "F.SilkS")
 			(effects
@@
 		)
 	)
+	(gr_text "OUT"
+		(at 159.258 124.968 0)
+		(layer "F.SilkS")
+		(effects
+			(font
+				(size 1 1)
+				(thickness 0.1)
+			)
+			(justify left bottom)
+		)
+	)
+	(gr_text "IN"
+		(at 153.162 124.968 0)
+		(layer "F.SilkS")
+		(effects
+			(font
+				(size 1 1)
+				(thickness 0.1)
+			)
+			(justify left bottom)
+		)
+	)
 	(gr_text "G  D  S"
 		(at 140.335 108.585 270)
@@
 		)
 	)
+	(gr_text "OUT"
+		(at 159.512 106.172 0)
+		(layer "F.SilkS")
+		(effects
+			(font
+				(size 1 1)
+				(thickness 0.1)
+			)
+			(justify left bottom)
+		)
+	)
 	(gr_text "D P GND1 5V"
 		(at 128.27 61.595 0)
@@
 			)
 			(justify left bottom)
+		)
+	)
+	(gr_text "IN"
+		(at 152.908 106.2736 0)
+		(layer "F.SilkS")
+		(effects
+			(font
+				(size 1 1)
+				(thickness 0.1)
+			)
+			(justify left bottom)
