File: MD旧.改/MD旧.改.kicad_sch (KiCad schematic)
At the start: 42 parts, among them J1 Conn_01x04_Pin, J2 Conn_02x04_Odd_Even, J3 XT60-M, J4 XT60-M

Commit message: 今から頑張ります
Parts:
- R2: value 200Ω -> 200Ω
Changed lines of the file:
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@@
 			)
 		)
-		(property "Value" "200Ω"
+		(property "Value" "200Ω"
 			(at 123.19 82.5499 0)
 			(effects

Commit message: 授業受けます！
Parts:
- D2: value 2.5V -> 5V/2
- R1, R10, R2, R3, R4, R5, R6, R7, R8, R9: footprint Resistor_THT:R_Axial_DIN0207_L6.3mm_D2.5mm_P10.16mm_Horizontal -> Library:R_Axial_DIN0207_L6.3mm_D2.5mm_P10.16mm_Horizontal_kai
Connections:
- net +2V5 renamed +5V/2
Changed lines of the file:
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@@
 			)
 		)
-		(property "Footprint" "Resistor_THT:R_Axial_DIN0207_L6.3mm_D2.5mm_P10.16mm_Horizontal"
+		(property "Footprint" "Library:R_Axial_DIN0207_L6.3mm_D2.5mm_P10.16mm_Horizontal_kai"
 			(at 207.772 64.77 90)
 			(effects
@@
 			)
 		)
-		(property "Footprint" "Resistor_THT:R_Axial_DIN0207_L6.3mm_D2.5mm_P10.16mm_Horizontal"
+		(property "Footprint" "Library:R_Axial_DIN0207_L6.3mm_D2.5mm_P10.16mm_Horizontal_kai"
 			(at 144.78 151.892 90)
 			(effects
@@
 			)
 		)
-		(property "Value" "+2V5"
+		(property "Value" "+5V/2"
 			(at 166.37 172.72 0)
 			(effects
@@
 			)
 		)
-		(property "Value" "+2V5"
+		(property "Value" "+5V/2"
 			(at 154.94 132.08 0)
 			(effects
@@
 			)
 		)
-		(property "Value" "+2V5"
+		(property "Value" "+5V/2"
 			(at 186.69 139.7 0)
 			(effects
@@
 			)
 		)
-		(property "Value" "2.5V"
+		(property "Value" "5V/2"
 			(at 124.46 91.7574 90)
 			(effects
@@
 			)
 		)
-		(property "Footprint" "Resistor_THT:R_Axial_DIN0207_L6.3mm_D2.5mm_P10.16mm_Horizontal"
+		(property "Footprint" "Library:R_Axial_DIN0207_L6.3mm_D2.5mm_P10.16mm_Horizontal_kai"
 			(at 106.172 78.74 90)
 			(effects
@@
 			)
 		)
-		(property "Footprint" "Resistor_THT:R_Axial_DIN0207_L6.3mm_D2.5mm_P10.16mm_Horizontal"
+		(property "Footprint" "Library:R_Axial_DIN0207_L6.3mm_D2.5mm_P10.16mm_Horizontal_kai"
 			(at 144.78 154.432 90)
 			(effects
@@
 			)
 		)
-		(property "Value" "+2V5"
+		(property "Value" "+5V/2"
 			(at 67.31 171.4499 90)
 			(effects
@@
 			)
 		)
-		(property "Footprint" "Resistor_THT:R_Axial_DIN0207_L6.3mm_D2.5mm_P10.16mm_Horizontal"
+		(property "Footprint" "Library:R_Axial_DIN0207_L6.3mm_D2.5mm_P10.16mm_Horizontal_kai"
 			(at 178.562 152.4 90)
 			(effects
@@
 			)
 		)
-		(property "Footprint" "Resistor_THT:R_Axial_DIN0207_L6.3mm_D2.5mm_P10.16mm_Horizontal"
+		(property "Footprint" "Library:R_Axial_DIN0207_L6.3mm_D2.5mm_P10.16mm_Horizontal_kai"
 			(at 118.872 81.28 90)
 			(effects
@@
 			)
 		)
-		(property "Value" "+2V5"
+		(property "Value" "+5V/2"
 			(at 120.65 72.39 0)
 			(effects
@@
 			)
 		)
-		(property "Value" "+2V5"
+		(property "Value" "+5V/2"
 			(at 67.31 139.6999 90)
 			(effects
@@
 			)
 		)
-		(property "Footprint" "Resistor_THT:R_Axial_DIN0207_L6.3mm_D2.5mm_P10.16mm_Horizontal"
+		(property "Footprint" "Library:R_Axial_DIN0207_L6.3mm_D2.5mm_P10.16mm_Horizontal_kai"
 			(at 170.942 149.86 90)
 			(effects
@@
 			)
 		)
-		(property "Footprint" "Resistor_THT:R_Axial_DIN0207_L6.3mm_D2.5mm_P10.16mm_Horizontal"
+		(property "Footprint" "Library:R_Axial_DIN0207_L6.3mm_D2.5mm_P10.16mm_Horizontal_kai"
 			(at 131.572 81.28 90)
 			(effects
@@
 			)
 		)
-		(property "Footprint" "Resistor_THT:R_Axial_DIN0207_L6.3mm_D2.5mm_P10.16mm_Horizontal"
+		(property "Footprint" "Library:R_Axial_DIN0207_L6.3mm_D2.5mm_P10.16mm_Horizontal_kai"
 			(at 207.772 102.87 90)
 			(effects
@@
 			)
 		)
-		(property "Footprint" "Resistor_THT:R_Axial_DIN0207_L6.3mm_D2.5mm_P10.16mm_Horizontal"
+		(property "Footprint" "Library:R_Axial_DIN0207_L6.3mm_D2.5mm_P10.16mm_Horizontal_kai"
 			(at 207.772 36.83 90)
 			(effects

Commit message: 詰め詰め
Parts:
- R11: footprint Resistor_THT:R_Axial_DIN0207_L6.3mm_D2.5mm_P10.16mm_Horizontal -> Library:R_Axial_DIN0207_L6.3mm_D2.5mm_P10.16mm_Horizontal_kai
Changed lines of the file:
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@@
 			)
 		)
-		(property "Footprint" "Resistor_THT:R_Axial_DIN0207_L6.3mm_D2.5mm_P10.16mm_Horizontal"
+		(property "Footprint" "Library:R_Axial_DIN0207_L6.3mm_D2.5mm_P10.16mm_Horizontal_kai"
 			(at 207.772 130.81 90)
 			(effects

Commit message: あ
Parts:
- removed J2: Conn_02x04_Odd_Even, Connector_PinHeader_2.54mm:PinHeader_2x04_P2.54mm_Vertical, symbol Connector_Generic:Conn_02x04_Odd_Even
Connections:
- net PWM2 is gone; now on net PWM1: IC2_AND1.1, IC2_AND1.4
