File: MD旧.改/MD旧.改.kicad_pcb (KiCad board)
At the start: 2 copper layers, 42 parts, among them J1 Conn_01x04_Pin, J2 Conn_02x04_Odd_Even, J3 XT60-M, J4 XT60-M

Commit message: 今から頑張ります
Parts:
- R2: value 200Ω -> 200Ω
- moved C1 47.3 mm to (17.9, 65.5)
- moved C2 38.7 mm to (63.6, 48.9)
- moved C4 37.8 mm to (63.6, 52.5)
- moved C6 37.0 mm to (63.6, 56.0)
- moved C7 36.1 mm to (63.6, 59.5)
- moved J1 35.7 mm to (37.8, 54.8)
- moved C8 35.2 mm to (63.6, 63.0)
- moved C9 34.4 mm to (63.6, 66.6)
- moved C10 33.5 mm to (63.6, 70.1)
- moved IC3 33.5 mm to (43.3, 18.2)
- moved IC4 33.5 mm to (54.1, 18.2)
- moved TLP2630 33.5 mm to (64.8, 18.2)
- moved C11 32.7 mm to (63.6, 73.6)
- moved D4 30.8 mm to (64.8, 41.9)
- moved D5 30.8 mm to (64.8, 45.4)
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
Commit message: 授業受けます！
Parts:
- D2: value 2.5V -> 5V/2
- R1, R10, R2, R3, R4, R5, R6, R7, R8, R9: footprint Resistor_THT:R_Axial_DIN0207_L6.3mm_D2.5mm_P10.16mm_Horizontal -> Library:R_Axial_DIN0207_L6.3mm_D2.5mm_P10.16mm_Horizontal_kai
- moved D4 46.2 mm to (24.5, 64.3)
- moved J2 46.2 mm to (25.2, 52.6)
- moved D5 46.2 mm to (24.5, 67.8)
- moved C3 34.4 mm to (39.0, 57.1)
- moved C5 34.4 mm to (39.0, 63.7)
- moved C2 33.2 mm to (38.4, 27.4)
- moved C9 33.2 mm to (38.4, 45.0)
- moved C10 33.2 mm to (38.4, 48.5)
- moved C11 33.2 mm to (38.4, 52.1)
- moved C4 33.2 mm to (38.4, 30.9)
- moved C6 33.2 mm to (38.4, 34.5)
- moved C7 33.2 mm to (38.4, 38.0)
- moved C8 33.2 mm to (38.4, 41.5)
- moved R11 32.3 mm to (46.7, 69.5)
- moved D1 31.8 mm to (47.6, 29.4)
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Connections:
- net +2V5 renamed +5V/2

Commit message: 詰め詰め
Parts:
- R11: footprint Resistor_THT:R_Axial_DIN0207_L6.3mm_D2.5mm_P10.16mm_Horizontal -> Library:R_Axial_DIN0207_L6.3mm_D2.5mm_P10.16mm_Horizontal_kai
- moved R2 162.4 mm to (124.2, 139.4), turned to 90 degrees
- moved FET1 159.4 mm to (102.9, 158.4), turned to -90 degrees
- moved R3 156.5 mm to (119.9, 139.4), turned to 90 degrees
- moved C6 153.0 mm to (117.6, 165.3)
- moved FET2 149.9 mm to (93.9, 158.4), turned to -90 degrees
- moved J3 146.5 mm to (97.7, 172.7), turned to 180 degrees
- moved C2 146.2 mm to (109.0, 155.4)
- moved J4 143.4 mm to (117.3, 172.7), turned to 180 degrees
- moved R8 141.6 mm to (99.5, 157.2), turned to -90 degrees
- moved C1 139.2 mm to (109.2, 162.6)
- moved FET3 138.6 mm to (102.7, 146.6), turned to -90 degrees
- moved D2 136.8 mm to (126.2, 148.8), turned to 180 degrees
- moved D3 136.1 mm to (126.2, 155.4), turned to 180 degrees
- moved C4 134.0 mm to (108.7, 145.0)
- moved R9 133.1 mm to (90.4, 157.4), turned to -90 degrees
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Other:
- board outline added: 41 x 77 mm

Commit message: あ
Parts:
- removed J2: Conn_02x04_Odd_Even, Connector_PinHeader_2.54mm:PinHeader_2x04_P2.54mm_Vertical
- moved R7 0.12 mm to (125.8, 104.7)
Connections:
- IC2_AND1 pad 1: PWM2 -> PWM1
- IC2_AND1 pad 4: PWM2 -> PWM1
Routing:
- net +5V/2: track 0.00 -> 90.2 mm, vias 0 -> 1
- net PWM_NOT: track 0.00 -> 49.6 mm, vias 0 -> 1
- net +12V: track 0.00 -> 39.4 mm
- net DIGITAL_NOT: track 0.00 -> 28.1 mm
- net DIGITAL_IN: track 0.00 -> 25.0 mm, vias 0 -> 1
- net DIGITAL: track 0.00 -> 24.0 mm
- net GATE2: track 0.00 -> 22.5 mm
- net PWM1: track 0.00 -> 21.9 mm
- net Net-(D4-K): track 0.00 -> 21.9 mm
- net PWM_IN: track 0.00 -> 19.5 mm
- net GND2: track 0.00 -> 17.0 mm
- net Net-(D1-A): track 0.00 -> 7.49 mm
- net Net-(D5-K): track 0.00 -> 4.32 mm
- net Net-(R5-Pad1): track 0.00 -> 3.44 mm
- net Net-(R4-Pad1): track 0.00 -> 2.71 mm

Commit message: 配線中,,,
Parts:
- moved C5 15.2 mm to (117.7, 144.0)
- moved C3 14.5 mm to (117.5, 158.8)
- moved C4 5.06 mm to (113.8, 144.4), turned to 180 degrees
Routing:
- net MOUT2: track 0.00 -> 47.2 mm
- net Net-(D5-K): track 4.32 -> 46.3 mm
- net GATE1: track 0.00 -> 38.6 mm, vias 0 -> 1
- net MOUT1: track 0.00 -> 36.1 mm
- net PWM1: track 21.9 -> 57.4 mm, vias 0 -> 2
- net Net-(FET2-G): track 0.00 -> 33.7 mm
- net +12V: track 39.4 -> 71.6 mm
- net Net-(FET4-G): track 0.00 -> 30.6 mm
- net Net-(FET1-G): track 0.00 -> 30.3 mm
- net Net-(FET3-G): track 0.00 -> 20.0 mm

Commit message: 塗りつぶしゾーンを描きたい
Routing:
- net +5V/2: track 90.2 -> 147.4 mm, vias 1 -> 4
- net Net-(D3-A): track 0.00 -> 39.0 mm
- net Net-(D2-A): track 0.00 -> 23.9 mm, vias 0 -> 1
Changed lines of the file:
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@@
+	)
+	(segment
+		(start 117.221 140.843)
+		(end 124.206 140.843)
+		(width 1)
+		(layer "F.Cu")
+		(net 4)
+	)
+	(segment
+		(start 117.983 148.082)
+		(end 117.983 153.67)
+		(width 1)
+		(layer "F.Cu")
+		(net 4)
 	)
 	(segment
@@
 	)
 	(segment
+		(start 116.713 148.082)
+		(end 117.983 148.082)
+		(width 1)
+		(layer "F.Cu")
+		(net 4)
+	)
+	(segment
 		(start 117.983 104.648)
 		(end 125.73 104.648)
@@
 	)
 	(segment
+		(start 124.206 140.843)
+		(end 124.23 140.819)
+		(width 0.2)
+		(layer "F.Cu")
+		(net 4)
+	)
+	(segment
 		(start 117.983 104.648)
 		(end 117.983 101.833)
+		(width 1)
+		(layer "F.Cu")
+		(net 4)
+	)
+	(segment
+		(start 117.983 153.67)
+		(end 122.602 158.289)
 		(width 1)
 		(layer "F.Cu")
@@
 	)
 	(segment
+		(start 124.23 140.819)
+		(end 124.23 139.4032)
+		(width 1)
+		(layer "F.Cu")
+		(net 4)
+	)
+	(segment
+		(start 122.602 158.289)
+		(end 122.602 165.354)
+		(width 1)
+		(layer "F.Cu")
+		(net 4)
+	)
+	(segment
+		(start 116.332 147.701)
+		(end 116.713 148.082)
+		(width 1)
+		(layer "F.Cu")
+		(net 4)
+	)
+	(segment
 		(start 127.923 126.077)
 		(end 127.923 104.65)
@@
 	)
 	(segment
+		(start 115.062 138.684)
+		(end 111.506 142.24)
+		(width 1)
+		(layer "F.Cu")
+		(net 4)
+	)
+	(segment
 		(start 127.818 104.648)
 		(end 125.73 104.648)
@@
 	)
 	(segment
+		(start 111.506 142.24)
+		(end 108.712 142.24)
+		(width 1)
+		(layer "F.Cu")
+		(net 4)
+	)
+	(segment
 		(start 118.7625 129.5225)
 		(end 121.92 126.365)
 		(width 1)
 		(layer "F.Cu")
+		(net 4)
+	)
+	(via
+		(at 108.712 142.24)
+		(size 0.6)
+		(drill 0.3)
+		(layers "F.Cu" "B.Cu")
+		(net 4)
+	)
+	(via
+		(at 116.332 147.701)
+		(size 0.6)
+		(drill 0.3)
+		(layers "F.Cu" "B.Cu")
+		(net 4)
+	)
+	(via
+		(at 117.221 140.843)
+		(size 0.6)
+		(drill 0.3)
+		(layers "F.Cu" "B.Cu")
 		(net 4)
 	)
@@
 	)
 	(segment
+		(start 106.553 142.24)
+		(end 106.553 146.939)
+		(width 1)
+		(layer "B.Cu")
+		(net 4)
+	)
+	(segment
+		(start 106.553 146.939)
+		(end 115.57 146.939)
+		(width 1)
+		(layer "B.Cu")
+		(net 4)
+	)
+	(segment
 		(start 112.98 128.855)
 		(end 102.92 128.855)
@@
 	)
 	(segment
+		(start 115.57 146.939)
+		(end 116.332 147.701)
+		(width 1)
+		(layer "B.Cu")
+		(net 4)
+	)
+	(segment
 		(start 104.775 123.19)
 		(end 102.87 125.095)
+		(width 1)
+		(layer "B.Cu")
+		(net 4)
+	)
+	(segment
+		(start 108.712 142.24)
+		(end 106.553 142.24)
+		(width 1)
+		(layer "B.Cu")
+		(net 4)
+	)
+	(segment
+		(start 115.062 138.684)
+		(end 117.221 140.843)
 		(width 1)
 		(layer "B.Cu")
@@
 	)
 	(segment
+		(start 123.703 148.844)
+		(end 123.703 143.134)
+		(width 0.6)
+		(layer "F.Cu")
+		(net 11)
+	)
+	(segment
+		(start 123.698 143.129)
+		(end 127.381 143.129)
+		(width 0.6)
+		(layer "F.Cu")
+		(net 11)
+	)
+	(segment
+		(start 127.381 143.129)
+		(end 127.381 131.826)
+		(width 0.6)
+		(layer "F.Cu")
+		(net 11)
+	)
+	(segment
+		(start 123.703 143.134)
+		(end 123.698 143.129)
+		(width 0.2)
+		(layer "F.Cu")
+		(net 11)
+	)
+	(via
+		(at 127.381 131.826)
+		(size 0.6)
+		(drill 0.3)
+		(layers "F.Cu" "B.Cu")
+		(net 11)
+	)
+	(segment
+		(start 127.381 131.826)
+		(end 124.2732 131.826)
+		(width 0.6)
+		(layer "B.Cu")
+		(net 11)
+	)
+	(segment
+		(start 124.2732 131.826)
+		(end 124.23 131.8692)
+		(width 0.6)
+		(layer "B.Cu")
+		(net 11)
+	)
+	(segment
+		(start 121.031 141.859)
+		(end 121.031 155.302372)
+		(width 0.6)
+		(layer "F.Cu")
+		(net 12)
+	)
+	(segment
+		(start 121.176628 155.448)
+		(end 123.698 155.448)
+		(width 0.6)
+		(layer "F.Cu")
+		(net 12)
+	)
+	(segment
+		(start 125.984 130.556)
+		(end 125.984 141.859)
+		(width 0.6)
+		(layer "F.Cu")
+		(net 12)
+	)
+	(segment
+		(start 121.4958 131.8692)
+		(end 122.809 130.556)
+		(width 0.6)
+		(layer "F.Cu")
+		(net 12)
+	)
+	(segment
+		(start 122.809 130.556)
+		(end 125.984 130.556)
+		(width 0.6)
+		(layer "F.Cu")
+		(net 12)
+	)
+	(segment
+		(start 121.031 155.302372)
+		(end 121.176628 155.448)
+		(width 0.6)
+		(layer "F.Cu")
+		(net 12)
+	)
+	(segment
+		(start 125.984 141.859)
+		(end 121.031 141.859)
+		(width 0.6)
+		(layer "F.Cu")
+		(net 12)
+	)
+	(segment
+		(start 119.912 131.8692)
+		(end 121.4958 131.8692)
+		(width 0.6)
+		(layer "F.Cu")
+		(net 12)
+	)
+	(segment
