File: MD旧.改/_autosave-MD旧.改.kicad_pcb (KiCad board)
At the start: 2 copper layers, 41 x 77 mm, 41 parts, among them J1 Conn_01x04_Pin, J3 XT60-M, J4 XT60-M

Commit message: 塗りつぶしたら未配線35でした泣
Routing:
- net Net-(FET4-G): track 30.6 -> 23.8 mm
- net GATE1: track 38.6 -> 34.0 mm
- net Net-(D5-K): track 46.3 -> 47.3 mm
