File: MDv3/MDv3.kicad_pcb (KiCad board)
At the start: 2 copper layers, 41 parts, among them J1 Conn_01x04_Pin, J3 XT60-M, J4 XT60-M

Commit message: 詰める
Parts:
- moved R2 154.2 mm to (142.2, 113.0), turned to 90 degrees
- moved R3 147.7 mm to (137.1, 113.0), turned to 90 degrees
- moved FET1 143.8 mm to (119.4, 134.6), turned to -90 degrees
- moved J4 142.9 mm to (132.1, 154.9)
- moved J3 141.4 mm to (111.8, 154.9)
- moved FET2 132.9 mm to (109.2, 134.6), turned to -90 degrees
- moved C3 132.6 mm to (137.2, 132.1)
- moved C1 130.7 mm to (127.0, 139.7)
- moved R8 129.0 mm to (114.3, 132.2), turned to -90 degrees
- moved R7 127.8 mm to (139.7, 77.5), turned to -90 degrees
- moved FET3 125.3 mm to (119.4, 121.9), turned to -90 degrees
- moved C6 124.2 mm to (137.2, 139.7)
- moved R6 124.1 mm to (134.6, 77.5), turned to -90 degrees
- moved C5 122.8 mm to (137.2, 119.4)
- moved REG12V1 122.4 mm to (127.0, 127.0)
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
Commit message: 詰めた、配線する
Parts:
- moved J4 7.93 mm to (128.0, 148.1), turned to 180 degrees
- moved J3 6.81 mm to (111.6, 148.1), turned to 180 degrees
- moved D3 6.50 mm to (141.0, 130.7)
- moved D2 6.50 mm to (141.0, 123.1)
- moved C1 5.86 mm to (124.1, 134.6)
- moved C6 5.78 mm to (132.2, 136.6)
- moved C2 5.37 mm to (122.8, 128.7)
- moved R2 5.21 mm to (137.0, 113.0)
- moved C3 4.90 mm to (132.4, 130.9)
- moved C5 4.85 mm to (132.3, 119.9)
- moved R3 4.45 mm to (132.7, 112.9)
- moved REFG5V1 4.44 mm to (122.9, 116.1)
- moved C4 4.39 mm to (122.8, 120.5)
- moved REG12V1 4.39 mm to (122.9, 125.3)
- moved FET1 4.31 mm to (116.2, 131.7)
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Other:
- board outline added: 44.4 x 76.2 mm

Commit message: やりなおし
Parts:
- added J2: XT60PW-M, XT60-M:AMASS_XT60PW-M, F.Cu at (64.0, 26.7)
- C10, C11: value 1.5 -> 1.5μF
- C2, C4, C6, C7, C8, C9: value 0.1 -> 0.1μF
- J1: value Conn_01x04_Pin -> XT60PW-M; footprint Connector_PinHeader_2.54mm:PinHeader_1x04_P2.54mm_Vertical -> XT60-M:AMASS_XT60PW-M
- J3, J4: value XT60-M -> XT30PW-M; footprint XT60-M:AMASS_XT60PW-M -> XT60-M:AMASS_XT30PW-M
- moved R2 151.7 mm to (15.8, 21.6), turned to 0 degrees
- moved R3 145.8 mm to (15.8, 25.7), turned to 0 degrees
- moved FET1 141.8 mm to (29.9, 19.2), turned to 0 degrees
- moved D3 134.4 mm to (17.0, 78.8), turned to 0 degrees
- moved D2 134.4 mm to (17.0, 71.3), turned to 0 degrees
- moved FET2 131.3 mm to (29.9, 25.3), turned to 0 degrees
- moved C6 130.3 mm to (26.4, 60.6)
- moved R8 127.9 mm to (15.8, 45.9), turned to 0 degrees
- moved R7 127.5 mm to (15.8, 41.9), turned to 0 degrees
- moved R6 124.7 mm to (15.8, 37.8), turned to 0 degrees
- moved FET3 123.8 mm to (29.9, 31.3), turned to 0 degrees
- moved C2 122.2 mm to (26.4, 53.6)
- moved REG12V1 120.0 mm to (29.9, 49.5)
- moved R9 118.4 mm to (15.8, 50.0), turned to 0 degrees
- moved REFG5V1 118.0 mm to (29.9, 43.4)
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Connections:
- J1 pad 1: +5V -> MOUT1
- J1 pad 2: GND1 -> MOUT2
- J3 pad N: MOUT2 -> GND1
- J3 pad P: MOUT1 -> +5V
- J4 pad N: GND2 -> DIGITAL_IN
- J4 pad P: +24V -> PWM_IN
Other:
- board outline removed

Commit message: がんばるんば
Parts:
- C10, C11: value 1.5μF -> 1.5
- C2, C4, C6, C7, C8, C9: value 0.1μF -> 0.1

Commit message: 配線前
Parts:
- C4, C6: value 0.1 -> 0.1μF
- moved R2 173.3 mm to (139.5, 143.0), turned to 90 degrees
- moved FET1 170.9 mm to (120.9, 163.8), turned to 90 degrees
- moved R3 167.5 mm to (135.4, 143.0), turned to 90 degrees
- moved J2 164.7 mm to (129.5, 177.8), turned to 180 degrees
- moved J1 164.2 mm to (111.1, 177.8), turned to 180 degrees
- moved FET2 160.7 mm to (111.3, 163.8), turned to 90 degrees
- moved R8 155.8 mm to (116.1, 165.2), turned to 90 degrees
- moved C2 155.7 mm to (135.4, 164.8)
- moved FET3 151.6 mm to (120.8, 152.7), turned to 90 degrees
- moved R9 146.4 mm to (106.4, 165.0), turned to 90 degrees
- moved REG12V1 143.9 mm to (127.0, 155.8)
- moved REFG5V1 142.6 mm to (127.0, 147.8)
- moved R10 141.2 mm to (115.8, 153.7), turned to 90 degrees
- moved FET4 141.1 mm to (111.3, 152.7), turned to 90 degrees
- moved C6 139.4 mm to (136.7, 146.0)
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Connections:
- J3 pad P: +5V -> GND1

Commit message: 本当の配線前
Parts:
- added REF**: MountingHole_3.2mm_M3, MountingHole:MountingHole_3.2mm_M3, F.Cu at (140.0, 116.0)
- added REF**: MountingHole_3.2mm_M3, MountingHole:MountingHole_3.2mm_M3, F.Cu at (93.0, 116.0)
- added REF**: MountingHole_3.2mm_M3, MountingHole:MountingHole_3.2mm_M3, F.Cu at (93.0, 176.0)
- added REF**: MountingHole_3.2mm_M3, MountingHole:MountingHole_3.2mm_M3, F.Cu at (140.0, 176.0)
- moved D1 3.56 mm to (98.8, 121.0)
- moved R1 3.06 mm to (102.6, 115.9)
- moved R4 1.35 mm to (114.3, 118.6)
- moved R5 1.35 mm to (114.3, 122.5)
- moved TLP2630 1.30 mm to (117.1, 115.1)
- moved R6 0.63 mm to (127.1, 116.6)
- moved R7 0.63 mm to (127.1, 120.9)
Other:
- board outline added: 54.6 x 67.8 mm

Commit message: 配線前確認よろしくお願いします！
Parts:
- C10, C11: value 1.5 -> 1.5μF
- C2, C7, C8, C9: value 0.1 -> 0.1μF
- R1: value 200Ω -> 330Ω
- moved C4 1.92 mm to (131.2, 151.4)
- moved REG12V1 0.46 mm to (127.0, 156.2)
Connections:
- J3 pad P: GND1 -> +5V
Other:
- board text added: "24V24V24V"
- board text added: "5V5V"
- board text added: "GND1"
- board text added: "GND2"
- board text added: "MOUT1"
- board text added: "MOUT2"
- board text added: "PWM_IN"
Changed lines of the file:
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@@
 	(net 41 "Net-(R4-Pad1)")
 	(net 42 "Net-(R5-Pad1)")
+	(net 43 "+5V")
 	(footprint "Library:R_Axial_DIN0207_L6.3mm_D2.5mm_P10.16mm_Horizontal_kai"
 		(layer "F.Cu")
@@
 		)
 		(fp_line
-			(start -3 12.25)
-			(end -2 12.25)
+			(start -6.4436 12.25)
+			(end -5.4436 12.25)
 			(stroke
 				(width 0.127)
@@
 		)
 		(fp_line
-			(start -2.5 12.75)
-			(end -2.5 11.75)
+			(start -5.9436 12.75)
+			(end -5.9436 11.75)
 			(stroke
 				(width 0.127)
@@
 		)
 		(fp_line
-			(start -3 12.25)
-			(end -2 12.25)
+			(start -6.4436 12.25)
+			(end -5.4436 12.25)
 			(stroke
 				(width 0.127)
@@
 		)
 		(fp_line
-			(start -2.5 12.75)
-			(end -2.5 11.75)
+			(start -5.9436 12.75)
+			(end -5.9436 11.75)
 			(stroke
 				(width 0.127)
@@
 			)
 		)
-		(property "Value" "1.5"
+		(property "Value" "1.5μF"
 			(at 2.5125 0.0375 90)
 			(unlocked yes)
@@
 			(layer "F.CrtYd")
 		)
-		(fp_text user "${REFERENCE}"
-			(at 0 0 0)
-			(layer "F.Fab")
-			(effects
-				(font
-					(size 1 1)
-					(thickness 0.15)
-				)
-			)
-		)
 		(pad "" np_thru_hole circle
 			(at 0 0)
@@
 			(at 0 4.15 0)
 			(layer "F.Fab")
+			(hide yes)
 			(effects
 				(font
@@
 			(layer "F.CrtYd")
 		)
-		(fp_text user "${REFERENCE}"
-			(at 0 0 0)
-			(layer "F.Fab")
-			(effects
-				(font
-					(size 1 1)
-					(thickness 0.15)
-				)
-			)
-		)
 		(pad "" np_thru_hole circle
 			(at 0 0)
@@
 			)
 		)
-		(property "Value" "0.1"
+		(property "Value" "0.1μF"
 			(at 2.5125 0.0375 90)
 			(unlocked yes)
@@
 			)
 		)
-		(property "Value" "200Ω"
+		(property "Value" "330Ω"
 			(at 3.7332 0.024 90)
 			(unlocked yes)
@@
 	(footprint "footprints:PG-TO220-3_INF"
 		(layer "F.Cu")
-		(at 127 155.7528)
+		(at 127 156.21)
 		(tags "IRLB3813PBF ")
 		(property "Reference" "REG12V1"
@@
 			)
 		)
-		(property "Value" "0.1"
+		(property "Value" "0.1μF"
 			(at 2.5125 0.0375 90)
 			(unlocked yes)
@@
 			)
 		)
-		(property "Value" "1.5"
+		(property "Value" "1.5μF"
 			(at 2.7665 0.0375 90)
 			(unlocked yes)
@@
 	(footprint "Library:C_Disc_D11.0mm_W5.0mm_P5.0mm_kai"
 		(layer "F.Cu")
-		(at 129.2585 151.174 180)
+		(at 131.1635 151.384 180)
 		(property "Reference" "C4"
 			(at 5 -2 180)
@@
 			)
 		)
-		(property "Value" "0.1"
+		(property "Value" "0.1μF"
 			(at 2.5125 0.0375 0)
 			(unlocked yes)
@@
 			)
 		)
-		(property "Value" "0.1"
+		(property "Value" "0.1μF"
 			(at 2.5125 0.0375 0)
 			(unlocked yes)
@@
 			(layer "F.CrtYd")
 		)
-		(fp_text user "${REFERENCE}"
-			(at 0 0 0)
-			(layer "F.Fab")
-			(effects
-				(font
-					(size 1 1)
-					(thickness 0.15)
-				)
-			)
-		)
 		(pad "" np_thru_hole circle
 			(at 0 0)
@@
 		)
 		(fp_line
-			(start 2 12.25)
-			(end 3 12.25)
+			(start 4.834 12.2428)
+			(end 5.834 12.2428)
 			(stroke
 				(width 0.127)
@@
 		)
 		(fp_line
-			(start -3 12.25)
-			(end -2 12.25)
+			(start -2.9892 13.5128)
+			(end -1.9892 13.5128)
 			(stroke
 				(width 0.127)
@@
 		)
 		(fp_line
-			(start -2.5 12.75)
-			(end -2.5 11.75)
+			(start -2.4892 14.0128)
+			(end -2.4892 13.0128)
 			(stroke
 				(width 0.127)
@@
 		)
 		(fp_line
-			(start 2 12.25)
-			(end 3 12.25)
+			(start 4.834 12.2428)
+			(end 5.834 12.2428)
 			(stroke
 				(width 0.127)
@@
 		)
 		(fp_line
-			(start -3 12.25)
-			(end -2 12.25)
+			(start -2.9892 13.5128)
+			(end -1.9892 13.5128)
 			(stroke
 				(width 0.127)
@@
 		)
 		(fp_line
-			(start -2.5 12.75)
-			(end -2.5 11.75)
+			(start -2.4892 14.0128)
+			(end -2.4892 13.0128)
 			(stroke
 				(width 0.127)
@@
 			(layers "*.Cu" "*.Mask")
 			(remove_unused_layers no)
-			(net 9 "GND1")
+			(net 43 "+5V")
 			(pinfunction "P")
 			(pintype "power_in")
@@
 			(layer "F.CrtYd")
 		)
-		(fp_text user "${REFERENCE}"
-			(at 0 0 0)
-			(layer "F.Fab")
-			(effects
-				(font
-					(size 1 1)
-					(thickness 0.15)
-				)
-			)
-		)
 		(pad "" np_thru_hole circle
 			(at 0 0)
@@
 		(layer "Edge.Cuts")
 	)
+	(gr_text "GND1"
+		(at 102.743 161.671 270)
+		(layer "F.SilkS" knockout)
+		(effects
+			(font
+				(size 0.7 0.7)
+				(thickness 0.12)
+				(bold yes)
+			)
+			(justify left bottom)
+		)
+	)
+	(gr_text "MOUT1"
+		(at 105.791 169.672 0)
+		(layer "F.SilkS" knockout)
+		(effects
+			(font
+				(size 0.7 0.7)
+				(thickness 0.12)
+				(bold yes)
+			)
+			(justify left bottom)
+		)
+	)
+	(gr_text "GND2"
+		(at 131.572 169.672 0)
+		(layer "F.SilkS" knockout)
+		(effects
+			(font
+				(size 0.7 0.7)
+				(thickness 0.12)
+				(bold yes)
+			)
+			(justify left bottom)
+		)
+	)
+	(gr_text "MOUT2"
+		(at 112.776 169.672 0)
+		(layer "F.SilkS" knockout)
+		(effects
+			(font
+				(size 0.7 0.7)
+				(thickness 0.12)
+				(bold yes)
+			)
+			(justify left bottom)
+		)
+	)
+	(gr_text "24V24V24V"
+		(at 121.79 169.95 0)
+		(layer "F.SilkS" knockout)
+		(effects
+			(font
+				(size 1 1)
+				(thickness 0.15)
+			)
+			(justify left bottom)
+		)
+	)
+	(gr_text "5V5V"
+		(at 102.743 165.608 270)
+		(layer "F.SilkS" knockout)
+		(effects
+			(font
+				(size 1 1)
+				(thickness 0.15)
+			)
+			(justify left bottom)
+		)
+	)
+	(gr_text "PWM_IN"
+		(at 102.96775 152.4 270)
+		(layer "F.SilkS" knockout)
+		(effects
+			(font
+				(size 0.7 0.7)
+				(thickness 0.12)
+				(bold yes)
+			)
+			(justify left bottom)
+		)
+	)
+	(segment
+		(start 116.62 120.142)
+		(end 117.099 120.142)
+		(width 0.2)
+		(layer "F.Cu")
+		(net 42)
+	)
 	(embedded_fonts no)

Commit message: ちぇっくかんりょう
Parts:
- moved FET3 0.14 mm to (120.9, 152.7)
Connections:
- J3 pad P: +5V -> GND1
Other:
- board text removed: "5V5V"
Changed lines of the file:
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@@
 	(net 41 "Net-(R4-Pad1)")
 	(net 42 "Net-(R5-Pad1)")
-	(net 43 "+5V")
 	(footprint "Library:R_Axial_DIN0207_L6.3mm_D2.5mm_P10.16mm_Horizontal_kai"
 		(layer "F.Cu")
@@
 			)
 		)
-		(property "Datasheet" ""
+		(property "Datasheet" "~"
 			(at 0 0 180)
 			(unlocked yes)
@@
 			)
 		)
-		(property "Datasheet" ""
+		(property "Datasheet" "~"
 			(at 0 0 0)
 			(layer "F.Fab")
@@
 			)
 		)
-		(property "Datasheet" ""
+		(property "Datasheet" "~"
 			(at 0 0 90)
 			(unlocked yes)
@@
 			)
 		)
-		(property "Datasheet" ""
+		(property "Datasheet" "~"
 			(at 0 0 90)
 			(unlocked yes)
@@
 			)
 		)
-		(property "Datasheet" ""
+		(property "Datasheet" "~"
 			(at 0 0 90)
 			(unlocked yes)
@@
 	(footprint "footprints:PG-TO220-3_INF"
 		(layer "F.Cu")
-		(at 120.7643 152.654 90)
+		(at 120.904 152.654 90)
 		(tags "IRLB3813PBF ")
 		(property "Reference" "FET3"
@@
 			)
 		)
-		(property "Datasheet" ""
+		(property "Datasheet" "~"
 			(at 0 0 90)
 			(unlocked yes)
@@
 			)
 		)
-		(property "Datasheet" ""
+		(property "Datasheet" "~"
 			(at 0 0 0)
 			(layer "F.Fab")
@@
 			)
 		)
-		(property "Datasheet" ""
+		(property "Datasheet" "~"
 			(at 0 0 270)
 			(unlocked yes)
@@
 			)
 		)
-		(property "Datasheet" ""
+		(property "Datasheet" "~"
 			(at 0 0 0)
 			(layer "F.Fab")
@@
 			)
 		)
-		(property "Datasheet" ""
+		(property "Datasheet" "~"
 			(at 0 0 0)
 			(layer "F.Fab")
@@
 			)
 		)
-		(property "Datasheet" ""
+		(property "Datasheet" "~"
 			(at 0 0 0)
 			(unlocked yes)
@@
 			)
 		)
-		(property "Datasheet" ""
+		(property "Datasheet" "~"
 			(at 0 0 90)
 			(unlocked yes)
@@
 			)
 		)
-		(property "Datasheet" ""
+		(property "Datasheet" "~"
 			(at 0 0 90)
 			(layer "F.Fab")
@@
 			)
 		)
-		(property "Datasheet" ""
+		(property "Datasheet" "~"
 			(at 0 0 90)
 			(unlocked yes)
@@
 			)
 		)
-		(property "Datasheet" ""
+		(property "Datasheet" "~"
 			(at 0 0 90)
 			(unlocked yes)
@@
 			)
 		)
-		(property "Datasheet" ""
+		(property "Datasheet" "~"
 			(at 0 0 180)
 			(unlocked yes)
@@
 			)
 		)
-		(property "Datasheet" ""
+		(property "Datasheet" "~"
 			(at 0 0 90)
 			(layer "F.Fab")
@@
 			)
 		)
-		(property "Datasheet" ""
+		(property "Datasheet" "~"
 			(at 0 0 0)
 			(unlocked yes)
@@
 			)
 		)
-		(property "Datasheet" ""
+		(property "Datasheet" "~"
 			(at 0 0 0)
 			(unlocked yes)
@@
 			)
 		)
-		(property "Datasheet" ""
+		(property "Datasheet" "~"
 			(at 0 0 180)
 			(unlocked yes)
@@
 			)
 		)
-		(property "Datasheet" ""
+		(property "Datasheet" "~"
 			(at 0 0 0)
 			(unlocked yes)
@@
 			(layers "*.Cu" "*.Mask")
 			(remove_unused_layers no)
-			(net 43 "+5V")
+			(net 9 "GND1")
 			(pinfunction "P")
 			(pintype "power_in")
@@
 			)
 		)
-		(property "Datasheet" ""
+		(property "Datasheet" "~"
 			(at 0 0 0)
 			(layer "F.Fab")
@@
 			)
 		)
-		(property "Datasheet" ""
+		(property "Datasheet" "~"
 			(at 0 0 90)
 			(unlocked yes)
@@
 			)
 		)
-		(property "Datasheet" ""
+		(property "Datasheet" "~"
 			(at 0 0 90)
 			(unlocked yes)
@@
 			)
 		)
-		(property "Datasheet" ""
+		(property "Datasheet" "~"
 			(at 0 0 0)
 			(unlocked yes)
@@
 			)
 		)
-		(property "Datasheet" ""
+		(property "Datasheet" "~"
 			(at 0 0 0)
 			(layer "F.Fab")
@@
 			)
 		)
-		(property "Datasheet" ""
+		(property "Datasheet" "~"
 			(at 0 0 90)
 			(unlocked yes)
@@
 		(layer "F.SilkS" knockout)
 		(effects
-			(font
-				(size 1 1)
-				(thickness 0.15)
-			)
-			(justify left bottom)
-		)
-	)
-	(gr_text "5V5V"
-		(at 102.743 165.608 270)
-		(layer "F.SilkS" knockout)
-		(effects
