File: MDv3/MDv3.kicad_sch (KiCad schematic)
At the start: 41 parts, among them J1 Conn_01x04_Pin, J3 XT60-M, J4 XT60-M

Commit message: やりなおし
Parts:
- removed J1: Conn_01x04_Pin, Connector_PinHeader_2.54mm:PinHeader_1x04_P2.54mm_Vertical, symbol Connector:Conn_01x04_Pin
- removed J3, J4: XT60-M, XT60-M:AMASS_XT60PW-M, symbol XT60-M:XT60-M
- added J1, J2: XT60PW-M, XT60-M:AMASS_XT60PW-M, symbol XT60PW-M:XT60PW-M
- added J3, J4: XT30PW-M, XT60-M:AMASS_XT30PW-M, symbol XT30UPB-M:XT30PW-M
Connections:
- net +24V: now also J2.1 (+)
- net +5V: now also J3.P
- net DIGITAL_IN: now also J4.N
- net GND1: now also J3.N
- net GND2: now also J2.2 (-)
- net MOUT1: now also J1.1 (+)
- net MOUT2: now also J1.2 (-)
- net PWM_IN: now also J4.P

Commit message: 配線前確認よろしくお願いします！
Parts:
- R1: value 200Ω -> 330Ω
Changed lines of the file:
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@@
 			)
 		)
-		(property "Value" "200Ω"
+		(property "Value" "330Ω"
 			(at 110.49 78.7399 0)
 			(effects

Commit message: ちぇっくかんりょう
Connections:
- net +5V is gone; now on net GND1: J3.P
Changed lines of the file:
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@@
 	(wire
 		(pts
-			(xy 40.64 71.12) (xy 40.64 72.39)
-		)
-		(stroke
-			(width 0)
-			(type default)
-		)
-	)
-	(wire
-		(pts
 			(xy 273.05 57.15) (xy 273.05 69.85)
 		)
@@
 	)
 	(symbol
+		(lib_id "power:GND")
+		(at 40.64 72.39 90)
+		(unit 1)
+		(exclude_from_sim no)
+		(in_bom yes)
+		(on_board yes)
+		(dnp no)
+		(fields_autoplaced yes)
+		(property "Reference" "#PWR010"
+			(at 46.99 72.39 0)
+			(effects
+				(font
+					(size 1.27 1.27)
+				)
+				(hide yes)
+			)
+		)
+		(property "Value" "GND1"
+			(at 44.45 72.3899 90)
+			(effects
+				(font
+					(size 1.27 1.27)
+				)
+				(justify right)
+			)
+		)
+		(property "Footprint" ""
+			(at 40.64 72.39 0)
+			(effects
+				(font
+					(size 1.27 1.27)
+				)
+				(hide yes)
+			)
+		)
+		(property "Datasheet" ""
+			(at 40.64 72.39 0)
+			(effects
+				(font
+					(size 1.27 1.27)
+				)
+				(hide yes)
+			)
+		)
+		(property "Description" "Power symbol creates a global label with name \"GND\" , ground"
+			(at 40.64 72.39 0)
+			(effects
+				(font
+					(size 1.27 1.27)
+				)
+				(hide yes)
+			)
+		)
+		(pin "1"
+		)
+		(instances
+			(project "MDv3"
+				(path "/e92de8da-f869-4b2e-adc8-868d43df9d3b"
+					(reference "#PWR010")
+					(unit 1)
+				)
+			)
+		)
+	)
+	(symbol
 		(lib_id "Device:R")
 		(at 172.72 148.59 0)
@@
 					(unit 1)
 				)
-			)
-		)
-	)
-	(symbol
-		(lib_id "power:+5V")
-		(at 40.64 71.12 0)
-		(unit 1)
-		(exclude_from_sim no)
-		(in_bom yes)
-		(on_board yes)
-		(dnp no)
-		(fields_autoplaced yes)
-		(property "Reference" "#PWR010"
-			(at 40.64 74.93 0)
-			(effects
-				(font
-					(size 1.27 1.27)
-				)
-				(hide yes)
-			)
-		)
-		(property "Value" "+5V"
-			(at 40.64 66.04 0)
-			(effects
-				(font
-					(size 1.27 1.27)
-				)
-			)
-		)
-		(property "Footprint" ""
-			(at 40.64 71.12 0)
-			(effects
-				(font
-					(size 1.27 1.27)
-				)
-				(hide yes)
-			)
-		)
-		(property "Datasheet" ""
-			(at 40.64 71.12 0)
-			(effects
-				(font
-					(size 1.27 1.27)
-				)
-				(hide yes)
-			)
-		)
-		(property "Description" "Power symbol creates a global label with name \"+5V\""
-			(at 40.64 71.12 0)
-			(effects
-				(font
-					(size 1.27 1.27)
-				)
-				(hide yes)
-			)
-		)
-		(pin "1"
-		)
-		(instances
-			(project "MDv3"
-				(path "/e92de8da-f869-4b2e-adc8-868d43df9d3b"
-					(reference "#PWR010")
-					(unit 1)
-				)
