File: MDv3 配線し直し/MDv3.kicad_pcb (KiCad board)
At the start: 2 copper layers, 59.3 x 78.1 mm, 46 parts, among them J1 XT60PW-M, J2 XT60PW-M, J3 XT30PW-M, J4 XT30PW-M

Commit message: 配置変え前
Routing:
- net +5V/2: track 125.9 -> 1.42 mm
- net +12V: track 76.7 -> 1.84 mm
- net PWM_IN: track 68.2 -> 0.00 mm, vias 2 -> 0
- net Net-(FET1-G): track 59.0 -> 0.00 mm, vias 12 -> 0
- net GND1: track 59.0 -> 0.00 mm, vias 1 -> 0
- net DIGITAL_IN: track 54.4 -> 0.06 mm
- net MOUT1: track 42.3 -> 0.00 mm, vias 4 -> 0
- net PWM1: track 33.9 -> 0.00 mm
- net Net-(FET2-G): track 33.0 -> 0.00 mm, vias 3 -> 0
- net DIGITAL: track 26.7 -> 0.00 mm, vias 2 -> 0
- net PWM_NOT: track 25.5 -> 0.26 mm
- net DIGITAL_NOT: track 24.1 -> 0.51 mm
- net GATE1: track 22.4 -> 0.48 mm, vias 4 -> 0
- net Net-(D2-A): track 21.9 -> 0.00 mm
- net Net-(FET4-G): track 19.0 -> 0.00 mm
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- removed copper zone on B.Cu, net +24V
- removed copper zone on B.Cu, net GND1
- removed copper zone on B.Cu, net GND2
- removed copper zone on F.Cu, net GND2
- removed copper zone on F.Cu, net MOUT1
- removed copper zone on F.Cu, net MOUT2

Commit message: 配置変え後
Parts:
- moved R10 8.22 mm to (123.1, 148.4), turned to 180 degrees
- moved R8 8.22 mm to (123.2, 159.8), turned to 180 degrees
- moved R9 7.68 mm to (111.8, 159.7), turned to 180 degrees
- moved R11 7.49 mm to (111.8, 148.4), turned to 180 degrees
- moved FET4 1.14 mm to (110.4, 151.9), turned to 180 degrees
- moved FET2 1.01 mm to (110.5, 163.2), turned to 180 degrees
- moved FET3 0.84 mm to (121.9, 151.8), turned to 180 degrees
- moved FET1 0.65 mm to (121.9, 163.2), turned to 180 degrees
