File: MDv3 配置変え/MDv3.kicad_pcb (KiCad board)
At the start: 2 copper layers, 59.3 x 76.1 mm, 46 parts, among them J1 XT60PW-M, J2 XT60PW-M, J3 XT30PW-M, J4 XT30PW-M

Commit message: MDv3完成、発注に取り掛かる
Parts:
- moved C9 10.7 mm to (123.4, 111.7)
- moved R10 8.22 mm to (123.1, 148.4), turned to 180 degrees
- moved R8 8.22 mm to (123.2, 159.8), turned to 180 degrees
- moved R9 7.68 mm to (111.8, 159.7), turned to 180 degrees
- moved R11 7.49 mm to (111.8, 148.4), turned to 180 degrees
- moved R1 2.21 mm to (102.1, 113.6)
- moved REF** 2.00 mm to (142.0, 113.0)
- moved REF** 2.00 mm to (90.0, 113.0)
- moved R4 1.78 mm to (114.4, 116.9)
- moved R5 1.78 mm to (114.4, 120.7)
- moved D1 1.61 mm to (97.7, 119.4)
- moved FET4 1.14 mm to (110.4, 151.9), turned to 180 degrees
- moved FET2 1.01 mm to (110.5, 163.2), turned to 180 degrees
- moved FET3 0.84 mm to (121.9, 151.8), turned to 180 degrees
- moved FET1 0.65 mm to (121.9, 163.2), turned to 180 degrees
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Routing:
- net GATE2: track 11.8 -> 99.0 mm, vias 0 -> 4
- net GND1: track 0.00 -> 78.7 mm, vias 0 -> 1
- net GATE1: track 20.2 -> 62.0 mm
- net MOUT2: track 40.5 -> 23.1 mm
- net +5V/2: track 114.8 -> 126.3 mm
- net PWM_NOT: track 25.5 -> 36.8 mm, vias 0 -> 3
- net Net-(FET4-G): track 22.5 -> 11.6 mm
- net Net-(D2-A): track 15.6 -> 26.1 mm, vias 2 -> 0
- net Net-(FET3-G): track 15.9 -> 9.13 mm
- net Net-(FET2-G): track 31.9 -> 38.0 mm, vias 1 -> 6
- net PWM_IN: track 64.5 -> 67.8 mm, vias 0 -> 1
- net MOUT1: track 41.4 -> 39.3 mm
- net Net-(D1-A): track 7.92 -> 9.87 mm
- net Net-(FET1-G): track 41.8 -> 43.7 mm, vias 1 -> 2
- net +12V: track 71.4 -> 73.1 mm
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- removed copper zone on B.Cu, net GND1
Other:
- board size 59.3 x 76.1 mm -> 59.3 x 78.1 mm
