File: MD/MDv3/MDv3.kicad_sch (KiCad schematic)
At the start: 42 parts, among them J1 XT60PW-M, J2 XT60PW-M, J3 XT30PW-M, J4 XT30PW-M

Commit message: XT60PW-Mどっかいってもたーください
Parts:
- J3, J4: footprint XT60-M:AMASS_XT30PW-M -> XT30PW-M:AMASS_XT30PW-M
Changed lines of the file:
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@@
 			)
 		)
-		(property "Footprint" "XT60-M:AMASS_XT30PW-M"
+		(property "Footprint" "XT30PW-M:AMASS_XT30PW-M"
 			(at 31.75 80.01 0)
 			(effects
@@
 			)
 		)
-		(property "Footprint" "XT60-M:AMASS_XT30PW-M"
+		(property "Footprint" "XT30PW-M:AMASS_XT30PW-M"
 			(at 31.75 72.39 0)
 			(effects

Commit message: 綺麗になったよ☺
Parts:
- J1, J2: footprint XT60-M:AMASS_XT60PW-M -> XT60PW-M:AMASS_XT60PW-M
Changed lines of the file:
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@@
 			)
 		)
-		(property "Footprint" "XT60-M:AMASS_XT60PW-M"
+		(property "Footprint" "XT60PW-M:AMASS_XT60PW-M"
 			(at 68.58 69.85 0)
 			(effects
@@
 			)
 		)
-		(property "Footprint" "XT60-M:AMASS_XT60PW-M"
+		(property "Footprint" "XT60PW-M:AMASS_XT60PW-M"
 			(at 88.9 69.85 0)
 			(effects
