File: MD/MDv3/MDv3.kicad_pcb (KiCad board)
At the start: 2 copper layers, 59.3 x 78.1 mm, 46 parts, among them J1 XT60PW-M, J2 XT60PW-M, J3 XT30PW-M, J4 XT30PW-M

Commit message: 綺麗になったよ☺
Changed lines of the file:
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@@
 		(start 98.30035 168.108)
 		(end 98.30035 163.108)
-		(width 0.2)
+		(width 0.6)
 		(layer "B.Cu")
 		(net 9)
