File: ESP32-WROOM-32E/ESP32-ROS-IO-V5.0/ESP32-ROS-IO-V5.0.kicad_pcb (KiCad board)
At the start: 2 copper layers, 100 x 100 mm, 60 parts, among them J1 Conn_01x19_Socket, J10 XT30UPB-F, J11 XT30UPB-F, J12 XT30UPB-F, J13 XT30UPB-F, J14 XT30UPB-F, J15 XT30UPB-F, J16 XT60-M, J17 XT60-M, J2 Conn_01x19_Socket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

Commit message: 修正配線済みのメイン基板
Connections:
- R1 pad 1: Net-(R120-Pin_2) -> CANH
Routing:
- net GND: track 0.00 -> 459.9 mm, vias 0 -> 2
- net CANH: track 0.00 -> 172.4 mm, vias 0 -> 1
- net +24V: track 0.00 -> 154.3 mm, vias 0 -> 3
- net GPIO18: track 0.00 -> 150.4 mm, vias 0 -> 3
- net CANL: track 0.00 -> 147.4 mm, vias 0 -> 2
- net GPIO16: track 0.00 -> 144.8 mm
- net 5V: track 0.00 -> 141.0 mm, vias 0 -> 2
- net GPIO15: track 0.00 -> 138.5 mm, vias 0 -> 2
- net GPIO14: track 0.00 -> 131.3 mm
- net GPIO13: track 0.00 -> 120.1 mm
- net GPIO5: track 0.00 -> 110.8 mm
- net GPIO12: track 0.00 -> 103.4 mm
- net GPIO22: track 0.00 -> 102.7 mm, vias 0 -> 1
- net O1: track 0.00 -> 90.7 mm, vias 0 -> 2
- net GPIO17: track 0.00 -> 90.5 mm
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