File: ESP32-WROOM-32E/ESP32-ROS-IO-V5.0/ESP32-ROS-IO-V5.0.kicad_sch (KiCad schematic)
At the start: 54 parts, among them J1 Conn_01x19_Socket, J10 XT30UPB-F, J11 XT30UPB-F, J12 XT30UPB-F, J13 XT30UPB-F, J14 XT30UPB-F, J15 XT30UPB-F, J16 XT60-M, J17 XT60-M, J2 Conn_01x19_Socket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

Commit message: 修正配線済みのメイン基板
Connections:
- net CANH: now also R1.1
- net CANL: now also R120.2 (Pin_2)
Other:
- moved on the sheet: R1, R120
Changed lines of the file:
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@@
 		)
 	)
+	(junction
+		(at 128.27 231.14)
+		(diameter 0)
+		(color 0 0 0 0)
+	)
+	(junction
+		(at 128.27 223.52)
+		(diameter 0)
+		(color 0 0 0 0)
+	)
 	(no_connect
 		(at 133.35 210.82)
@@
 	(wire
 		(pts
+			(xy 128.27 231.14) (xy 124.46 231.14)
+		)
+		(stroke
+			(width 0)
+			(type default)
+		)
+	)
+	(wire
+		(pts
 			(xy 195.58 137.16) (xy 198.12 137.16)
 		)
@@
 	(wire
 		(pts
+			(xy 130.81 228.6) (xy 132.08 228.6)
+		)
+		(stroke
+			(width 0)
+			(type default)
+		)
+	)
+	(wire
+		(pts
 			(xy 77.47 144.78) (xy 67.31 144.78)
 		)
@@
 	(wire
 		(pts
+			(xy 128.27 223.52) (xy 124.46 223.52)
+		)
+		(stroke
+			(width 0)
+			(type default)
+		)
+	)
+	(wire
+		(pts
 			(xy 77.47 132.08) (xy 67.31 132.08)
 		)
@@
 	(wire
 		(pts
-			(xy 77.47 137.16) (xy 67.31 137.16)
+			(xy 130.81 231.14) (xy 128.27 231.14)
 		)
 		(stroke
@@
 	(wire
 		(pts
-			(xy 77.47 149.86) (xy 67.31 149.86)
+			(xy 77.47 137.16) (xy 67.31 137.16)
 		)
 		(stroke
@@
 	(wire
 		(pts
-			(xy 77.47 160.02) (xy 67.31 160.02)
+			(xy 77.47 149.86) (xy 67.31 149.86)
 		)
 		(stroke
@@
 	(wire
 		(pts
-			(xy 124.46 233.68) (xy 124.46 234.95)
+			(xy 77.47 160.02) (xy 67.31 160.02)
 		)
 		(stroke
@@
 	(wire
 		(pts
+			(xy 130.81 231.14) (xy 130.81 228.6)
+		)
+		(stroke
+			(width 0)
+			(type default)
+		)
+	)
+	(wire
+		(pts
 			(xy 73.66 234.95) (xy 77.47 234.95)
 		)
@@
 	(wire
 		(pts
+			(xy 132.08 226.06) (xy 130.81 226.06)
+		)
+		(stroke
+			(width 0)
+			(type default)
+		)
+	)
+	(wire
+		(pts
 			(xy 198.12 181.61) (xy 195.58 181.61)
 		)
@@
 	(wire
 		(pts
+			(xy 130.81 226.06) (xy 130.81 223.52)
+		)
+		(stroke
+			(width 0)
+			(type default)
+		)
+	)
+	(wire
+		(pts
 			(xy 67.31 234.95) (xy 71.12 234.95)
 		)
@@
 	(wire
 		(pts
+			(xy 130.81 223.52) (xy 128.27 223.52)
+		)
+		(stroke
+			(width 0)
+			(type default)
+		)
+	)
+	(wire
+		(pts
 			(xy 121.92 135.89) (xy 121.92 137.16)
 		)
@@
 	(global_label "CANL"
 		(shape input)
-		(at 124.46 234.95 180)
+		(at 124.46 231.14 180)
 		(fields_autoplaced yes)
 		(effects
@@
 		)
 		(property "Intersheetrefs" "${INTERSHEET_REFS}"
-			(at 116.7576 234.95 0)
+			(at 116.7576 231.14 0)
 			(effects
 				(font
@@
 	(symbol
 		(lib_id "Device:R")
-		(at 124.46 229.87 0)
+		(at 128.27 227.33 0)
 		(unit 1)
 		(exclude_from_sim no)
@@
 		(on_board yes)
 		(dnp no)
-		(fields_autoplaced yes)
 		(property "Reference" "R1"
-			(at 127 228.5999 0)
+			(at 123.19 226.06 0)
 			(effects
 				(font
@@
 		)
 		(property "Value" "120"
-			(at 127 231.1399 0)
+			(at 123.19 228.6 0)
 			(effects
 				(font
@@
 		)
 		(property "Footprint" "Resistor_THT:R_Axial_DIN0207_L6.3mm_D2.5mm_P10.16mm_Horizontal"
-			(at 122.682 229.87 90)
+			(at 126.492 227.33 90)
 			(effects
 				(font
@@
 		)
 		(property "Datasheet" "~"
-			(at 124.46 229.87 0)
+			(at 128.27 227.33 0)
 			(effects
 				(font
@@
 		)
 		(property "Description" "Resistor"
-			(at 124.46 229.87 0)
+			(at 128.27 227.33 0)
 			(effects
 				(font
@@
 	(symbol
 		(lib_id "Connector:Conn_01x02_Pin")
-		(at 129.54 223.52 0)
+		(at 137.16 226.06 0)
 		(mirror y)
 		(unit 1)
@@
 		(fields_autoplaced yes)
 		(property "Reference" "R120"
-			(at 130.81 223.5199 0)
+			(at 138.43 226.0599 0)
 			(effects
 				(font
@@
 		)
 		(property "Value" "R120"
-			(at 130.81 226.0599 0)
+			(at 138.43 228.5999 0)
 			(effects
 				(font
@@
 		)
 		(property "Footprint" "Connector_PinHeader_2.54mm:PinHeader_1x02_P2.54mm_Vertical"
-			(at 129.54 223.52 0)
+			(at 137.16 226.06 0)
 			(effects
 				(font
@@
 		)
 		(property "Datasheet" "~"
-			(at 129.54 223.52 0)
+			(at 137.16 226.06 0)
 			(effects
 				(font
@@
 		)
 		(property "Description" "Generic connector, single row, 01x02, script generated"
-			(at 129.54 223.52 0)
+			(at 137.16 226.06 0)
 			(effects
 				(font
