File: ESP32-WROOM-32E/ESP32-S3-ROS-IO-V1.0/ESP32-S3-ROS-IO-V1.0.kicad_pcb (KiCad board)
At the start: 2 copper layers, 100 x 100 mm, 53 parts, among them J1 Conn_01x22_Socket, J16 XT60-M, J17 XT60-M, J2 Conn_01x22_Socket, J3 Conn_01x22_Socket, J4 Conn_01x22_Socket, SW1 SW1, SW2 SW2, SW3 SW3, SW4 SW4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

Commit message: 自動配線後
Routing:
- net CANL: track 0.00 -> 201.6 mm
- net CANH: track 0.00 -> 200.1 mm
- net +24V: track 0.00 -> 178.0 mm, vias 0 -> 1
- net TR6_Bypass_OUT: track 0.00 -> 129.6 mm, vias 0 -> 2
- net O5: track 0.00 -> 115.1 mm, vias 0 -> 1
- net TR6/SW2: track 0.00 -> 114.9 mm, vias 0 -> 2
- net O6: track 0.00 -> 111.6 mm, vias 0 -> 1
- net O1: track 0.00 -> 110.9 mm, vias 0 -> 1
- net O2: track 0.00 -> 104.6 mm, vias 0 -> 2
- net O7: track 0.00 -> 103.8 mm, vias 0 -> 1
- net O3: track 0.00 -> 101.6 mm, vias 0 -> 1
- net O4: track 0.00 -> 99.9 mm, vias 0 -> 1
- net GPIO10: track 0.00 -> 99.2 mm, vias 0 -> 1
- net GPIO11: track 0.00 -> 89.7 mm, vias 0 -> 1
- net GPIO41: track 0.00 -> 86.0 mm, vias 0 -> 1
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Other:
- board text added: "ESP32-S3-DevKitC V1"
- board text added: "ESP32-S3-IO-Board-V1.0 2026, NHK-Project, RRST"
- board text removed: "ESP32-IO-Board-V6.0 2026, NHK-Project, RRST"
- board text removed: "ESP32-S3-DevKitC V6"

Commit message: atohaisenikko
Routing:
- net GPIO4: track 73.7 -> 75.1 mm
- net CAN_RX: vias 1 -> 2
- net TR6/SW2: vias 2 -> 4
- net GPIO38: vias 0 -> 2
- net GPIO35: vias 0 -> 2
- net CANH: vias 0 -> 3
Changed lines of the file:
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@@
 	)
 	(segment
+		(start 115.9226 65.6336)
+		(end 115.9226 68.7832)
+		(width 0.2)
+		(layer "F.Cu")
+		(net 1)
+	)
+	(segment
 		(start 120.1225 41.6851)
 		(end 118.7716 43.036)
@@
 	)
 	(segment
-		(start 116.6862 73.4168)
-		(end 115.3838 72.1144)
+		(start 116.487 95.25)
+		(end 122.837 101.6)
 		(width 0.2)
-		(layer "B.Cu")
+		(layer "F.Cu")
+		(net 1)
+	)
+	(via
+		(at 116.487 95.25)
+		(size 0.6)
+		(drill 0.3)
+		(layers "F.Cu" "B.Cu")
+		(net 1)
+	)
+	(via
+		(at 115.9226 68.7832)
+		(size 0.6)
+		(drill 0.3)
+		(layers "F.Cu" "B.Cu")
+		(net 1)
+	)
+	(via
+		(at 115.9226 65.6336)
+		(size 0.6)
+		(drill 0.3)
+		(layers "F.Cu" "B.Cu")
 		(net 1)
 	)
 	(segment
-		(start 109.26 26.526)
-		(end 109.26 34.781)
+		(start 116.6862 73.4168)
+		(end 115.3838 72.1144)
 		(width 0.2)
 		(layer "B.Cu")
@@
 	)
 	(segment
-		(start 122.837 101.6)
-		(end 116.487 95.25)
+		(start 109.26 26.526)
+		(end 109.26 34.781)
 		(width 0.2)
 		(layer "B.Cu")
@@
 	)
 	(segment
+		(start 115.9226 65.6336)
+		(end 115.9226 45.885)
+		(width 0.2)
+		(layer "B.Cu")
+		(net 1)
+	)
+	(segment
 		(start 115.3838 72.1144)
 		(end 115.3838 70.5158)
@@
 	(segment
 		(start 115.9226 69.977)
-		(end 115.9226 45.885)
+		(end 115.9226 68.7832)
 		(width 0.2)
 		(layer "B.Cu")
@@
 	)
 	(segment
-		(start 100.9093 68.4276)
+		(start 127.3526 69.5)
 		(end 128.425 68.4276)
 		(width 0.2)
@@
 	(segment
 		(start 97.9699 71.367)
-		(end 100.9093 68.4276)
+		(end 99.8369 69.5)
+		(width 0.2)
+		(layer "F.Cu")
+		(net 15)
+	)
+	(segment
+		(start 99.8369 69.5)
+		(end 127.3526 69.5)
 		(width 0.2)
 		(layer "F.Cu")
@@
 	)
 	(segment
-		(start 96.8669 95.0635)
-		(end 96.8669 72.47)
+		(start 99.5 72.8971)
+		(end 97.9699 71.367)
 		(width 0.2)
 		(layer "B.Cu")
@@
 	)
 	(segment
-		(start 96.8669 72.47)
-		(end 97.9699 71.367)
+		(start 98.0186 96.2152)
+		(end 99.5 94.7338)
 		(width 0.2)
 		(layer "B.Cu")
@@
 	)
 	(segment
-		(start 98.0186 96.2152)
-		(end 96.8669 95.0635)
+		(start 99.5 94.7338)
+		(end 99.5 72.8971)
 		(width 0.2)
 		(layer "B.Cu")
@@
 		(net 18)
 	)
+	(segment
+		(start 116.363 97.0221)
+		(end 116.363 105.534)
+		(width 0.2)
+		(layer "F.Cu")
+		(net 18)
+	)
+	(segment
+		(start 116.363 105.534)
+		(end 115.217 106.68)
+		(width 0.2)
+		(layer "F.Cu")
+		(net 18)
+	)
 	(via
-		(at 115.852 91.9967)
+		(at 116.363 97.0221)
 		(size 0.6)
 		(drill 0.3)
@@
 		(net 18)
 	)
-	(segment
-		(start 116.363 105.534)
-		(end 116.363 97.0221)
-		(width 0.2)
-		(layer "B.Cu")
+	(via
+		(at 115.852 91.9967)
+		(size 0.6)
+		(drill 0.3)
+		(layers "F.Cu" "B.Cu")
 		(net 18)
 	)
@@
 	)
 	(segment
-		(start 115.217 106.68)
-		(end 116.363 105.534)
-		(width 0.2)
-		(layer "B.Cu")
-		(net 18)
-	)
-	(segment
 		(start 128.425 109.0676)
 		(end 132.207 109.0676)
@@
 	)
 	(segment
-		(start 100.853 65.8876)
+		(start 127.5374 65)
 		(end 128.425 65.8876)
 		(width 0.2)
@@
 	)
 	(segment
+		(start 101.7406 65)
+		(end 127.5374 65)
+		(width 0.2)
+		(layer "F.Cu")
+		(net 22)
+	)
+	(segment
 		(start 98.3207 68.4199)
-		(end 100.853 65.8876)
+		(end 101.7406 65)
 		(width 0.2)
 		(layer "F.Cu")
@@
 	)
 	(segment
-		(start 99.1926 105.2012)
-		(end 99.1926 69.2918)
+		(start 100 70.0992)
+		(end 98.3207 68.4199)
 		(width 0.2)
 		(layer "B.Cu")
@@
 	)
 	(segment
-		(start 98.0186 106.3752)
-		(end 99.1926 105.2012)
+		(start 100 104.3938)
+		(end 100 70.0992)
 		(width 0.2)
 		(layer "B.Cu")
@@
 	)
 	(segment
-		(start 99.1926 69.2918)
-		(end 98.3207 68.4199)
+		(start 98.0186 106.3752)
+		(end 100 104.3938)
 		(width 0.2)
 		(layer "B.Cu")
@@
 	)
 	(segment
+		(start 164.93935 51.40135)
+		(end 163.00895 53.33175)
+		(width 0.2)
+		(layer "F.Cu")
+		(net 36)
+	)
+	(segment
 		(start 161.389 88.7476)
 		(end 157.607 88.7476)
@@
 		(net 36)
 	)
+	(via
+		(at 163.00895 53.33175)
+		(size 0.6)
+		(drill 0.3)
+		(layers "F.Cu" "B.Cu")
+		(net 36)
+	)
+	(via
+		(at 164.93935 51.40135)
+		(size 0.6)
+		(drill 0.3)
+		(layers "F.Cu" "B.Cu")
+		(net 36)
+	)
 	(segment
 		(start 157.607 88.7476)
@@
 	(segment
 		(start 159.2291 57.1116)
+		(end 163.00895 53.33175)
+		(width 0.2)
+		(layer "B.Cu")
+		(net 36)
+	)
+	(segment
+		(start 164.93935 51.40135)
 		(end 167.6275 48.7132)
 		(width 0.2)
@@
 	)
 	(segment
+		(start 158.7909 51.3846)
+		(end 158.7909 53.3517)
+		(width 0.2)
+		(layer "F.Cu")
+		(net 40)
+	)
+	(via
+		(at 158.7909 51.3846)
+		(size 0.6)
+		(drill 0.3)
+		(layers "F.Cu" "B.Cu")
+		(net 40)
+	)
+	(via
+		(at 158.7909 53.3517)
+		(size 0.6)
+		(drill 0.3)
+		(layers "F.Cu" "B.Cu")
+		(net 40)
+	)
+	(segment
+		(start 158.7909 50.6951)
+		(end 161.9623 47.5237)
+		(width 0.2)
+		(layer "B.Cu")
+		(net 40)
+	)
+	(segment
 		(start 161.9623 47.5237)
 		(end 166.45 43.036)
@@
 	)
 	(segment
-		(start 158.7909 50.6951)
-		(end 161.9623 47.5237)
+		(start 158.7909 79.9437)
+		(end 157.607 81.1276)
 		(width 0.2)
 		(layer "B.Cu")
@@
 	)
 	(segment
-		(start 158.7909 79.9437)
+		(start 158.7909 51.3846)
 		(end 158.7909 50.6951)
 		(width 0.2)
@@
 	)
 	(segment
-		(start 157.607 81.1276)
+		(start 158.7909 53.3517)
 		(end 158.7909 79.9437)
 		(width 0.2)
@@
 	)
 	(segment
+		(start 168.4855 62.6872)
+		(end 168.4855 65.1764)
+		(width 0.2)
+		(layer "F.Cu")
+		(net 46)
+	)
+	(segment
 		(start 169.0057 48.0445)
 		(end 176.2627 48.0445)
@@
 	)
 	(via
+		(at 168.4855 65.1764)
+		(size 0.6)
+		(drill 0.3)
+		(layers "F.Cu" "B.Cu")
+		(net 46)
+	)
+	(via
+		(at 168.4855 62.6872)
+		(size 0.6)
+		(drill 0.3)
+		(layers "F.Cu" "B.Cu")
+		(net 46)
+	)
+	(via
 		(at 168.8124 47.8512)
 		(size 0.6)
@@
 	)
 	(segment
+		(start 168.4855 65.1764)
+		(end 168.4855 76.8612)
+		(width 0.2)
+		(layer "B.Cu")
+		(net 46)
+	)
+	(segment
 		(start 168.4001 77.8407)
 		(end 168.88 78.3206)
@@
 	(segment
 		(start 168.4855 48.1781)
-		(end 168.4855 76.8612)
+		(end 168.4855 62.6872)
 		(width 0.2)
 		(layer "B.Cu")
@@
 		(polygon
 			(pts
-				(xy 97 14.5) (xy 191.5 14.5) (xy 193.5 16.5) (xy 193.5 111.5) (xy 191.5 113.5) (xy 96.5 113.5) (xy 94.5 111.5)
-				(xy 94.5 17)
+				(xy 191.5 14.5) (xy 193.5 16.5) (xy 193.5 111.5) (xy 191.5 113.5) (xy 186 113.5) (xy 186 106) (xy 178 106)
+				(xy 178 113.5) (xy 111.5 113.5) (xy 111.5 106.5) (xy 103.5 106.5) (xy 103.5 113.5) (xy 96.5 113.5)
+				(xy 94.5 111.5) (xy 94.5 55.5) (xy 111 55.5) (xy 111 48.5) (xy 105.5 48.5) (xy 105.5 14.5)
 			)
 		)

Commit message: dekitayo
Routing:
- net TR6_Bypass_OUT: vias 2 -> 4
- net O3: vias 1 -> 3
- net GPIO48: vias 0 -> 2
- net ENC3_A: vias 1 -> 3
- net +24V: vias 1 -> 3
Changed lines of the file:
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@@
 		(net 12)
 	)
+	(segment
+		(start 171.1673 55.718)
+		(end 171.1673 59.3852)
+		(width 0.2)
+		(layer "F.Cu")
+		(net 12)
+	)
+	(via
+		(at 171.1673 59.3852)
+		(size 0.6)
+		(drill 0.3)
+		(layers "F.Cu" "B.Cu")
+		(net 12)
+	)
 	(via
 		(at 169.0511 77.2612)
@@
 		(net 12)
 	)
+	(via
+		(at 171.1673 55.718)
+		(size 0.6)
+		(drill 0.3)
+		(layers "F.Cu" "B.Cu")
+		(net 12)
+	)
+	(segment
+		(start 171.1673 55.718)
+		(end 171.1673 52.832)
+		(width 0.2)
+		(layer "B.Cu")
+		(net 12)
+	)
+	(segment
+		(start 171.1673 52.832)
+		(end 172.319 52.832)
+		(width 0.2)
+		(layer "B.Cu")
+		(net 12)
+	)
 	(segment
 		(start 171.1673 75.145)
-		(end 171.1673 52.832)
-		(width 0.2)
-		(layer "B.Cu")
-		(net 12)
-	)
-	(segment
-		(start 172.319 52.832)
-		(end 171.1673 52.832)
+		(end 171.1673 59.3852)
 		(width 0.2)
 		(layer "B.Cu")
@@
 	)
 	(segment
+		(start 176.1744 55.718)
+		(end 176.1744 59.4868)
+		(width 0.2)
+		(layer "F.Cu")
+		(net 31)
+	)
+	(via
+		(at 176.1744 59.4868)
+		(size 0.6)
+		(drill 0.3)
+		(layers "F.Cu" "B.Cu")
+		(net 31)
+	)
+	(via
+		(at 176.1744 55.718)
+		(size 0.6)
+		(drill 0.3)
+		(layers "F.Cu" "B.Cu")
+		(net 31)
+	)
+	(segment
+		(start 167.748 104.4841)
+		(end 173.739 98.4931)
+		(width 0.2)
+		(layer "B.Cu")
+		(net 31)
+	)
+	(segment
+		(start 173.739 97.8454)
+		(end 174.5564 97.028)
+		(width 0.2)
+		(layer "B.Cu")
+		(net 31)
+	)
+	(segment
+		(start 176.5738 50.535657)
+		(end 176.7332 50.376257)
+		(width 0.2)
+		(layer "B.Cu")
+		(net 31)
+	)
+	(segment
 		(start 161.389 96.3676)
 		(end 165.623 100.6016)
@@
 	)
 	(segment
+		(start 176.7332 45.9158)
+		(end 178.707 43.942)
+		(width 0.2)
+		(layer "B.Cu")
+		(net 31)
+	)
+	(segment
+		(start 166.7991 104.4841)
+		(end 167.748 104.4841)
+		(width 0.2)
+		(layer "B.Cu")
+		(net 31)
+	)
+	(segment
+		(start 176.7332 50.376257)
+		(end 176.7332 45.9158)
+		(width 0.2)
+		(layer "B.Cu")
+		(net 31)
+	)
+	(segment
+		(start 175.2843 97.028)
+		(end 176.1744 96.1379)
+		(width 0.2)
+		(layer "B.Cu")
+		(net 31)
+	)
+	(segment
+		(start 165.623 103.308)
+		(end 166.7991 104.4841)
+		(width 0.2)
+		(layer "B.Cu")
+		(net 31)
+	)
+	(segment
 		(start 173.739 98.4931)
 		(end 173.739 97.8454)
@@
 	)
 	(segment
+		(start 176.1744 51.432943)
+		(end 176.5738 51.033543)
+		(width 0.2)
+		(layer "B.Cu")
+		(net 31)
+	)
+	(segment
+		(start 165.623 100.6016)
+		(end 165.623 103.308)
+		(width 0.2)
+		(layer "B.Cu")
+		(net 31)
+	)
+	(segment
+		(start 176.5738 51.033543)
+		(end 176.5738 50.535657)
+		(width 0.2)
+		(layer "B.Cu")
+		(net 31)
+	)
+	(segment
+		(start 176.1744 55.718)
+		(end 176.1744 51.432943)
+		(width 0.2)
+		(layer "B.Cu")
+		(net 31)
+	)
+	(segment
 		(start 174.5564 97.028)
 		(end 175.2843 97.028)
@@
 	)
 	(segment
-		(start 167.748 104.4841)
-		(end 173.739 98.4931)
-		(width 0.2)
-		(layer "B.Cu")
-		(net 31)
-	)
-	(segment
-		(start 166.7991 104.4841)
-		(end 167.748 104.4841)
-		(width 0.2)
-		(layer "B.Cu")
-		(net 31)
-	)
-	(segment
-		(start 176.1548 96.1575)
-		(end 176.1548 46.4942)
-		(width 0.2)
-		(layer "B.Cu")
-		(net 31)
-	)
-	(segment
-		(start 165.623 103.308)
-		(end 166.7991 104.4841)
-		(width 0.2)
-		(layer "B.Cu")
-		(net 31)
-	)
-	(segment
-		(start 165.623 100.6016)
-		(end 165.623 103.308)
-		(width 0.2)
-		(layer "B.Cu")
-		(net 31)
-	)
-	(segment
-		(start 176.1548 46.4942)
-		(end 178.707 43.942)
-		(width 0.2)
-		(layer "B.Cu")
-		(net 31)
-	)
-	(segment
-		(start 173.739 97.8454)
-		(end 174.5564 97.028)
-		(width 0.2)
-		(layer "B.Cu")
-		(net 31)
-	)
-	(segment
-		(start 175.2843 97.028)
-		(end 176.1548 96.1575)
+		(start 176.1744 96.1379)
+		(end 176.1744 59.4868)
 		(width 0.2)
 		(layer "B.Cu")
@@
 	)
 	(segment
+		(start 177.0011 55.718)
+		(end 177.0011 59.5376)
+		(width 0.2)
+		(layer "F.Cu")
+		(net 45)
+	)
+	(segment
 		(start 177.1748 50.7846)
 		(end 153.8692 50.7846)
@@
 	)
 	(via
+		(at 177.0011 59.5376)
+		(size 0.6)
+		(drill 0.3)
+		(layers "F.Cu" "B.Cu")
+		(net 45)
+	)
+	(via
 		(at 177.1748 50.7846)
 		(size 0.6)
@@
 	(via
 		(at 153.8692 50.7846)
+		(size 0.6)
+		(drill 0.3)
+		(layers "F.Cu" "B.Cu")
+		(net 45)
+	)
+	(via
+		(at 177.0011 55.718)
 		(size 0.6)
 		(drill 0.3)
@@
 	)
 	(segment
-		(start 177.0011 50.9583)
+		(start 177.0011 59.5376)
 		(end 177.0011 97.8068)
+		(width 0.2)
+		(layer "B.Cu")
+		(net 45)
+	)
+	(segment
+		(start 177.0011 55.718)
+		(end 177.0011 50.9583)
 		(width 0.2)
 		(layer "B.Cu")
@@
 	)
 	(segment
-		(start 177.1748 50.7846)
-		(end 177.0011 50.9583)
-		(width 0.2)
-		(layer "B.Cu")
-		(net 45)
-	)
-	(segment
 		(start 173.642 99.568)
 		(end 167.292 105.918)
@@
 		(start 177.1748 50.7846)
 		(end 177.1748 47.3742)
+		(width 0.2)
+		(layer "B.Cu")
+		(net 45)
+	)
+	(segment
+		(start 177.0011 50.9583)
+		(end 177.1748 50.7846)
 		(width 0.2)
 		(layer "B.Cu")
@@
 	)
 	(segment
+		(start 178.2045 55.718)
+		(end 178.2045 60.0456)
+		(width 0.2)
+		(layer "F.Cu")
+		(net 48)
+	)
+	(segment
 		(start 178.0308 48.2501)
 		(end 177.8265 48.4544)
@@
 	)
 	(via
+		(at 178.2045 60.0456)
+		(size 0.6)
+		(drill 0.3)
+		(layers "F.Cu" "B.Cu")
+		(net 48)
+	)
+	(via
+		(at 178.2045 55.718)
+		(size 0.6)
+		(drill 0.3)
+		(layers "F.Cu" "B.Cu")
+		(net 48)
+	)
+	(via
 		(at 178.0308 48.2501)
 		(size 0.6)
@@
 	)
 	(segment
+		(start 178.2045 55.718)
+		(end 178.2045 48.4238)
+		(width 0.2)
+		(layer "B.Cu")
+		(net 48)
+	)
+	(segment
 		(start 178.2045 105.1655)
-		(end 178.2045 48.4238)
+		(end 178.2045 60.0456)
 		(width 0.2)
 		(layer "B.Cu")
@@
 	)
 	(segment
+		(start 178.2045 48.4238)
+		(end 178.0308 48.2501)
+		(width 0.2)
+		(layer "B.Cu")
+		(net 48)
+	)
+	(segment
 		(start 140.0537 33.2488)
 		(end 140.1572 33.3523)
@@
 	)
 	(segment
-		(start 178.2045 48.4238)
-		(end 178.0308 48.2501)
-		(width 0.2)
-		(layer "B.Cu")
-		(net 48)
-	)
-	(segment
 		(start 140.1572 26.526)
 		(end 140.0537 26.6295)
@@
 	)
 	(segment
+		(start 173.569 55.718)
+		(end 173.569 59.2328)
+		(width 0.2)
+		(layer "F.Cu")
+		(net 51)
+	)
+	(segment
 		(start 169.1261 39.5072)
 		(end 133.0866 39.5072)
@@
 	)
 	(via
+		(at 173.569 59.2328)
+		(size 0.6)
+		(drill 0.3)
+		(layers "F.Cu" "B.Cu")
+		(net 51)
+	)
+	(via
 		(at 169.1261 39.5072)
 		(size 0.6)
@@
 		(net 51)
 	)
+	(via
+		(at 173.569 55.718)
+		(size 0.6)
+		(drill 0.3)
+		(layers "F.Cu" "B.Cu")
+		(net 51)
+	)
 	(segment
 		(start 173.569 94.415)
+		(end 173.569 59.2328)
+		(width 0.2)
+		(layer "B.Cu")
+		(net 51)
+	)
+	(segment
+		(start 170.1483 40.5294)
+		(end 169.1261 39.5072)
+		(width 0.2)
+		(layer "B.Cu")
+		(net 51)
+	)
+	(segment
+		(start 173.569 46.9959)
+		(end 170.1483 43.5752)
+		(width 0.2)
+		(layer "B.Cu")
+		(net 51)
+	)
+	(segment
+		(start 174.912 95.758)
+		(end 173.569 94.415)
+		(width 0.2)
+		(layer "B.Cu")
+		(net 51)
+	)
+	(segment
+		(start 173.569 55.718)
 		(end 173.569 46.9959)
 		(width 0.2)
@@
 		(width 0.2)
 		(layer "B.Cu")
-		(net 51)
-	)
-	(segment
-		(start 170.1483 40.5294)
-		(end 169.1261 39.5072)
-		(width 0.2)
-		(layer "B.Cu")
-		(net 51)
-	)
-	(segment
-		(start 174.912 95.758)
-		(end 173.569 94.415)
-		(width 0.2)
-		(layer "B.Cu")
-		(net 51)
-	)
-	(segment
-		(start 173.569 46.9959)
-		(end 170.1483 43.5752)
-		(width 0.2)
-		(layer "B.Cu")

Commit message: yarinaoshi
Routing:
- net CANL: track 201.6 -> 0.00 mm
- net CANH: track 200.1 -> 0.00 mm, vias 3 -> 0
- net +24V: track 178.0 -> 0.00 mm, vias 3 -> 0
- net TR6_Bypass_OUT: track 129.6 -> 0.00 mm, vias 4 -> 0
- net O5: track 115.1 -> 0.00 mm, vias 1 -> 0
- net TR6/SW2: track 114.9 -> 0.00 mm, vias 4 -> 0
- net O6: track 111.6 -> 0.00 mm, vias 1 -> 0
- net O1: track 110.9 -> 0.00 mm, vias 1 -> 0
- net O2: track 104.6 -> 0.00 mm, vias 2 -> 0
- net O7: track 103.8 -> 0.00 mm, vias 1 -> 0
- net O3: track 101.6 -> 0.00 mm, vias 3 -> 0
- net O4: track 99.9 -> 0.00 mm, vias 1 -> 0
- net GPIO10: track 99.2 -> 0.00 mm, vias 1 -> 0
- net GPIO11: track 89.7 -> 0.00 mm, vias 1 -> 0
- net GPIO41: track 86.0 -> 0.00 mm, vias 1 -> 0
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
Commit message: 自動配線前
Parts:
- renumbered TR7_EN to J5, TR6_EN to J6, 120R_EN to R120
Connections:
- ENC1 pad 1: VDD33 -> 5VD
- ENC2 pad 1: VDD33 -> 5VD
- ENC3 pad 1: VDD33 -> 5VD
- ENC4 pad 1: VDD33 -> 5VD

Commit message: kansei?
Routing:
- net CANL: track 0.00 -> 210.4 mm
- net CANH: track 0.00 -> 199.3 mm
- net +24V: track 0.00 -> 190.2 mm, vias 0 -> 2
- net TR6_Bypass_OUT: track 0.00 -> 131.3 mm, vias 0 -> 4
- net 5VD: track 0.00 -> 121.7 mm, vias 0 -> 2
- net TR6/SW2: track 0.00 -> 120.4 mm, vias 0 -> 4
- net O5: track 0.00 -> 116.1 mm, vias 0 -> 1
- net O1: track 0.00 -> 114.4 mm, vias 0 -> 1
- net O6: track 0.00 -> 108.4 mm, vias 0 -> 1
- net O2: track 0.00 -> 108.3 mm, vias 0 -> 3
- net O3: track 0.00 -> 107.3 mm, vias 0 -> 3
- net O7: track 0.00 -> 105.5 mm, vias 0 -> 1
- net GPIO11: track 0.00 -> 101.8 mm, vias 0 -> 1
- net GPIO10: track 0.00 -> 101.5 mm, vias 0 -> 3
- net O4: track 0.00 -> 100.9 mm, vias 0 -> 5
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
Commit message: 発注する
Routing:
- net GND: vias 0 -> 22
Changed lines of the file:
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@@
 		(net 6)
+	)
+	(via
+		(at 99.9744 60.5536)
+		(size 0.6)
+		(drill 0.3)
+		(layers "F.Cu" "B.Cu")
+		(free yes)
+		(net 7)
+	)
+	(via
+		(at 163.0172 23.2664)
+		(size 0.6)
+		(drill 0.3)
+		(layers "F.Cu" "B.Cu")
+		(free yes)
+		(net 7)
+	)
+	(via
+		(at 184.2008 97.2312)
+		(size 0.6)
+		(drill 0.3)
+		(layers "F.Cu" "B.Cu")
+		(free yes)
+		(net 7)
+	)
+	(via
+		(at 146.1008 109.5756)
+		(size 0.6)
+		(drill 0.3)
+		(layers "F.Cu" "B.Cu")
+		(free yes)
+		(net 7)
+	)
+	(via
+		(at 162.9664 39.2176)
+		(size 0.6)
+		(drill 0.3)
+		(layers "F.Cu" "B.Cu")
+		(free yes)
+		(net 7)
+	)
+	(via
+		(at 124.6632 22.9108)
+		(size 0.6)
+		(drill 0.3)
+		(layers "F.Cu" "B.Cu")
+		(free yes)
+		(net 7)
+	)
+	(via
+		(at 150.8252 59.0296)
+		(size 0.6)
+		(drill 0.3)
+		(layers "F.Cu" "B.Cu")
+		(free yes)
+		(net 7)
+	)
+	(via
+		(at 143.8148 39.1668)
+		(size 0.6)
+		(drill 0.3)
+		(layers "F.Cu" "B.Cu")
+		(free yes)
+		(net 7)
+	)
+	(via
+		(at 183.9468 80.2132)
+		(size 0.6)
+		(drill 0.3)
+		(layers "F.Cu" "B.Cu")
+		(free yes)
+		(net 7)
+	)
+	(via
+		(at 110.2868 99.9744)
+		(size 0.6)
+		(drill 0.3)
+		(layers "F.Cu" "B.Cu")
+		(free yes)
+		(net 7)
+	)
+	(via
+		(at 143.9672 23.0632)
+		(size 0.6)
+		(drill 0.3)
+		(layers "F.Cu" "B.Cu")
+		(free yes)
+		(net 7)
+	)
+	(via
+		(at 152.8572 39.2176)
+		(size 0.6)
+		(drill 0.3)
+		(layers "F.Cu" "B.Cu")
+		(free yes)
+		(net 7)
+	)
+	(via
+		(at 142.9512 58.2168)
+		(size 0.6)
+		(drill 0.3)
+		(layers "F.Cu" "B.Cu")
+		(free yes)
+		(net 7)
+	)
+	(via
+		(at 109.9312 78.7908)
+		(size 0.6)
+		(drill 0.3)
+		(layers "F.Cu" "B.Cu")
+		(free yes)
+		(net 7)
+	)
+	(via
+		(at 192.1256 28.6004)
+		(size 0.6)
+		(drill 0.3)
+		(layers "F.Cu" "B.Cu")
+		(free yes)
+		(net 7)
+	)
+	(via
+		(at 115.1128 39.4716)
+		(size 0.6)
+		(drill 0.3)
+		(layers "F.Cu" "B.Cu")
+		(free yes)
+		(net 7)
+	)
+	(via
+		(at 134.2644 23.0632)
+		(size 0.6)
+		(drill 0.3)
+		(layers "F.Cu" "B.Cu")
+		(free yes)
+		(net 7)
+	)
+	(via
+		(at 115.062 22.9616)
+		(size 0.6)
+		(drill 0.3)
+		(layers "F.Cu" "B.Cu")
+		(free yes)
+		(net 7)
+	)
+	(via
+		(at 189.4332 49.1744)
+		(size 0.6)
+		(drill 0.3)
+		(layers "F.Cu" "B.Cu")
+		(free yes)
+		(net 7)
+	)
+	(via
+		(at 124.8156 39.2176)
+		(size 0.6)
+		(drill 0.3)
+		(layers "F.Cu" "B.Cu")
+		(free yes)
+		(net 7)
+	)
+	(via
+		(at 134.112 39.0144)
+		(size 0.6)
+		(drill 0.3)
+		(layers "F.Cu" "B.Cu")
+		(free yes)
+		(net 7)
+	)
+	(via
+		(at 147.2184 92.9132)
+		(size 0.6)
+		(drill 0.3)
+		(layers "F.Cu" "B.Cu")
+		(free yes)
+		(net 7)
 	)
 	(segment
