File: RRST-ESP32-S3-Rev.1/RRST-ESP32-S3-Rev.1.kicad_sch (KiCad schematic)
At the start: 29 parts, among them J1 Conn_01x22_Pin, J2 USB_C_Receptacle_USB2.0_16P, J3 Conn_01x22_Pin, SW1 SW_Push, SW2 SW_Push, U1 ESP32-S3-WROOM-1, U2 LD1117S33TR_SOT223

Commit message: 製造ファイル出力3
Parts:
- R3, R4: footprint Resistor_SMD:R_0402_1005Metric -> Resistor_SMD:R_0603_1608Metric
Changed lines of the file:
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@@
 			)
 		)
-		(property "Footprint" "Resistor_SMD:R_0402_1005Metric"
+		(property "Footprint" "Resistor_SMD:R_0603_1608Metric"
 			(at 203.962 74.93 90)
 			(effects
@@
 			)
 		)
-		(property "Footprint" "Resistor_SMD:R_0402_1005Metric"
+		(property "Footprint" "Resistor_SMD:R_0603_1608Metric"
 			(at 212.852 74.93 90)
 			(effects
