File: ESP32-S3-WROOM-32E/ESP32-S3-ROS-IO-V2.0/ESP32-S3-ROS-IO-V2.0.kicad_pcb (KiCad board)
At the start: 2 copper layers, 41 parts, among them J1 Conn_01x22_Socket, J10 XT30UPB-F, J11 XT30UPB-F, J12 XT30UPB-F, J13 XT30UPB-F, J14 XT30UPB-F, J15 XT30UPB-F, J16 XT60-M, J17 XT60-M, J2 Conn_01x22_Socket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

Commit message: XT30メスのフットプリントがほしい
Parts:
- added G***6: LOGO, LOGO, F.Cu at (172.5, 116.6)
- added REF**1: MountingHole_3.2mm_M3, MountingHole:MountingHole_3.2mm_M3, F.Cu at (185.0, 103.0)
- added REF**2: MountingHole_3.2mm_M3, MountingHole:MountingHole_3.2mm_M3, F.Cu at (185.0, 158.0)
- added REF**3: MountingHole_3.2mm_M3, MountingHole:MountingHole_3.2mm_M3, F.Cu at (125.0, 158.0)
- added REF**4: MountingHole_3.2mm_M3, MountingHole:MountingHole_3.2mm_M3, F.Cu at (125.0, 113.0)
- moved R1 171.1 mm to (185.6, 150.0), turned to 180 degrees
- moved R2 167.8 mm to (185.6, 145.9), turned to 180 degrees
- moved R120 155.5 mm to (200.5, 81.2)
- moved U2 135.0 mm to (176.7, 110.6)
- moved J16 126.8 mm to (195.5, 73.3)
- moved U1 118.0 mm to (176.7, 133.5)
- moved Servo1 108.6 mm to (176.5, 69.3)
- moved Servo2 108.6 mm to (176.5, 77.1)
- moved Servo3 108.6 mm to (176.5, 84.9)
- moved Servo4 108.6 mm to (176.5, 92.7)
- moved SV4 103.6 mm to (151.9, 77.1)
- moved SV2 101.1 mm to (151.9, 69.5)
- moved SV6 100.0 mm to (151.9, 84.7)
- moved SV3 99.3 mm to (142.0, 77.1)
- moved SV5 94.9 mm to (142.0, 84.7)
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Connections:
- ENC1 pad 1: 5VD -> 5V0
- ENC2 pad 1: 5VD -> 5V0
Other:
- board outline added: 100 x 100 mm
- board text added: "+ GND"
- board text added: "120R_EN"
- board text added: "24V 24V"
- board text added: "5V0 G A B"
- board text added: "ESP32-S3-IO-Board-V2.0 2026, NHK-Project, RRST"
- board text added: "GND +"
- board text added: "H L"
- board text added: "S + GND"
- board text added: "SERVO"
- board text added: "USB"

Commit message: 配置決め
Parts:
- moved J9 213.6 mm to (200.2, 143.5), turned to 90 degrees
- moved J8 210.0 mm to (200.2, 129.5), turned to 90 degrees
- moved J12 193.4 mm to (190.0, 142.9), turned to -90 degrees
- moved J13 184.0 mm to (190.0, 128.9), turned to -90 degrees
- moved J10 141.2 mm to (109.5, 144.6), turned to -90 degrees
- moved J11 125.4 mm to (109.5, 130.6), turned to -90 degrees
- moved J15 123.0 mm to (120.1, 143.5), turned to 90 degrees
- moved J14 119.1 mm to (120.1, 129.5), turned to 90 degrees
- moved G***6 2.29 mm to (170.2, 116.6)
- moved J1 2.29 mm to (133.3, 101.6)
- moved J2 2.29 mm to (137.9, 101.6)
- moved J3 2.29 mm to (160.8, 101.6)
- moved R1 2.29 mm to (183.3, 150.0)
- moved R2 2.29 mm to (183.3, 145.9)
- moved U1 2.29 mm to (174.4, 133.5)
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
Commit message: モタドラ動確取ってから考える
Parts:
- moved REF**4 29.1 mm to (112.0, 87.0)
- moved REF**1 20.6 mm to (190.0, 83.0)
Changed lines of the file:
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@@
 	(footprint "MountingHole:MountingHole_3.2mm_M3"
 		(layer "F.Cu")
-		(at 125.042 112.99)
+		(at 112 87)
 		(descr "Mounting Hole 3.2mm, M3, no annular, generated by kicad-footprint-generator mountinghole.py")
 		(tags "mountinghole M3")
@@
 	(footprint "MountingHole:MountingHole_3.2mm_M3"
 		(layer "F.Cu")
-		(at 185.042 102.99)
+		(at 190 83)
 		(descr "Mounting Hole 3.2mm, M3, no annular, generated by kicad-footprint-generator mountinghole.py")
 		(tags "mountinghole M3")
