File: ESP32-S3-WROOM-32E/ESP32-S3-ROS-IO-V2.0/ESP32-S3-ROS-IO-V2.0.kicad_sch (KiCad schematic)
At the start: 51 parts, among them J1 Conn_01x22_Socket, J10 XT30UPB-F, J11 XT30UPB-F, J12 XT30UPB-F, J13 XT30UPB-F, J14 XT30UPB-F, J15 XT30UPB-F, J16 XT60-M, J17 XT60-M, J2 Conn_01x22_Socket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

Commit message: 新MD配置
Parts:
- removed CAN_BUS5, CAN_BUS6, CAN_BUS7, CAN_BUS8: CAN_BUS, Connector_JST:JST_XH_B2B-XH-A_1x02_P2.50mm_Vertical, symbol Connector:Conn_01x02_Pin
- removed J5: Conn_01x02_Pin, Connector_PinHeader_2.54mm:PinHeader_1x02_P2.54mm_Vertical, symbol Connector:Conn_01x02_Pin
- removed SV7: SV7, Connector_JST:JST_XH_B2B-XH-A_1x02_P2.50mm_Vertical, symbol Connector:Conn_01x02_Pin
- removed SW6: SW6, Connector_JST:JST_XH_B2B-XH-A_1x02_P2.50mm_Vertical, symbol Connector:Conn_01x02_Pin
- removed SW7: SW7, Connector_JST:JST_XH_B2B-XH-A_1x02_P2.50mm_Vertical, symbol Connector:Conn_01x02_Pin
- removed SW8: SW8, Connector_JST:JST_XH_B2B-XH-A_1x02_P2.50mm_Vertical, symbol Connector:Conn_01x02_Pin
- removed SW9: SW9, Connector_JST:JST_XH_B2B-XH-A_1x02_P2.50mm_Vertical, symbol Connector:Conn_01x02_Pin
Connections:
- net O7: no longer names the net of U2.10 (O7)
- net TR7: no longer names the net of U2.7 (I7)
- no-connect marks 1 -> 3
Other:
- note removed: "バイパス用"

Commit message: 変換基板一応できた
Connections:
- net 5VD is gone; now on net 5V0: ENC1.1 (Pin_1), ENC2.1 (Pin_1), J1.21 (Pin_21), J2.21 (Pin_21)
Changed lines of the file:
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@@
 		)
 	)
-	(global_label "5VD"
+	(global_label "5V0"
 		(shape input)
 		(at 97.79 78.74 180)
@@
 		)
 		(property "Intersheetrefs" "${INTERSHEET_REFS}"
-			(at 91.2367 78.74 0)
+			(at 91.2972 78.74 0)
 			(effects
 				(font
@@
 		)
 	)
-	(global_label "5VD"
+	(global_label "5V0"
 		(shape input)
 		(at 245.11 50.8 0)
@@
 		)
 		(property "Intersheetrefs" "${INTERSHEET_REFS}"
-			(at 251.6633 50.8 0)
+			(at 251.6028 50.8 0)
 			(effects
 				(font
@@
 		)
 	)
-	(global_label "5VD"
+	(global_label "5V0"
 		(shape input)
 		(at 38.1 78.74 180)
@@
 		)
 		(property "Intersheetrefs" "${INTERSHEET_REFS}"
-			(at 31.5467 78.74 0)
+			(at 31.6072 78.74 0)
 			(effects
 				(font
@@
 		)
 	)
-	(global_label "5VD"
+	(global_label "5V0"
 		(shape input)
 		(at 245.11 30.48 0)
@@
 		)
 		(property "Intersheetrefs" "${INTERSHEET_REFS}"
-			(at 251.6633 30.48 0)
+			(at 251.6028 30.48 0)
 			(effects
 				(font
