File: PH to XH/PH to XH.kicad_sch (KiCad schematic)
At the start: 2 parts

Commit message: 回路図ほぼ確定？
Parts:
- PH-F1: footprint (none) -> Connector_JST:JST_XH_B4B-XH-A_1x04_P2.50mm_Vertical
Other:
- note added: "ENC"
- note added: "SDM"
- moved on the sheet: PH-F1
Changed lines of the file:
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@@
 	(generator_version "9.0")
 	(paper "A4")
+	(rectangle
+		(start 49.53 15.24)
+		(end 80.01 46.99)
+		(stroke
+			(width 0)
+			(type default)
+		)
+		(fill
+			(type none)
+		)
+	)
+	(rectangle
+		(start 15.24 15.24)
+		(end 45.72 46.99)
+		(stroke
+			(width 0)
+			(type default)
+		)
+		(fill
+			(type none)
+		)
+	)
+	(text "SDM"
+		(exclude_from_sim no)
+		(at 20.066 18.288 0)
+		(effects
+			(font
+				(size 2.032 2.032)
+			)
+		)
+	)
+	(text "ENC"
+		(exclude_from_sim no)
+		(at 54.356 18.288 0)
+		(effects
+			(font
+				(size 2.032 2.032)
+			)
+		)
+	)
 	(no_connect
-		(at 60.96 39.37)
+		(at 58.42 39.37)
 	)
 	(wire
@@
 	(wire
 		(pts
-			(xy 60.96 36.83) (xy 78.74 36.83)
+			(xy 58.42 36.83) (xy 76.2 36.83)
 		)
 		(stroke
@@
 	(global_label "TX"
 		(shape input)
-		(at 60.96 31.75 0)
-		(fields_autoplaced yes)
-		(effects
-			(font
-				(size 1.27 1.27)
-			)
-			(justify left)
-		)
-		(property "Intersheetrefs" "${INTERSHEET_REFS}"
-			(at 66.1223 31.75 0)
+		(at 58.42 31.75 0)
+		(fields_autoplaced yes)
+		(effects
+			(font
+				(size 1.27 1.27)
+			)
+			(justify left)
+		)
+		(property "Intersheetrefs" "${INTERSHEET_REFS}"
+			(at 63.5823 31.75 0)
 			(effects
 				(font
@@
 	(global_label "5V0"
 		(shape input)
-		(at 60.96 29.21 0)
-		(fields_autoplaced yes)
-		(effects
-			(font
-				(size 1.27 1.27)
-			)
-			(justify left)
-		)
-		(property "Intersheetrefs" "${INTERSHEET_REFS}"
-			(at 67.4528 29.21 0)
+		(at 58.42 29.21 0)
+		(fields_autoplaced yes)
+		(effects
+			(font
+				(size 1.27 1.27)
+			)
+			(justify left)
+		)
+		(property "Intersheetrefs" "${INTERSHEET_REFS}"
+			(at 64.9128 29.21 0)
 			(effects
 				(font
@@
 	(global_label "RX"
 		(shape input)
-		(at 60.96 34.29 0)
-		(fields_autoplaced yes)
-		(effects
-			(font
-				(size 1.27 1.27)
-			)
-			(justify left)
-		)
-		(property "Intersheetrefs" "${INTERSHEET_REFS}"
-			(at 66.4247 34.29 0)
+		(at 58.42 34.29 0)
+		(fields_autoplaced yes)
+		(effects
+			(font
+				(size 1.27 1.27)
+			)
+			(justify left)
+		)
+		(property "Intersheetrefs" "${INTERSHEET_REFS}"
+			(at 63.8847 34.29 0)
 			(effects
 				(font
@@
 	(symbol
 		(lib_id "Connector:Conn_01x05_Pin")
-		(at 55.88 34.29 0)
+		(at 53.34 34.29 0)
 		(unit 1)
 		(exclude_from_sim no)
@@
 		(fields_autoplaced yes)
 		(property "Reference" "PH-F1"
-			(at 56.515 24.13 0)
+			(at 53.975 24.13 0)
 			(effects
 				(font
@@
 		)
 		(property "Value" "PH-F1"
-			(at 56.515 26.67 0)
-			(effects
-				(font
-					(size 1.27 1.27)
-				)
-			)
-		)
-		(property "Footprint" ""
-			(at 55.88 34.29 0)
+			(at 53.975 26.67 0)
+			(effects
+				(font
+					(size 1.27 1.27)
+				)
+			)
+		)
+		(property "Footprint" "Connector_JST:JST_XH_B4B-XH-A_1x04_P2.50mm_Vertical"
+			(at 53.34 34.29 0)
 			(effects
 				(font
@@
 		)
 		(property "Datasheet" "~"
-			(at 55.88 34.29 0)
+			(at 53.34 34.29 0)
 			(effects
 				(font
@@
 		)
 		(property "Description" "Generic connector, single row, 01x05, script generated"
-			(at 55.88 34.29 0)
+			(at 53.34 34.29 0)
 			(effects
 				(font
@@
 	(symbol
 		(lib_id "power:GND")
-		(at 78.74 36.83 0)
+		(at 76.2 36.83 0)
 		(unit 1)
 		(exclude_from_sim no)
@@
 		(fields_autoplaced yes)
 		(property "Reference" "#PWR01"
-			(at 78.74 43.18 0)
+			(at 76.2 43.18 0)
 			(effects
 				(font
@@
 		)
 		(property "Value" "GND"
-			(at 78.74 41.91 0)
+			(at 76.2 41.91 0)
 			(effects
 				(font
@@
 		)
 		(property "Footprint" ""
-			(at 78.74 36.83 0)
+			(at 76.2 36.83 0)
 			(effects
 				(font
@@
 		)
 		(property "Datasheet" ""
-			(at 78.74 36.83 0)
+			(at 76.2 36.83 0)
 			(effects
 				(font
@@
 		)
 		(property "Description" "Power symbol creates a global label with name \"GND\" , ground"
-			(at 78.74 36.83 0)
-			(effects
-				(font
+			(at 76.2 36.83 0)
+			(effects
+				(font

Commit message: 変換基板一応できた
Parts:
- PH-F1: footprint Connector_JST:JST_XH_B4B-XH-A_1x04_P2.50mm_Vertical -> Connector_JST:JST_PH_B5B-PH-K_1x05_P2.00mm_Vertical
Connections:
- net 5V0: now also XH-F1.4 (Pin_4); no longer XH-F1.1 (Pin_1)
- net GND: now also XH-F1.3 (Pin_3); no longer XH-F1.2 (Pin_2)
- net RX: now also XH-F1.1 (Pin_1); no longer XH-F1.4 (Pin_4)
- net TX: now also XH-F1.2 (Pin_2); no longer XH-F1.3 (Pin_3)
Changed lines of the file:
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@@
+		)
+	)
+	(text "ENC"
+		(exclude_from_sim no)
+		(at 20.066 18.288 0)
+		(effects
+			(font
+				(size 2.032 2.032)
+			)
 		)
 	)
 	(text "SDM"
-		(exclude_from_sim no)
-		(at 20.066 18.288 0)
-		(effects
-			(font
-				(size 2.032 2.032)
-			)
-		)
-	)
-	(text "ENC"
 		(exclude_from_sim no)
 		(at 54.356 18.288 0)
@@
 	(wire
 		(pts
-			(xy 24.13 31.75) (xy 41.91 31.75)
+			(xy 24.13 34.29) (xy 41.91 34.29)
 		)
 		(stroke
@@
 		)
 	)
+	(global_label "5V0"
+		(shape input)
+		(at 24.13 36.83 0)
+		(fields_autoplaced yes)
+		(effects
+			(font
+				(size 1.27 1.27)
+			)
+			(justify left)
+		)
+		(property "Intersheetrefs" "${INTERSHEET_REFS}"
+			(at 30.6228 36.83 0)
+			(effects
+				(font
+					(size 1.27 1.27)
+				)
+				(justify left)
+				(hide yes)
+			)
+		)
+	)
+	(global_label "5V0"
+		(shape input)
+		(at 58.42 29.21 0)
+		(fields_autoplaced yes)
+		(effects
+			(font
+				(size 1.27 1.27)
+			)
+			(justify left)
+		)
+		(property "Intersheetrefs" "${INTERSHEET_REFS}"
+			(at 64.9128 29.21 0)
+			(effects
+				(font
+					(size 1.27 1.27)
+				)
+				(justify left)
+				(hide yes)
+			)
+		)
+	)
+	(global_label "RX"
+		(shape input)
+		(at 58.42 34.29 0)
+		(fields_autoplaced yes)
+		(effects
+			(font
+				(size 1.27 1.27)
+			)
+			(justify left)
+		)
+		(property "Intersheetrefs" "${INTERSHEET_REFS}"
+			(at 63.8847 34.29 0)
+			(effects
+				(font
+					(size 1.27 1.27)
+				)
+				(justify left)
+				(hide yes)
+			)
+		)
+	)
+	(global_label "RX"
+		(shape input)
+		(at 24.13 29.21 0)
+		(fields_autoplaced yes)
+		(effects
+			(font
+				(size 1.27 1.27)
+			)
+			(justify left)
+		)
+		(property "Intersheetrefs" "${INTERSHEET_REFS}"
+			(at 29.5947 29.21 0)
+			(effects
+				(font
+					(size 1.27 1.27)
+				)
+				(justify left)
+				(hide yes)
+			)
+		)
+	)
 	(global_label "TX"
 		(shape input)
-		(at 24.13 34.29 0)
-		(fields_autoplaced yes)
-		(effects
-			(font
-				(size 1.27 1.27)
-			)
-			(justify left)
-		)
-		(property "Intersheetrefs" "${INTERSHEET_REFS}"
-			(at 29.2923 34.29 0)
-			(effects
-				(font
-					(size 1.27 1.27)
-				)
-				(justify left)
-				(hide yes)
-			)
-		)
-	)
-	(global_label "5V0"
-		(shape input)
-		(at 24.13 29.21 0)
-		(fields_autoplaced yes)
-		(effects
-			(font
-				(size 1.27 1.27)
-			)
-			(justify left)
-		)
-		(property "Intersheetrefs" "${INTERSHEET_REFS}"
-			(at 30.6228 29.21 0)
-			(effects
-				(font
-					(size 1.27 1.27)
-				)
-				(justify left)
-				(hide yes)
-			)
-		)
-	)
-	(global_label "5V0"
-		(shape input)
-		(at 58.42 29.21 0)
-		(fields_autoplaced yes)
-		(effects
-			(font
-				(size 1.27 1.27)
-			)
-			(justify left)
-		)
-		(property "Intersheetrefs" "${INTERSHEET_REFS}"
-			(at 64.9128 29.21 0)
-			(effects
-				(font
-					(size 1.27 1.27)
-				)
-				(justify left)
-				(hide yes)
-			)
-		)
-	)
-	(global_label "RX"
-		(shape input)
-		(at 58.42 34.29 0)
-		(fields_autoplaced yes)
-		(effects
-			(font
-				(size 1.27 1.27)
-			)
-			(justify left)
-		)
-		(property "Intersheetrefs" "${INTERSHEET_REFS}"
-			(at 63.8847 34.29 0)
-			(effects
-				(font
-					(size 1.27 1.27)
-				)
-				(justify left)
-				(hide yes)
-			)
-		)
-	)
-	(global_label "RX"
-		(shape input)
-		(at 24.13 36.83 0)
-		(fields_autoplaced yes)
-		(effects
-			(font
-				(size 1.27 1.27)
-			)
-			(justify left)
-		)
-		(property "Intersheetrefs" "${INTERSHEET_REFS}"
-			(at 29.5947 36.83 0)
+		(at 24.13 31.75 0)
+		(fields_autoplaced yes)
+		(effects
+			(font
+				(size 1.27 1.27)
+			)
+			(justify left)
+		)
+		(property "Intersheetrefs" "${INTERSHEET_REFS}"
+			(at 29.2923 31.75 0)
 			(effects
 				(font
@@
 			)
 		)
-		(property "Footprint" "Connector_JST:JST_XH_B4B-XH-A_1x04_P2.50mm_Vertical"
+		(property "Footprint" "Connector_JST:JST_PH_B5B-PH-K_1x05_P2.00mm_Vertical"
 			(at 53.34 34.29 0)
 			(effects
@@
 	(symbol
 		(lib_id "power:GND")
-		(at 41.91 31.75 0)
+		(at 41.91 34.29 0)
 		(unit 1)
 		(exclude_from_sim no)
@@
 		(dnp no)
 		(fields_autoplaced yes)
-		(property "Reference" "#PWR023"
-			(at 41.91 38.1 0)
+		(property "Reference" "#PWR02"
+			(at 41.91 40.64 0)
 			(effects
 				(font
@@
 		)
 		(property "Value" "GND"
-			(at 41.91 36.83 0)
+			(at 41.91 39.37 0)
 			(effects
 				(font
@@
 		)
 		(property "Footprint" ""
-			(at 41.91 31.75 0)
+			(at 41.91 34.29 0)
 			(effects
 				(font
@@
 		)
 		(property "Datasheet" ""
-			(at 41.91 31.75 0)
+			(at 41.91 34.29 0)
 			(effects
 				(font
@@
 		)
 		(property "Description" "Power symbol creates a global label with name \"GND\" , ground"
-			(at 41.91 31.75 0)
+			(at 41.91 34.29 0)
 			(effects
 				(font
@@
 			(project "PH to XH"
 				(path "/82bfc97a-c2ee-48b2-bb37-dd46fdea9ad1"
-					(reference "#PWR023")
+					(reference "#PWR02")
 					(unit 1)
 				)

Commit message: 変換基板ほぼかんせ
Parts:
- PH-F1: footprint Connector_JST:JST_PH_B5B-PH-K_1x05_P2.00mm_Vertical -> Connector_JST:JST_PH_S5B-PH-K_1x05_P2.00mm_Horizontal
- XH-F1: footprint Connector_JST:JST_XH_B4B-XH-A_1x04_P2.50mm_Vertical -> Connector_JST:JST_XH_S4B-XH-A-1_1x04_P2.50mm_Horizontal
Changed lines of the file:
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@@
 			)
 		)
-		(property "Footprint" "Connector_JST:JST_PH_B5B-PH-K_1x05_P2.00mm_Vertical"
+		(property "Footprint" "Connector_JST:JST_PH_S5B-PH-K_1x05_P2.00mm_Horizontal"
 			(at 53.34 34.29 0)
 			(effects
@@
 			)
 		)
-		(property "Footprint" "Connector_JST:JST_XH_B4B-XH-A_1x04_P2.50mm_Vertical"
+		(property "Footprint" "Connector_JST:JST_XH_S4B-XH-A-1_1x04_P2.50mm_Horizontal"
 			(at 19.05 31.75 0)
 			(effects
