File: PH to XH/PH to XH.kicad_pcb (KiCad board)
At the start: 2 copper layers, 16 x 14 mm, 2 parts

Commit message: 変換基板ほぼかんせ
Parts:
- added REF**: MountingHole_3.2mm_M3, MountingHole:MountingHole_3.2mm_M3, F.Cu at (59.0, 54.0)
- added REF**: MountingHole_3.2mm_M3, MountingHole:MountingHole_3.2mm_M3, F.Cu at (81.0, 54.0)
- PH-F1: footprint Connector_JST:JST_PH_B5B-PH-K_1x05_P2.00mm_Vertical -> Connector_JST:JST_PH_S5B-PH-K_1x05_P2.00mm_Horizontal
- XH-F1: footprint Connector_JST:JST_XH_B4B-XH-A_1x04_P2.50mm_Vertical -> Connector_JST:JST_XH_S4B-XH-A-1_1x04_P2.50mm_Horizontal; moved to F.Cu
- moved PH-F1 57.9 mm to (66.0, 58.7)
- moved XH-F1 51.0 mm to (73.8, 50.7)
Routing:
- net 5V0: track 4.10 -> 8.12 mm
- net TX: track 5.35 -> 9.37 mm
- net RX: track 5.55 -> 9.57 mm
- net GND: track 5.35 -> 9.33 mm
Other:
- board size 16 x 14 mm -> 32 x 28 mm

Commit message: とりあえず基板二つ完成しましたよ、あとメイン基板届いた
Routing:
- added copper zone on F.Cu, net GND
Changed lines of the file:
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@@
 		(net 5)
+	)
+	(zone
+		(net 5)
+		(net_name "GND")
+		(layer "F.Cu")
+		(hatch edge 0.5)
+		(connect_pads
+			(clearance 0.5)
+		)
+		(min_thickness 0.25)
+		(filled_areas_thickness no)
+		(fill yes
+			(thermal_gap 0.5)
+			(thermal_bridge_width 0.5)
+		)
+		(polygon
+			(pts
+				(xy 56 41) (xy 84 41) (xy 85 42) (xy 85 66) (xy 84 67) (xy 56 67) (xy 55 66) (xy 55 42)
+			)
+		)
 	)
 	(embedded_fonts no)

Commit message: ビア忘れてた
Routing:
- net GND: vias 0 -> 6
- added copper zone on B.Cu, net GND
Changed lines of the file:
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@@
 		(net 4)
+	)
+	(via
+		(at 59 46)
+		(size 0.6)
+		(drill 0.3)
+		(layers "F.Cu" "B.Cu")
+		(free yes)
+		(net 5)
+	)
+	(via
+		(at 81 62)
+		(size 0.6)
+		(drill 0.3)
+		(layers "F.Cu" "B.Cu")
+		(free yes)
+		(net 5)
+	)
+	(via
+		(at 68 53)
+		(size 0.6)
+		(drill 0.3)
+		(layers "F.Cu" "B.Cu")
+		(free yes)
+		(net 5)
+	)
+	(via
+		(at 59 62)
+		(size 0.6)
+		(drill 0.3)
+		(layers "F.Cu" "B.Cu")
+		(free yes)
+		(net 5)
+	)
+	(via
+		(at 74 56)
+		(size 0.6)
+		(drill 0.3)
+		(layers "F.Cu" "B.Cu")
+		(free yes)
+		(net 5)
+	)
+	(via
+		(at 81 46)
+		(size 0.6)
+		(drill 0.3)
+		(layers "F.Cu" "B.Cu")
+		(free yes)
+		(net 5)
 	)
 	(segment
@@
 		(net 5)
 		(net_name "GND")
-		(layer "F.Cu")
+		(layers "F.Cu" "B.Cu")
 		(hatch edge 0.5)
 		(connect_pads
