File: XIAO ESP32-S3/XIAO ESP32-S3.kicad_pcb (KiCad board)
At the start: 2 copper layers, 8 parts, among them J1 Conn_01x07_Socket, J2 Conn_01x07_Socket, J3 Conn_01x07_Socket, J4 Conn_01x07_Socket

Commit message: 基板ほぼ完成
Parts:
- moved J1 59.5 mm to (77.2, 56.7), turned to 180 degrees
- moved SMD1 53.9 mm to (71.5, 22.5)
- moved SMD2 53.8 mm to (71.5, 31.0)
- moved J3 50.1 mm to (73.0, 56.7), turned to 180 degrees
- moved J2 45.8 mm to (61.0, 56.7), turned to 180 degrees
- moved J4 40.5 mm to (57.0, 56.7), turned to 180 degrees
- moved ENC2 36.9 mm to (55.5, 31.0)
- moved ENC1 36.8 mm to (55.5, 22.8)
Connections:
- net GPIO9 renamed NC2
- J1 pad 7: unconnected-(J1-Pin_7-Pad7) -> NC1
- J2 pad 7: unconnected-(J2-Pin_7-Pad7) -> NC3
- J3 pad 7: unconnected-(J3-Pin_7-Pad7) -> NC1
- J4 pad 7: unconnected-(J4-Pin_7-Pad7) -> NC3

Commit message: 基板ほぼかんせ　ねむい
Parts:
- removed SMD2: SMD2, Connector_JST:JST_XH_B4B-XH-A_1x04_P2.50mm_Vertical
- added REF1**: MountingHole_3.2mm_M3, MountingHole:MountingHole_3.2mm_M3, F.Cu at (84.0, 44.0)
- added REF2**: MountingHole_3.2mm_M3, MountingHole:MountingHole_3.2mm_M3, F.Cu at (84.0, 74.0)
- added REF3**: MountingHole_3.2mm_M3, MountingHole:MountingHole_3.2mm_M3, F.Cu at (45.0, 74.0)
- added REF4**: MountingHole_3.2mm_M3, MountingHole:MountingHole_3.2mm_M3, F.Cu at (45.0, 44.0)
- moved SMD1 26.8 mm to (68.4, 49.1)
- moved ENC1 21.1 mm to (53.3, 43.8)
- moved ENC2 21.1 mm to (53.3, 52.0)
- moved J2 21.0 mm to (53.4, 76.3)
- moved J1 19.6 mm to (76.2, 76.2)
- moved J3 19.5 mm to (72.4, 76.2)
- moved J4 19.5 mm to (57.1, 76.2)
Routing:
- net 5V: track 0.00 -> 53.7 mm
- net GND: track 0.00 -> 51.3 mm
- net ENC1_A: track 0.00 -> 43.9 mm
- net ENC1_B: track 0.00 -> 41.2 mm
- net ENC2_A: track 0.00 -> 28.8 mm
- net ENC2_B: track 0.00 -> 25.2 mm
- net GPIO5: track 0.00 -> 21.4 mm
- net GPIO6: track 0.00 -> 20.0 mm
- net 3V3: track 0.00 -> 3.81 mm
- net NC3: track 0.00 -> 3.81 mm
- net GPIO7: track 0.00 -> 3.81 mm
- net NC2: track 0.00 -> 3.81 mm
- net GPIO8: track 0.00 -> 3.81 mm
- net NC1: track 0.00 -> 3.80 mm
Other:
- board outline added: 49 x 40 mm

Commit message: とりあえず基板二つ完成しましたよ、あとメイン基板届いた
Parts:
- renumbered SMD1 to SMD
Routing:
- added copper zone on B.Cu, net GND
- added copper zone on F.Cu, net GND
Changed lines of the file:
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@@
 		(descr "JST XH series connector, B4B-XH-A (http://www.jst-mfg.com/product/pdf/eng/eXH.pdf), generated with kicad-footprint-generator")
 		(tags "connector JST XH vertical")
-		(property "Reference" "SMD1"
+		(property "Reference" "SMD"
 			(at 3.75 -3.55 0)
 			(layer "F.SilkS")
@@
 		(net 14)
 	)
+	(zone
+		(net 3)
+		(net_name "GND")
+		(layers "F.Cu" "B.Cu")
+		(hatch edge 0.5)
+		(connect_pads
+			(clearance 0.5)
+		)
+		(min_thickness 0.25)
+		(filled_areas_thickness no)
+		(fill yes
+			(thermal_gap 0.5)
+			(thermal_bridge_width 0.5)
+		)
+		(polygon
+			(pts
+				(xy 42 40) (xy 87 40) (xy 88 41) (xy 88 77) (xy 87 78) (xy 42 78) (xy 41 77) (xy 41 41)
+			)
+		)
+	)
 	(embedded_fonts no)

Commit message: ビア忘れてた
Routing:
- net GND: vias 0 -> 14
Changed lines of the file:
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@@
+		(net 3)
+	)
+	(via
+		(at 62 74.5)
+		(size 0.6)
+		(drill 0.3)
+		(layers "F.Cu" "B.Cu")
+		(free yes)
+		(net 3)
+	)
+	(via
+		(at 46.5 58.5)
+		(size 0.6)
+		(drill 0.3)
+		(layers "F.Cu" "B.Cu")
+		(free yes)
+		(net 3)
+	)
+	(via
+		(at 68 56)
+		(size 0.6)
+		(drill 0.3)
+		(layers "F.Cu" "B.Cu")
+		(free yes)
+		(net 3)
+	)
+	(via
+		(at 54.5 48.5)
+		(size 0.6)
+		(drill 0.3)
+		(layers "F.Cu" "B.Cu")
+		(free yes)
+		(net 3)
+	)
+	(via
+		(at 83.5 66)
+		(size 0.6)
+		(drill 0.3)
+		(layers "F.Cu" "B.Cu")
+		(free yes)
+		(net 3)
+	)
+	(via
+		(at 54.5 57)
+		(size 0.6)
+		(drill 0.3)
+		(layers "F.Cu" "B.Cu")
+		(free yes)
+		(net 3)
+	)
+	(via
+		(at 83.5 52)
+		(size 0.6)
+		(drill 0.3)
+		(layers "F.Cu" "B.Cu")
+		(free yes)
+		(net 3)
+	)
+	(via
+		(at 83.5 59)
+		(size 0.6)
+		(drill 0.3)
+		(layers "F.Cu" "B.Cu")
+		(free yes)
+		(net 3)
+	)
+	(via
+		(at 75 43.5)
+		(size 0.6)
+		(drill 0.3)
+		(layers "F.Cu" "B.Cu")
+		(free yes)
+		(net 3)
+	)
+	(via
+		(at 66.5 74.5)
+		(size 0.6)
+		(drill 0.3)
+		(layers "F.Cu" "B.Cu")
+		(free yes)
+		(net 3)
+	)
+	(via
+		(at 46.5 51)
+		(size 0.6)
+		(drill 0.3)
+		(layers "F.Cu" "B.Cu")
+		(free yes)
+		(net 3)
+	)
+	(via
+		(at 68.5 43.5)
+		(size 0.6)
+		(drill 0.3)
+		(layers "F.Cu" "B.Cu")
+		(free yes)
+		(net 3)
+	)
+	(via
+		(at 46.5 65)
+		(size 0.6)
+		(drill 0.3)
+		(layers "F.Cu" "B.Cu")
+		(free yes)
+		(net 3)
+	)
+	(via
+		(at 62 69)
+		(size 0.6)
+		(drill 0.3)
+		(layers "F.Cu" "B.Cu")
+		(free yes)
 		(net 3)
 	)

Commit message: ええんちゃうの
Parts:
- removed ENC2: ENC2, Connector_JST:JST_XH_B4B-XH-A_1x04_P2.50mm_Vertical
- removed SMD: SMD1, Connector_JST:JST_XH_B4B-XH-A_1x04_P2.50mm_Vertical
- added G***6: LOGO, LOGO, B.Cu at (63.0, 49.0)
- added Serial1: Serial1, Connector_JST:JST_PH_S5B-PH-K_1x05_P2.00mm_Horizontal, F.Cu at (73.5, 54.6)
- ENC1: footprint Connector_JST:JST_XH_B4B-XH-A_1x04_P2.50mm_Vertical -> Connector_JST:JST_XH_S4B-XH-A_1x04_P2.50mm_Horizontal
- moved ENC1 12.9 mm to (59.6, 55.0), turned to 180 degrees
- moved REF1** 5.66 mm to (80.0, 48.0)
- moved REF2** 4.00 mm to (80.0, 74.0)
- moved REF4** 4.00 mm to (45.0, 48.0)
- moved J2 2.19 mm to (51.2, 76.3)
- moved J1 2.19 mm to (74.0, 76.2)
- moved J3 2.19 mm to (70.2, 76.2)
- moved J4 2.19 mm to (55.0, 76.2)
Connections:
- net ENC2_A renamed GPIO3
- net ENC2_B renamed GPIO4
- J1 pad 5: GPIO5 -> NC1
- J1 pad 6: GPIO6 -> NC2
- J1 pad 7: NC1 -> NC3
- J2 pad 4: NC2 -> NC4
- J2 pad 7: NC3 -> NC5
- J3 pad 5: GPIO5 -> NC1
- J3 pad 6: GPIO6 -> NC2
- J3 pad 7: NC1 -> NC3
- J4 pad 4: NC2 -> NC4
- J4 pad 7: NC3 -> NC5
Routing:
- net GND: track 51.3 -> 0.00 mm, vias 14 -> 0
- net 5V: track 53.7 -> 27.1 mm
- net GPIO5: track 21.4 -> 0.00 mm
- net GPIO6: track 20.0 -> 0.00 mm
- net GPIO3: track 28.8 -> 21.4 mm
- net ENC1_A: track 43.9 -> 37.1 mm
- net GPIO4: track 25.2 -> 18.5 mm
- net NC5: track 0.00 -> 3.81 mm
- net NC4: track 0.00 -> 3.81 mm
- net ENC1_B: track 41.2 -> 40.1 mm, vias 0 -> 1
Other:
- board size 49 x 40 mm -> 45 x 36 mm
- board text added: "B A G 5V"
- board text added: "G RX TX 5V"
- board text added: "USB"
