File: ESP32-WROOM-32E/ESP32-ROS-O/ESP32-ROS-O.kicad_pcb (KiCad board)
At the start: 2 copper layers, 80 x 79 mm, 21 parts, among them J1 Conn_01x19_Socket, J16 XT60-M, J17 XT60-M, J2 Conn_01x19_Socket, J3 Conn_01x19_Socket, J4 Conn_01x19_Socket

Commit message: 専用基板作るんやから良い設計が上がることを期待しています
Parts:
- moved Servo3 15.1 mm to (119.3, 93.8)
- moved Servo2 15.0 mm to (132.4, 85.7)
- moved SV2 0.51 mm to (108.5, 85.6)
- moved SV4 0.51 mm to (108.5, 94.0)
- moved Servo1 0.44 mm to (119.4, 85.7)
- moved D1 0.38 mm to (135.6, 102.7)
- moved Servo4 0.13 mm to (132.4, 93.9)
Other:
- board text added: "GND +"
- board text added: "S + GND"
