File: ESP32-WROOM-32E/ESP32-ROS-I/ESP32-ROS-I.kicad_sch (KiCad schematic)
At the start: 0 parts

Commit message: 足回り専用基板
Parts:
- added CAN_BUS1, CAN_BUS2, CAN_BUS3, CAN_BUS4: CAN_BUS, Connector_JST:JST_XH_B2B-XH-A_1x02_P2.50mm_Vertical, symbol Connector:Conn_01x02_Pin
- added D1: LED, LED_THT:LED_D5.0mm, symbol Device:LED
- added ENC1: ENC1, Connector_JST:JST_XH_B4B-XH-A_1x04_P2.50mm_Vertical, symbol Connector:Conn_01x04_Pin
- added ENC2: ENC2, Connector_JST:JST_XH_B4B-XH-A_1x04_P2.50mm_Vertical, symbol Connector:Conn_01x04_Pin
- added ENC3: ENC3, Connector_JST:JST_XH_B4B-XH-A_1x04_P2.50mm_Vertical, symbol Connector:Conn_01x04_Pin
- added ENC4: ENC4, Connector_JST:JST_XH_B4B-XH-A_1x04_P2.50mm_Vertical, symbol Connector:Conn_01x04_Pin
- added J1, J2, J3, J4: Conn_01x19_Socket, Connector_PinSocket_2.54mm:PinSocket_1x19_P2.54mm_Vertical, symbol Connector:Conn_01x19_Socket
- added R1: 120, Resistor_THT:R_Axial_DIN0207_L6.3mm_D2.5mm_P10.16mm_Horizontal, symbol Device:R
- added R120: R120, Connector_PinHeader_2.54mm:PinHeader_1x02_P2.54mm_Vertical, symbol Connector:Conn_01x02_Pin
- added R2: 330, Resistor_THT:R_Axial_DIN0207_L6.3mm_D2.5mm_P10.16mm_Horizontal, symbol Device:R
- added U1: ~, Package_DIP:DIP-8_W7.62mm, symbol New_Library:MCP2561
- added VMD1/VMD2: VMD1/VMD2, Connector_PinHeader_2.54mm:PinHeader_1x11_P2.54mm_Vertical, symbol Connector:Conn_01x11_Pin
- added VMD3/VMD4: VMD3/VMD4, Connector_PinHeader_2.54mm:PinHeader_1x11_P2.54mm_Vertical, symbol Connector:Conn_01x11_Pin
Connections:
- new net: D1.1 (K), R2.1
- new net 3V3: D1.2 (A), J1.1 (Pin_1), J2.1 (Pin_1)
- new net 5V0: J1.19 (Pin_19), J2.19 (Pin_19), U1.3 (Vdd)
- new net CANH: CAN_BUS1.1 (Pin_1), CAN_BUS2.1 (Pin_1), CAN_BUS3.1 (Pin_1), CAN_BUS4.1 (Pin_1), R1.1, R120.1 (Pin_1), U1.7 (CANH)
- new net CANL: CAN_BUS1.2 (Pin_2), CAN_BUS2.2 (Pin_2), CAN_BUS3.2 (Pin_2), CAN_BUS4.2 (Pin_2), R1.2, R120.2 (Pin_2), U1.6 (CANL)
- new net CAN_RX: J3.15 (Pin_15), J4.15 (Pin_15), U1.4 (Rxd)
- new net CAN_TX: J3.13 (Pin_13), J4.13 (Pin_13), U1.1 (Txd)
- new net ENC1_A: ENC1.3 (Pin_3), J3.8 (Pin_8), J4.8 (Pin_8)
- new net ENC1_B: ENC1.4 (Pin_4), J3.6 (Pin_6), J4.6 (Pin_6)
- new net ENC2_A: ENC2.3 (Pin_3), J3.3 (Pin_3), J4.3 (Pin_3)
- new net ENC2_B: ENC2.4 (Pin_4), J3.2 (Pin_2), J4.2 (Pin_2)
- new net ENC3_A: ENC3.3 (Pin_3), J1.9 (Pin_9), J2.9 (Pin_9)
- new net ENC3_B: ENC3.4 (Pin_4), J1.10 (Pin_10), J2.10 (Pin_10)
- new net ENC4_A: ENC4.3 (Pin_3), J1.11 (Pin_11), J2.11 (Pin_11)
- new net ENC4_B: ENC4.4 (Pin_4), J1.7 (Pin_7), J2.7 (Pin_7)
- new net GND: ENC1.2 (Pin_2), ENC2.2 (Pin_2), ENC3.2 (Pin_2), ENC4.2 (Pin_2), J1.14 (Pin_14), J2.14 (Pin_14), J3.1 (Pin_1), J3.7 (Pin_7), J4.1 (Pin_1), J4.7 (Pin_7), U1.2 (Vss), U1.8 (STBY), VMD1/VMD2.1 (Pin_1), VMD1/VMD2.3 (Pin_3), VMD3/VMD4.1 (Pin_1), VMD3/VMD4.3 (Pin_3)
- new net GPIO0: J3.14 (Pin_14), J4.14 (Pin_14), R2.2
- new net GPIO12: J1.13 (Pin_13), J2.13 (Pin_13), VMD1/VMD2.5 (Pin_5)
- new net GPIO13: J1.15 (Pin_15), J2.15 (Pin_15), VMD3/VMD4.9 (Pin_9)
- new net GPIO14: J1.12 (Pin_12), J2.12 (Pin_12), VMD3/VMD4.5 (Pin_5)
- new net GPIO15: J3.16 (Pin_16), J4.16 (Pin_16), VMD1/VMD2.11 (Pin_11)
- new net GPIO16: J3.12 (Pin_12), J4.12 (Pin_12), VMD1/VMD2.7 (Pin_7)
- new net GPIO17: J3.11 (Pin_11), J4.11 (Pin_11), VMD3/VMD4.11 (Pin_11)
- new net GPIO18: J3.9 (Pin_9), J4.9 (Pin_9), VMD3/VMD4.7 (Pin_7)
- new net GPIO5: J3.10 (Pin_10), J4.10 (Pin_10), VMD1/VMD2.9 (Pin_9)
- new net NC1: J1.2 (Pin_2), J2.2 (Pin_2)
- new net NC10: J3.4 (Pin_4), J4.4 (Pin_4)
- new net NC11: J3.5 (Pin_5), J4.5 (Pin_5)
- new net NC12: J3.17 (Pin_17), J4.17 (Pin_17)
- new net NC13: J3.18 (Pin_18), J4.18 (Pin_18)
- new net NC14: J3.19 (Pin_19), J4.19 (Pin_19)
- new net NC2: J1.3 (Pin_3), J2.3 (Pin_3)
- new net NC3: J1.4 (Pin_4), J2.4 (Pin_4)
- new net NC4: J1.5 (Pin_5), J2.5 (Pin_5)
- new net NC5: J1.6 (Pin_6), J2.6 (Pin_6)
- new net NC6: J1.8 (Pin_8), J2.8 (Pin_8)
- new net NC7: J1.16 (Pin_16), J2.16 (Pin_16)
- new net NC8: J1.17 (Pin_17), J2.17 (Pin_17)
- new net NC9: J1.18 (Pin_18), J2.18 (Pin_18)
- new net VDD33: ENC1.1 (Pin_1), ENC2.1 (Pin_1), ENC3.1 (Pin_1), ENC4.1 (Pin_1)
- no-connect marks 0 -> 1
Other:
- note added: "CAN"
- note added: "ESP32-DevKitC用ソケット"
- note added: "ESP32-DevKitC用ソケット(デバッグ用)"
- note added: "VMD/MD"
- note added: "エンコーダ-"
- note added: "ピン割り当て"
- note added: "状態表示"
