File: RRST-ESP32-S3-Rev.2/RRST-ESP32-S3-Rev.2.kicad_pcb (KiCad board)
At the start: 2 copper layers, 25.4 x 62.7 mm, 33 parts, among them J1 Conn_01x22_Pin, J2 USB_C_Receptacle_USB2.0_16P, J3 Conn_01x22_Pin, SW1 SW_Push, SW2 SW_Push, U1 ESP32-S3-WROOM-1, U2 LD1117S33TR_SOT223

Commit message: 自動配線&未配線の手直し完了
Other:
- copper layers 2 -> 4
