File: RRST-ESP32-S3-Rev.2-Sense-EXB/RRST-ESP32-S3-Rev.2-Sense-EXB.kicad_pcb (KiCad board)
At the start: 2 copper layers, 26 x 56.9 mm, 2 parts, among them J1 Conn_01x22_Pin, J3 Conn_01x22_Pin

Commit message: 拡張基盤迷走中
Parts:
- added CAN1: CAN, Connector_PinSocket_2.54mm:PinSocket_1x04_P2.54mm_Vertical, B.Cu at (88.9, 92.2)
- added D1: LED, LED_THT:LED_D3.0mm, F.Cu at (59.4, 107.7)
- added ENC1: ENC1, Connector_JST:JST_XH_B4B-XH-A_1x04_P2.50mm_Vertical, F.Cu at (42.3, 51.1)
- added ENC2: ENC2, Connector_JST:JST_XH_B4B-XH-A_1x04_P2.50mm_Vertical, F.Cu at (42.3, 57.9)
- added J16: XT60-M, Connector_AMASS:AMASS_XT30U-M_1x02_P5.0mm_Vertical, F.Cu at (152.4, 66.8)
- added J17: XT60-M, Connector_AMASS:AMASS_XT30U-F_1x02_P5.0mm_Vertical, F.Cu at (145.2, 66.8)
- added R2: 330, Resistor_THT:R_Axial_DIN0207_L6.3mm_D2.5mm_P10.16mm_Horizontal, F.Cu at (56.5, 112.8)
- added SV1: SV1, Connector_JST:JST_XH_B2B-XH-A_1x02_P2.50mm_Vertical, F.Cu at (141.0, 58.0)
- added SV2: SV2, Connector_JST:JST_XH_B2B-XH-A_1x02_P2.50mm_Vertical, F.Cu at (141.0, 49.4)
- added SV3: SV3, Connector_JST:JST_XH_B2B-XH-A_1x02_P2.50mm_Vertical, F.Cu at (141.0, 40.7)
- added SV4: SV4, Connector_JST:JST_XH_B2B-XH-A_1x02_P2.50mm_Vertical, F.Cu at (141.0, 32.1)
- added SV5: SV5, Connector_JST:JST_XH_B2B-XH-A_1x02_P2.50mm_Vertical, F.Cu at (38.0, 101.4)
- added SV6: SV6, Connector_JST:JST_XH_B2B-XH-A_1x02_P2.50mm_Vertical, F.Cu at (38.0, 109.2)
- added SW1: SW1, Connector_JST:JST_XH_B2B-XH-A_1x02_P2.50mm_Vertical, F.Cu at (55.6, 94.3)
- added SW2: SW2, Connector_JST:JST_XH_B2B-XH-A_1x02_P2.50mm_Vertical, F.Cu at (55.6, 85.6)
- added SW3: SW3, Connector_JST:JST_XH_B2B-XH-A_1x02_P2.50mm_Vertical, F.Cu at (55.6, 77.0)
- added SW4: SW4, Connector_JST:JST_XH_B2B-XH-A_1x02_P2.50mm_Vertical, F.Cu at (55.6, 68.4)
- added SW5: SW5, Connector_JST:JST_XH_B2B-XH-A_1x02_P2.50mm_Vertical, F.Cu at (38.0, 117.0)
- added Servo1: Servo1, Connector_JST:JST_XH_B3B-XH-A_1x03_P2.50mm_Vertical, F.Cu at (133.1, 37.0)
- added Servo2: Servo2, Connector_JST:JST_XH_B3B-XH-A_1x03_P2.50mm_Vertical, F.Cu at (133.1, 48.1)
- added Servo3: Servo3, Connector_JST:JST_XH_B3B-XH-A_1x03_P2.50mm_Vertical, F.Cu at (133.1, 59.2)
- added Servo4: Servo4, Connector_JST:JST_XH_B3B-XH-A_1x03_P2.50mm_Vertical, F.Cu at (133.1, 70.3)
- added U2: ~, Package_DIP:DIP-16_W7.62mm, F.Cu at (127.5, 83.6)
- J1, J3: value Conn_01x22_Pin -> Conn_01x22_Socket; footprint Connector_PinHeader_2.54mm:PinHeader_1x22_P2.54mm_Vertical -> Connector_PinSocket_2.54mm:PinSocket_1x22_P2.54mm_Vertical
- moved J1 50.9 mm to (76.2, 53.6)
- moved J3 50.9 mm to (99.1, 53.6)
Connections:
- net DN renamed NC7
- net DP renamed NC6
- net EN renamed NC1
- net IO10 renamed GPIO10
- net IO11 renamed GPIO11
- net IO4 renamed GPIO4
- net IO45 renamed NC5
- net IO46 renamed NC2
- net IO5 renamed GPIO5
- net IO6 renamed GPIO6
- net IO7 renamed GPIO7
- net IO8 renamed GPIO8
- net IO9 renamed GPIO9
- net RXD0 renamed NC4
- net TXD0 renamed NC3
- J1 pad 10: IO17 -> GPIO17
- J1 pad 11: IO18 -> GPIO18
- J1 pad 9: IO16 -> GPIO16
- J3 pad 10: IO38 -> GPIO38
- J3 pad 11: IO37 -> GPIO37
- J3 pad 12: IO36 -> GPIO36
- J3 pad 13: IO35 -> GPIO35
- J3 pad 14: IO0 -> GPIO0
- J3 pad 16: IO48 -> GPIO48
- J3 pad 17: IO47 -> GPIO47
- J3 pad 18: IO21 -> GPIO21
- J3 pad 4: IO1 -> GPIO1
- J3 pad 6: IO42 -> GPIO42
- J3 pad 7: IO41 -> GPIO41
- J3 pad 8: IO40 -> GPIO40
- J3 pad 9: IO39 -> GPIO39
Routing:
- net SERVO+: track 65.0 -> 0.00 mm
- net GND: track 57.2 -> 0.00 mm
