File: RRST-ESP32-S3-Rev.2-Sense-EXB/RRST-ESP32-S3-Rev.2-Sense-EXB.kicad_sch (KiCad schematic)
At the start: 28 parts, among them J1 Conn_01x22_Socket, J16 XT60-M, J17 XT60-M, J2 Conn_01x22_Socket, J3 Conn_01x22_Socket, J4 Conn_01x22_Socket, SW1 SW1, SW2 SW2, SW3 SW3, SW4 SW4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

Commit message: 拡張基盤迷走中
Parts:
- removed J2, J4: Conn_01x22_Socket, Connector_PinSocket_2.54mm:PinSocket_1x22_P2.54mm_Vertical, symbol Connector:Conn_01x22_Socket
- removed VMD1/VMD2: VMD1/VMD2, Connector_PinHeader_2.54mm:PinHeader_1x11_P2.54mm_Vertical, symbol Connector:Conn_01x11_Pin
- removed VMD3/VMD4: VMD3/VMD4, Connector_PinHeader_2.54mm:PinHeader_1x11_P2.54mm_Vertical, symbol Connector:Conn_01x11_Pin
- added CAN1: CAN, Connector_PinSocket_2.54mm:PinSocket_1x04_P2.54mm_Vertical, symbol Connector:Conn_01x04_Pin
- D1: footprint LED_THT:LED_D5.0mm -> LED_THT:LED_D3.0mm
- J16: footprint XT60-M:AMASS_XT60-M -> Connector_AMASS:AMASS_XT30U-M_1x02_P5.0mm_Vertical
- J17: footprint XT60-M:AMASS_XT60-M -> Connector_AMASS:AMASS_XT30U-F_1x02_P5.0mm_Vertical
Other:
- note removed: "ESP32-S3-DevKitC用ソケット(デバッグ用)"
- note removed: "VMD/MD"
