File: ESP32-WROOM-32E/ESP32-ROS-IO-susp-V1.0/ESP32-ROS-IO-susp-V1.0.kicad_pcb (KiCad board)
At the start: 2 copper layers, 21 parts, among them J1 Conn_01x19_Socket, J2 Conn_01x19_Socket, J3 Conn_01x19_Socket, J4 Conn_01x19_Socket

Commit message: ESP32-ROS-IO-susp-V1.0
Other:
- board text added: "ESP32-IO-Board-susp-V1.0 2026, NHK-Project, RRST"
- board text removed: "ESP32-susp-Board 2026, NHK-Project, RRST"
Changed lines of the file:
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@@
 			(fill yes)
 			(layer "F.SilkS")
-			(net 150902295)
 		)
 		(fp_poly
@@
 			(fill yes)
 			(layer "F.SilkS")
-			(net 150902295)
 		)
 		(fp_poly
@@
 			(fill yes)
 			(layer "F.SilkS")
-			(net 150902295)
 		)
 		(fp_poly
@@
 			(fill yes)
 			(layer "F.SilkS")
-			(net 150902295)
 		)
 		(fp_poly
@@
 			(fill yes)
 			(layer "F.SilkS")
-			(net 150902295)
 		)
 		(fp_poly
@@
 			(fill yes)
 			(layer "F.SilkS")
-			(net 150902295)
 		)
 		(fp_poly
@@
 			(fill yes)
 			(layer "F.SilkS")
-			(net 150902295)
 		)
 		(fp_poly
@@
 			(fill yes)
 			(layer "F.SilkS")
-			(net 150902295)
 		)
 		(fp_poly
@@
 			(fill yes)
 			(layer "F.SilkS")
-			(net 150902295)
 		)
 		(fp_poly
@@
 			(fill yes)
 			(layer "F.SilkS")
-			(net 150902295)
 		)
 		(fp_poly
@@
 			(fill yes)
 			(layer "F.SilkS")
-			(net 150902295)
 		)
 		(fp_poly
@@
 			(fill yes)
 			(layer "F.SilkS")
-			(net 150902295)
 		)
 		(fp_poly
@@
 			(fill yes)
 			(layer "F.SilkS")
-			(net 150902295)
 		)
 		(fp_poly
@@
 			(fill yes)
 			(layer "F.SilkS")
-			(net 150902295)
 		)
 		(fp_poly
@@
 			(fill yes)
 			(layer "F.SilkS")
-			(net 150902295)
 		)
 		(fp_poly
@@
 			(fill yes)
 			(layer "F.SilkS")
-			(net 150902295)
 		)
 		(fp_poly
@@
 			(fill yes)
 			(layer "F.SilkS")
-			(net 150902295)
 		)
 		(fp_poly
@@
 			(fill yes)
 			(layer "F.SilkS")
-			(net 150902295)
 		)
 		(fp_poly
@@
 			(fill yes)
 			(layer "F.SilkS")
-			(net 150902295)
 		)
 		(fp_poly
@@
 			(fill yes)
 			(layer "F.SilkS")
-			(net 150902295)
 		)
 		(fp_poly
@@
 			(fill yes)
 			(layer "F.SilkS")
-			(net 150902295)
 		)
 		(fp_poly
@@
 			(fill yes)
 			(layer "F.SilkS")
-			(net 150902295)
 		)
 		(fp_poly
@@
 			(fill yes)
 			(layer "F.SilkS")
-			(net 150902295)
 		)
 		(fp_poly
@@
 			(fill yes)
 			(layer "F.SilkS")
-			(net 150902295)
 		)
 		(fp_poly
@@
 			(fill yes)
 			(layer "F.SilkS")
-			(net 150902295)
 		)
 		(fp_poly
@@
 			(fill yes)
 			(layer "F.SilkS")
-			(net 150902295)
 		)
 		(fp_poly
@@
 			(fill yes)
 			(layer "F.SilkS")
-			(net 150902295)
 		)
 		(fp_poly
@@
 			(fill yes)
 			(layer "F.SilkS")
-			(net 150902295)
 		)
 		(fp_poly
@@
 			(fill yes)
 			(layer "F.SilkS")
-			(net 150902295)
 		)
 		(fp_poly
@@
 			(fill yes)
 			(layer "F.SilkS")
-			(net 150902295)
 		)
 		(fp_poly
@@
 			(fill yes)
 			(layer "F.SilkS")
-			(net 150902295)
 		)
 		(fp_poly
@@
 			(fill yes)
 			(layer "F.SilkS")
-			(net 150902295)
 		)
 		(fp_poly
@@
 			(fill yes)
 			(layer "F.SilkS")
-			(net 150902295)
 		)
 		(fp_poly
@@
 			(fill yes)
 			(layer "F.SilkS")
-			(net 150902295)
 		)
 		(fp_poly
@@
 			(fill yes)
 			(layer "F.SilkS")
-			(net 150902295)
 		)
 		(fp_poly
@@
 			(fill yes)
 			(layer "F.SilkS")
-			(net 150902295)
 		)
 		(fp_poly
@@
 			(fill yes)
 			(layer "F.SilkS")
-			(net 150902295)
 		)
 		(fp_poly
@@
 			(fill yes)
 			(layer "F.SilkS")
-			(net 150902295)
 		)
 		(fp_poly
@@
 			(fill yes)
 			(layer "F.SilkS")
-			(net 150902295)
 		)
 		(fp_poly
@@
 			(fill yes)
 			(layer "F.SilkS")
-			(net 150902295)
 		)
 		(fp_poly
@@
 			(fill yes)
 			(layer "F.SilkS")
-			(net 150902295)
 		)
 		(fp_poly
@@
 			(fill yes)
 			(layer "F.SilkS")
-			(net 150902295)
 		)
 		(fp_poly
@@
 			(fill yes)
 			(layer "F.SilkS")
-			(net 150902295)
 		)
 		(fp_poly
@@
 			(fill yes)
 			(layer "F.SilkS")
-			(net 150902295)
 		)
 		(fp_poly
@@
 			(fill yes)
 			(layer "F.SilkS")
-			(net 150902295)
 		)
 		(fp_poly
@@
 			(fill yes)
 			(layer "F.SilkS")
-			(net 150902295)
 		)
 		(fp_poly
@@
 			(fill yes)
 			(layer "F.SilkS")
-			(net 150902295)
 		)
 		(fp_poly
@@
 			(fill yes)
 			(layer "F.SilkS")
-			(net 150902295)
 		)
 		(fp_poly
@@
 			(fill yes)
 			(layer "F.SilkS")
-			(net 150902295)
 		)
 		(fp_poly
@@
 			(fill yes)
 			(layer "F.SilkS")
-			(net 150902295)
 		)
 		(fp_poly
@@
 			(fill yes)
 			(layer "F.SilkS")
-			(net 150902295)
 		)
 		(fp_poly
@@
 			(fill yes)
 			(layer "F.SilkS")
-			(net 150902295)
 		)
 		(fp_poly
@@
 			(fill yes)
 			(layer "F.SilkS")
-			(net 150902295)
 		)
 		(fp_poly
@@
 			(fill yes)
 			(layer "F.SilkS")
-			(net 150902295)
 		)
 		(fp_poly
@@
 			(fill yes)
 			(layer "F.SilkS")
-			(net 150902295)
 		)
 		(fp_poly
@@
 			(fill yes)
 			(layer "F.SilkS")
-			(net 150902295)
 		)
 		(fp_poly
@@
 			(fill yes)
 			(layer "F.SilkS")
-			(net 150902295)
 		)
 		(fp_poly
@@
 			(fill yes)
 			(layer "F.SilkS")
-			(net 150902295)
 		)
 		(fp_poly
@@
 			(fill yes)
 			(layer "F.SilkS")
-			(net 150902295)
 		)
 		(fp_poly
@@
 			(fill yes)
 			(layer "F.SilkS")
-			(net 150902295)
 		)
 		(fp_poly
@@
 			(fill yes)
 			(layer "F.SilkS")
-			(net 150902295)
 		)
 		(fp_poly
@@
 			(fill yes)
 			(layer "F.SilkS")
-			(net 150902295)
 		)
 		(fp_poly
@@
 			(fill yes)
 			(layer "F.SilkS")
-			(net 150902295)
 		)
 		(fp_poly
@@
 			(fill yes)
 			(layer "F.SilkS")
-			(net 150902295)
 		)
 		(fp_poly
@@
 			(fill yes)
 			(layer "F.SilkS")
-			(net 150902295)
 		)
 		(embedded_fonts no)
@@
 		)
 	)
-	(gr_text "ESP32-susp-Board\n2026, NHK-Project, RRST\n"
+	(gr_text "ESP32-IO-Board-susp-V1.0\n2026, NHK-Project, RRST\n"
 		(at 139.7 109.3216 90)
 		(layer "B.SilkS" knockout)

Commit message: can回路待ち
Parts:
- removed 120R_EN: R120, Connector_PinHeader_2.54mm:PinHeader_1x02_P2.54mm_Vertical
- added R120: R120, Connector_PinHeader_2.54mm:PinHeader_1x02_P2.54mm_Vertical, F.Cu at (156.2, 72.4)
- moved ENC4 2.36 mm to (174.0, 129.6)
- moved ENC3 1.47 mm to (119.4, 137.2)
- moved ENC2 1.13 mm to (165.2, 73.7)
- moved ENC1 0.86 mm to (119.5, 73.7)
Connections:
- ENC1 pad 1: VDD33 -> 5V0
- ENC2 pad 1: VDD33 -> 5V0
- ENC3 pad 1: VDD33 -> 5V0
- ENC4 pad 1: VDD33 -> 5V0
- R1 pad 1: CANH -> Net-(R120-Pin_2)

Commit message: 回路図できた
Parts:
- removed ?: , 
- removed G***6: LOGO, LOGO
- moved ENC4 156.2 mm to (41.7, 46.5), turned to 0 degrees
- moved J4 147.9 mm to (35.9, 22.0)
- moved J3 147.4 mm to (31.3, 22.0)
- moved VMD3/VMD4 136.1 mm to (69.0, 22.0), turned to 0 degrees
- moved J1 133.5 mm to (22.1, 22.0)
- moved U1 131.3 mm to (39.8, 52.9), turned to 0 degrees
- moved ENC2 130.7 mm to (41.7, 30.9)
- moved J2 125.5 mm to (26.7, 22.0)
- moved ENC3 125.5 mm to (41.7, 38.6), turned to 0 degrees
- moved R120 105.5 mm to (51.3, 61.3)
- moved VMD1/VMD2 102.9 mm to (64.4, 22.0)
- moved CAN_BUS2 99.5 mm to (56.1, 30.9)
- moved CAN_BUS4 96.6 mm to (56.1, 46.5)
- moved CAN_BUS1 94.7 mm to (56.1, 23.1)
- moved ENC1 92.8 mm to (41.7, 23.1)
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Connections:
- J1 pad 10: GPIO26 -> ENC3_B
- J1 pad 11: GPIO27 -> ENC4_A
- J1 pad 16: NC6 -> NC7
- J1 pad 17: NC7 -> NC8
- J1 pad 18: NC8 -> NC9
- J1 pad 7: GPIO32 -> ENC4_B
- J1 pad 8: GPIO33 -> NC6
- J1 pad 9: GPIO25 -> ENC3_A
- J2 pad 10: GPIO26 -> ENC3_B
- J2 pad 11: GPIO27 -> ENC4_A
- J2 pad 16: NC6 -> NC7
- J2 pad 17: NC7 -> NC8
- J2 pad 18: NC8 -> NC9
- J2 pad 7: GPIO32 -> ENC4_B
- J2 pad 8: GPIO33 -> NC6
- J2 pad 9: GPIO25 -> ENC3_A
- J3 pad 17: NC11 -> NC12
- J3 pad 18: NC12 -> NC13
- J3 pad 19: NC13 -> NC14
- J3 pad 2: GPIO23 -> ENC2_B
- J3 pad 3: GPIO22 -> ENC2_A
- J3 pad 4: NC9 -> NC10
- J3 pad 5: NC10 -> NC11
- J3 pad 6: GPIO21 -> ENC1_B
- J3 pad 8: GPIO19 -> ENC1_A
- J4 pad 17: NC11 -> NC12
- J4 pad 18: NC12 -> NC13
- J4 pad 19: NC13 -> NC14
- J4 pad 2: GPIO23 -> ENC2_B
- J4 pad 3: GPIO22 -> ENC2_A
- J4 pad 4: NC9 -> NC10
- J4 pad 5: NC10 -> NC11
- J4 pad 6: GPIO21 -> ENC1_B
- J4 pad 8: GPIO19 -> ENC1_A
Other:
- board text removed: "GND GND"
- board text removed: "H L"
