File: ESP32-S3N-WROOM-32E/ESP32-S3N-WROOM-32E.kicad_sch (KiCad schematic)
At the start: 59 parts, among them J1 Conn_01x19_Socket, J10 Conn_01x22_Socket, J16 XT60-M, J17 XT60-M, J2 Conn_01x19_Socket, J3 Conn_01x19_Socket, J4 Conn_01x19_Socket, J5 Conn_01x02_Pin, J6 Conn_01x02_Pin, J7 Conn_01x22_Socket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

Commit message: 回路図
Parts:
- removed VMD1: VMD1, XT30UPB-F:AMASS_XT30U-F_1x02_P5.0mm_Vertical, symbol XT30UPB-M:XT30UPB-M
- removed VMD2: VMD2, XT30UPB-F:AMASS_XT30U-F_1x02_P5.0mm_Vertical, symbol XT30UPB-M:XT30UPB-M
- removed VMD3: VMD3, XT30UPB-F:AMASS_XT30U-F_1x02_P5.0mm_Vertical, symbol XT30UPB-M:XT30UPB-M
- removed VMD4: VMD4, XT30UPB-F:AMASS_XT30U-F_1x02_P5.0mm_Vertical, symbol XT30UPB-M:XT30UPB-M
- removed VMDG1: VMDG1, XT30UPB-F:AMASS_XT30U-F_1x02_P5.0mm_Vertical, symbol XT30UPB-M:XT30UPB-M
- removed VMDG2: VMDG2, XT30UPB-F:AMASS_XT30U-F_1x02_P5.0mm_Vertical, symbol XT30UPB-M:XT30UPB-M
- removed VMDG3: VMDG3, XT30UPB-F:AMASS_XT30U-F_1x02_P5.0mm_Vertical, symbol XT30UPB-M:XT30UPB-M
- removed VMDG4: VMDG4, XT30UPB-F:AMASS_XT30U-F_1x02_P5.0mm_Vertical, symbol XT30UPB-M:XT30UPB-M
Connections:
- net CAN_RX: no longer J3.13 (Pin_13), J4.13 (Pin_13), J7.13 (Pin_13), J7.4 (Pin_4), J9.13 (Pin_13), J9.4 (Pin_4), U1.1 (Txd)
- net ENC1_A: no longer J1.13 (Pin_13), J2.13 (Pin_13), SW6.1 (Pin_1), VMD1/VMD2.5 (Pin_5)
- net ENC1_B: no longer J1.15 (Pin_15), J2.15 (Pin_15), SW4.1 (Pin_1), VMD3/VMD4.9 (Pin_9)
- net ENC2_A: no longer J1.12 (Pin_12), J2.12 (Pin_12), SW2.1 (Pin_1), VMD3/VMD4.5 (Pin_5)
- net ENC2_B: no longer J3.16 (Pin_16), J4.16 (Pin_16), SW7.1 (Pin_1), VMD1/VMD2.11 (Pin_11)
- net GPIO16: no longer J7.9 (Pin_9), J9.9 (Pin_9)
- net GPIO17: no longer J7.10 (Pin_10), J9.10 (Pin_10)
- net GPIO18: no longer J7.11 (Pin_11), J9.11 (Pin_11)
- net GPIO21: no longer J10.18 (Pin_18), J8.18 (Pin_18)
- net GPIO5: no longer J7.5 (Pin_5), J9.5 (Pin_5)
- net NC1: no longer J7.3 (Pin_3), J9.3 (Pin_3)
- net NC2: no longer J7.14 (Pin_14), J9.14 (Pin_14)
- net NC3: no longer J10.2 (Pin_2), J8.2 (Pin_2)
- net NC4: no longer J10.3 (Pin_3), J8.3 (Pin_3)
- net NC5: now also J9.14 (Pin_14); no longer J10.15 (Pin_15), J8.15 (Pin_15)
- net NC6: no longer J10.19 (Pin_19), J8.19 (Pin_19)
- net NC7: no longer J10.20 (Pin_20), J8.20 (Pin_20)
- net GPIO1 renamed GPIOS1
- net GPIO10 renamed GPIOS10
- net GPIO11 renamed GPIOS11
- net GPIO35 renamed GPIOS35
- net GPIO36 renamed GPIOS36
- net GPIO37 renamed GPIOS37
- net GPIO38 renamed GPIOS38
- net GPIO39 renamed GPIOS39
- net GPIO41 renamed GPIOS41
- net GPIO42 renamed GPIOS42
- net GPIO47 renamed GPIOS47
- net GPIO48 renamed GPIOS48
- net GPIO6 renamed GPIOS6
- net GPIO7 renamed GPIOS7
- net GPIO8 renamed GPIOS8
- net GPIO9 renamed GPIOS9
- new net CAN_TX: J3.13 (Pin_13), J4.13 (Pin_13), J7.13 (Pin_13), J9.13 (Pin_13), U1.1 (Txd)
- new net GPIO12: J1.13 (Pin_13), J2.13 (Pin_13), SW6.1 (Pin_1), VMD1/VMD2.5 (Pin_5)
- new net GPIO13: J1.15 (Pin_15), J2.15 (Pin_15), SW4.1 (Pin_1), VMD3/VMD4.9 (Pin_9)
- new net GPIO14: J1.12 (Pin_12), J2.12 (Pin_12), SW2.1 (Pin_1), VMD3/VMD4.5 (Pin_5)
- new net GPIO15: J3.16 (Pin_16), J4.16 (Pin_16), SW7.1 (Pin_1), VMD1/VMD2.11 (Pin_11)
- new net GPIOS16: J7.9 (Pin_9), J9.9 (Pin_9)
- new net GPIOS17: J7.10 (Pin_10), J9.10 (Pin_10)
- new net GPIOS18: J7.11 (Pin_11), J9.11 (Pin_11)
- new net GPIOS21: J10.18 (Pin_18), J8.18 (Pin_18)
- new net GPIOS4: J7.4 (Pin_4), J9.4 (Pin_4)
- new net GPIOS5: J7.5 (Pin_5), J9.5 (Pin_5)
- new net NC14: J7.3 (Pin_3), J9.3 (Pin_3)
- new net NC15: J7.14 (Pin_14)
- new net NC16: J10.2 (Pin_2), J8.2 (Pin_2)
- new net NC17: J10.3 (Pin_3), J8.3 (Pin_3)
- new net NC18: J10.15 (Pin_15), J8.15 (Pin_15)
- new net NC19: J10.19 (Pin_19), J8.19 (Pin_19)
- new net NC20: J10.20 (Pin_20), J8.20 (Pin_20)
Other:
- note added: "S3ピン割り当て"
- note added: "無印ピン割り当て"
- note removed: "ピン割り当て"
- moved on the sheet: D1, ENC1, ENC2, ENC3, ENC4, R2, VMD1/VMD2, VMD3/VMD4

Commit message: 回路図２
Parts:
- SW8: value SW7 -> SW8
Connections:
- net GPIO12: no longer VMD1/VMD2.5 (Pin_5)
- net GPIO13: no longer SW4.1 (Pin_1), VMD3/VMD4.9 (Pin_9)
- net GPIO14: no longer SW2.1 (Pin_1), VMD3/VMD4.5 (Pin_5)
- net GPIO15: no longer VMD1/VMD2.11 (Pin_11)
- net GPIO16: no longer SW5.1 (Pin_1), VMD1/VMD2.7 (Pin_7)
- net GPIO17: no longer SW3.1 (Pin_1), VMD3/VMD4.11 (Pin_11)
- net GPIO18: no longer SW1.1 (Pin_1), VMD3/VMD4.7 (Pin_7)
- net GPIO19: no longer Servo1.1 (Pin_1)
- net GPIO21: no longer Servo2.1 (Pin_1)
- net GPIO22: now also U2.7 (I7); no longer ENC2.4 (Pin_4), Servo3.1 (Pin_1)
- net GPIO23: no longer ENC2.3 (Pin_3), Servo4.1 (Pin_1)
- net GPIO25: no longer U2.1 (I1)
- net GPIO26: no longer U2.2 (I2)
- net GPIO27: no longer U2.3 (I3)
- net GPIO32: no longer ENC1.4 (Pin_4), U2.4 (I4)
- net GPIO33: no longer ENC1.3 (Pin_3), U2.5 (I5)
- net GPIO5: no longer VMD1/VMD2.9 (Pin_9)
- net GPIOS1: no longer U2.6 (I6)
- net TR7: no longer U2.7 (I7)
- new net GPIO12/GPIOS5: VMD1/VMD2.5 (Pin_5)
- new net GPIO13/GPIOS38: SW4.1 (Pin_1)
- new net GPIO13/GPIOS6: VMD3/VMD4.9 (Pin_9)
- new net GPIO14/GPIOS36: SW2.1 (Pin_1)
- new net GPIO14/GPIOS7: VMD3/VMD4.5 (Pin_5)
- new net GPIO15/GPIOS8: VMD1/VMD2.11 (Pin_11)
- new net GPIO16/GPIOS39: SW5.1 (Pin_1)
- new net GPIO16/GPIOS9: VMD1/VMD2.7 (Pin_7)
- new net GPIO17/GPIOS10: VMD3/VMD4.11 (Pin_11)
- new net GPIO17/GPIOS37: SW3.1 (Pin_1)
- new net GPIO18/GPIOS11: VMD3/VMD4.7 (Pin_7)
- new net GPIO18/GPIOS35: SW1.1 (Pin_1)
- new net GPIO19/GPIOS16: Servo1.1 (Pin_1)
- new net GPIO21/GPIOS17: Servo2.1 (Pin_1)
- new net GPIO22/GPIOS15: ENC2.4 (Pin_4)
- new net GPIO22/GPIOS18: Servo3.1 (Pin_1)
- new net GPIO23/GPIOS1: U2.6 (I6)
- new net GPIO23/GPIOS14: ENC2.3 (Pin_3)
- new net GPIO23/GPIOS21: Servo4.1 (Pin_1)
- new net GPIO25/GPIOS40: U2.1 (I1)
- new net GPIO26/GPIOS41: U2.2 (I2)
- new net GPIO27/GPIOS42: U2.3 (I3)
- new net GPIO32/GPIOS13: ENC1.4 (Pin_4)
- new net GPIO32/GPIOS47: U2.4 (I4)
- new net GPIO33/GPIOS12: ENC1.3 (Pin_3)
- new net GPIO33/GPIOS48: U2.5 (I5)
- new net GPIO5/GPIOS4: VMD1/VMD2.9 (Pin_9)
Other:
- moved on the sheet: D1, ENC1, ENC2, ENC3, ENC4, J10, J16, J17, J9, R2, SV1, SV2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

Commit message: 回路図
Connections:
- net CAN_TX: no longer U1.1 (Txd)
- new net GPIO4/GPIOS3: U1.1 (Txd)
Changed lines of the file:
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@@
 		)
 	)
-	(global_label "CAN_TX"
+	(global_label "GPIO4{slash}GPIOS3"
 		(shape input)
 		(at 105.41 201.93 180)
@@
 		)
 		(property "Intersheetrefs" "${INTERSHEET_REFS}"
-			(at 95.591 201.93 0)
+			(at 88.5152 201.93 0)
 			(effects
 				(font

Commit message: これならいけるか
Connections:
- net GPIO12/GPIOS5 is gone; now on net GPIO12: VMD1/VMD2.5 (Pin_5)
- net GPIO13/GPIOS38 is gone; now on net GPIO13: SW4.1 (Pin_1)
- net GPIO13/GPIOS6 is gone; now on net GPIO13: VMD3/VMD4.9 (Pin_9)
- net GPIO14/GPIOS36 is gone; now on net GPIO14: SW2.1 (Pin_1)
- net GPIO14/GPIOS7 is gone; now on net GPIO14: VMD3/VMD4.5 (Pin_5)
- net GPIO15/GPIOS8 is gone; now on net GPIO15: VMD1/VMD2.11 (Pin_11)
- net GPIO16/GPIOS39 is gone; now on net GPIO16: SW5.1 (Pin_1)
- net GPIO16/GPIOS9 is gone; now on net GPIO16: VMD1/VMD2.7 (Pin_7)
- net GPIO17/GPIOS10 is gone; now on net GPIO17: VMD3/VMD4.11 (Pin_11)
- net GPIO17/GPIOS37 is gone; now on net GPIO17: SW3.1 (Pin_1)
- net GPIO18/GPIOS11 is gone; now on net GPIO18: VMD3/VMD4.7 (Pin_7)
- net GPIO18/GPIOS35 is gone; now on net GPIO18: SW1.1 (Pin_1)
- net GPIO19/GPIOS16 is gone; now on net ENC4_B: Servo1.1 (Pin_1)
- net GPIO21/GPIOS17 is gone; now on net ENC4_A: Servo2.1 (Pin_1)
- net GPIO22/GPIOS15 is gone; now on net ENC2_B: ENC2.4 (Pin_4)
- net GPIO22/GPIOS18 is gone; now on net ENC2_B: Servo3.1 (Pin_1)
- net GPIO23 is gone; now on net ENC2_A: J3.2 (Pin_2), J4.2 (Pin_2), J5.2 (Pin_2)
- net GPIO23/GPIOS1 is gone; now on net GPIOS1: U2.6 (I6)
- net GPIO23/GPIOS14 is gone; now on net ENC2_A: ENC2.3 (Pin_3)
- net GPIO23/GPIOS21 is gone; now on net ENC2_A: Servo4.1 (Pin_1)
- net GPIO25/GPIOS40 is gone; now on net GPIO25: U2.1 (I1)
- net GPIO26/GPIOS41 is gone; now on net ENC3_B: U2.2 (I2)
- net GPIO27/GPIOS42 is gone; now on net ENC3_A: U2.3 (I3)
- net GPIO32 is gone; now on net ENC1_B: J1.7 (Pin_7), J2.7 (Pin_7)
- net GPIO32/GPIOS13 is gone; now on net ENC1_B: ENC1.4 (Pin_4)
- net GPIO32/GPIOS47 is gone; now on net ENC1_B: U2.4 (I4)
- net GPIO33 is gone; now on net ENC1_A: J1.8 (Pin_8), J2.8 (Pin_8)
- net GPIO33/GPIOS12 is gone; now on net ENC1_A: ENC1.3 (Pin_3)
- net GPIO33/GPIOS48 is gone; now on net ENC1_A: U2.5 (I5)
- net GPIO4/GPIOS3 is gone; now on net CAN_TX: U1.1 (Txd)
- net GPIO5/GPIOS4 is gone; now on net GPIO5: VMD1/VMD2.9 (Pin_9)
- net GPIOS10 is gone; now on net GPIO17: J7.16 (Pin_16), J9.16 (Pin_16)
- net GPIOS11 is gone; now on net GPIO18: J7.17 (Pin_17), J9.17 (Pin_17)
- net GPIOS16 is gone; now on net ENC4_B: J7.9 (Pin_9), J9.9 (Pin_9)
- net GPIOS17 is gone; now on net ENC4_A: J7.10 (Pin_10), J9.10 (Pin_10)
- net GPIOS18 is gone; now on net ENC2_B: J7.11 (Pin_11), J9.11 (Pin_11)
- net GPIOS21 is gone; now on net ENC2_A: J10.18 (Pin_18), J8.18 (Pin_18)
- net GPIOS35 is gone; now on net GPIO18: J10.13 (Pin_13), J8.13 (Pin_13)
- net GPIOS36 is gone; now on net GPIO14: J10.12 (Pin_12), J8.12 (Pin_12)
- net GPIOS37 is gone; now on net GPIO17: J10.11 (Pin_11), J8.11 (Pin_11)
- net GPIOS38 is gone; now on net GPIO13: J10.10 (Pin_10), J8.10 (Pin_10)
- net GPIOS39 is gone; now on net GPIO16: J10.9 (Pin_9), J8.9 (Pin_9)
- net GPIOS41 is gone; now on net ENC3_B: J10.7 (Pin_7), J8.7 (Pin_7)
- net GPIOS42 is gone; now on net ENC3_A: J10.6 (Pin_6), J8.6 (Pin_6)
- net GPIOS47 is gone; now on net ENC1_B: J10.17 (Pin_17), J8.17 (Pin_17)
- net GPIOS48 is gone; now on net ENC1_A: J10.16 (Pin_16), J8.16 (Pin_16)
- net GPIOS7 is gone; now on net GPIO14: J7.7 (Pin_7), J9.7 (Pin_7)
- net GPIOS8 is gone; now on net GPIO15: J7.12 (Pin_12), J9.12 (Pin_12)
- net GPIOS9 is gone; now on net GPIO16: J7.15 (Pin_15), J9.15 (Pin_15)
- net ENC2_B: now also J3.3 (Pin_3), J4.3 (Pin_3), J6.2 (Pin_2)
- net TR7: now also U2.7 (I7)
- net GPIO19 renamed ENC4_B
- net GPIO21 renamed ENC4_A
- removed net GPIO22: J3.3 (Pin_3), J4.3 (Pin_3), J6.2 (Pin_2), U2.7 (I7)
- net GPIO26 renamed ENC3_B
- net GPIO27 renamed ENC3_A
Other:
- moved on the sheet: CAN_BUS1, CAN_BUS2, CAN_BUS3, CAN_BUS4, CAN_BUS5, CAN_BUS6, CAN_BUS7, CAN_BUS8, D1, J17, J5, J6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
