File: XIAO-ESP32-S3-SS/XIAO-ESP32-S3-SS.kicad_sch (KiCad schematic)
At the start: 0 parts

Commit message: SS 回路図完成
Parts:
- added J1, J3: Conn_01x04_Socket, Connector_JST:JST_XH_B4B-XH-A_1x04_P2.50mm_Vertical, symbol Connector:Conn_01x04_Socket
- added J16, J17: XT60-M, XT60-M:AMASS_XT60-M, symbol XT60-M:XT60-M
- added R120: R120, Connector_PinHeader_2.54mm:PinHeader_1x02_P2.54mm_Vertical, symbol Connector:Conn_01x02_Pin
- added R3: 120, Resistor_THT:R_Axial_DIN0207_L6.3mm_D2.5mm_P10.16mm_Horizontal, symbol Device:R
- added SV1: SV1, Connector_JST:JST_XH_B2B-XH-A_1x02_P2.50mm_Vertical, symbol Connector:Conn_01x02_Pin
- added SV2: SV2, Connector_JST:JST_XH_B2B-XH-A_1x02_P2.50mm_Vertical, symbol Connector:Conn_01x02_Pin
- added SV3: SV3, Connector_JST:JST_XH_B2B-XH-A_1x02_P2.50mm_Vertical, symbol Connector:Conn_01x02_Pin
- added SV4: SV4, Connector_JST:JST_XH_B2B-XH-A_1x02_P2.50mm_Vertical, symbol Connector:Conn_01x02_Pin
- added Servo1: Servo1, Connector_JST:JST_XH_B3B-XH-A_1x03_P2.50mm_Vertical, symbol Connector:Conn_01x03_Pin
- added Servo2: Servo2, Connector_JST:JST_XH_B3B-XH-A_1x03_P2.50mm_Vertical, symbol Connector:Conn_01x03_Pin
- added Servo3: Servo3, Connector_JST:JST_XH_B3B-XH-A_1x03_P2.50mm_Vertical, symbol Connector:Conn_01x03_Pin
- added Servo4: Servo4, Connector_JST:JST_XH_B3B-XH-A_1x03_P2.50mm_Vertical, symbol Connector:Conn_01x03_Pin
- added Servo5: Servo5, Connector_JST:JST_XH_B3B-XH-A_1x03_P2.50mm_Vertical, symbol Connector:Conn_01x03_Pin
- added U1: (no value), Package_DIP:DIP-8_W7.62mm, symbol New_Library:MCP2561
- added U2: XIAO-ESP32-S3-SMD, Seeed Studio XIAO Series Library:XIAO-ESP32-S3-SMD, symbol Seeed_Studio_XIAO_Series:XIAO-ESP32-S3-SMD
- added U3: (no value), Package_DIP:DIP-16_W7.62mm, symbol New_Library:TBD62003APG
Connections:
- new net: R120.2 (Pin_2), R3.1
- new net +24V: J17.P (POS), SV1.2 (Pin_2), SV2.2 (Pin_2), SV3.2 (Pin_2), SV4.2 (Pin_2), U3.9 (COMMON)
- new net 3V3: U2.12 (3V3)
- new net 5V0: J1.1 (Pin_1), J3.1 (Pin_1), U1.3 (Vdd), U2.14 (VBUS)
- new net CANH: J1.3 (Pin_3), J3.3 (Pin_3), R120.1 (Pin_1), U1.7 (CANH)
- new net CANL: J1.4 (Pin_4), J3.4 (Pin_4), R3.2, U1.6 (CANL)
- new net CAN_RX: U1.4 (Rxd), U2.8 (GPIO44_D7_RX)
- new net CAN_TX: U1.1 (Txd), U2.7 (GPIO43_D6_TX)
- new net GND: J1.2 (Pin_2), J16.N (NEG), J17.N (NEG), J3.2 (Pin_2), Servo1.3 (Pin_3), Servo2.3 (Pin_3), Servo3.3 (Pin_3), Servo4.3 (Pin_3), Servo5.3 (Pin_3), U1.2 (Vss), U1.8 (STBY), U2.13 (GND), U2.27 (GND), U2.33 (GND), U3.8 (GND)
- new net GPIO1: Servo1.1 (Pin_1), U2.1 (GPIO1_A0_D0)
- new net GPIO2: Servo2.1 (Pin_1), U2.2 (GPIO2_A1_D1)
- new net GPIO3: Servo3.1 (Pin_1), U2.3 (GPIO3_A2_D2)
- new net GPIO4: Servo4.1 (Pin_1), U2.4 (GPIO4_A3_D3)
- new net GPIO5: Servo5.1 (Pin_1), U2.5 (GPIO5_A4_D4_SDA)
- new net GPIO6: U2.6 (GPIO6_A5_D5_SCL), U3.1 (I1)
- new net GPIO7: U2.9 (GPIO7_A8_D8_SCK), U3.2 (I2)
- new net GPIO8: U2.10 (GPIO8_A9_D9_MISO), U3.3 (I3)
- new net GPIO9: U2.11 (GPIO9_A10_D10_MOSI), U3.4 (I4)
- new net O1: SV1.1 (Pin_1), U3.16 (O1)
- new net O2: SV2.1 (Pin_1), U3.15 (O2)
- new net O3: SV3.1 (Pin_1), U3.14 (O3)
- new net O4: SV4.1 (Pin_1), U3.13 (O4)
- new net SERVO+: J16.P (POS), Servo1.2 (Pin_2), Servo2.2 (Pin_2), Servo3.2 (Pin_2), Servo4.2 (Pin_2), Servo5.2 (Pin_2)
- no-connect marks 0 -> 1
Other:
- note added: "CAN"
- note added: "サーボ"
- note added: "ソレノイドバルブ・表示灯"
- note added: "ピン割り当て"

Commit message: SS XT30に変更
Parts:
- removed J16, J17: XT60-M, XT60-M:AMASS_XT60-M, symbol XT60-M:XT60-M
- added J6, J7: Conn_01x02_Pin, Connector_AMASS:AMASS_XT30U-M_1x02_P5.0mm_Vertical, symbol Connector:Conn_01x02_Pin
Connections:
- net +24V: now also J6.2 (Pin_2)
- net GND: now also J6.1 (Pin_1), J7.1 (Pin_1)
- net SERVO+: now also J7.2 (Pin_2)

Commit message: SS 配置途中
Parts:
- renumbered J3 to J2, R3 to R1
Changed lines of the file:
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@@
 		(in_pos_files yes)
 		(dnp no)
-		(property "Reference" "J3"
+		(property "Reference" "J2"
 			(at 146.05 129.5399 0)
 			(show_name no)
@@
 			(project "XIAO-ESP32-S3-SS"
 				(path "/4e9a55bb-aa52-4145-afac-71373ee412d4"
-					(reference "J3")
+					(reference "J2")
 					(unit 1)
 				)
@@
 		(in_pos_files yes)
 		(dnp no)
-		(property "Reference" "R3"
+		(property "Reference" "R1"
 			(at 105.41 135.89 0)
 			(show_name no)
@@
 			(project "XIAO-ESP32-S3-SS"
 				(path "/4e9a55bb-aa52-4145-afac-71373ee412d4"
-					(reference "R3")
-					(unit 1)
-				)
+					(reference "R1")
+					(unit 1)
+				)
