File: CAN hub-ESC/CAN hub-ESC.kicad_sch (KiCad schematic)
At the start: 3 parts

Commit message: CAN hub-ENC
Parts:
- renumbered CAN_BUS_I1 to CAN_BUS1, CAN_BUS_ESC1 to CAN_BUS2, CAN_BUS_O1 to CAN_BUS3
Changed lines of the file:
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@@
 		(in_pos_files yes)
 		(dnp no)
-		(property "Reference" "CAN_BUS_ESC1"
-			(at 33.528 44.45 0)
+		(property "Reference" "CAN_BUS2"
+			(at 36.83 44.45 0)
 			(show_name no)
 			(do_not_autoplace no)
@@
 			(project "CAN hub-ESC"
 				(path "/69e9cccd-1b1f-431b-a94e-52c5c1905914"
-					(reference "CAN_BUS_ESC1")
+					(reference "CAN_BUS2")
 					(unit 1)
 				)
@@
 		(in_pos_files yes)
 		(dnp no)
-		(property "Reference" "CAN_BUS_O1"
-			(at 35.814 52.07 0)
+		(property "Reference" "CAN_BUS3"
+			(at 36.83 52.07 0)
 			(show_name no)
 			(do_not_autoplace no)
@@
 			(project "CAN hub-ESC"
 				(path "/69e9cccd-1b1f-431b-a94e-52c5c1905914"
-					(reference "CAN_BUS_O1")
+					(reference "CAN_BUS3")
 					(unit 1)
 				)
@@
 		(in_pos_files yes)
 		(dnp no)
-		(property "Reference" "CAN_BUS_I1"
-			(at 36.068 36.83 0)
+		(property "Reference" "CAN_BUS1"
+			(at 36.83 36.83 0)
 			(show_name no)
 			(do_not_autoplace no)
@@
 			(project "CAN hub-ESC"
 				(path "/69e9cccd-1b1f-431b-a94e-52c5c1905914"
-					(reference "CAN_BUS_I1")
+					(reference "CAN_BUS1")
 					(unit 1)
 				)
