File: CAN hub-ESC/CAN hub-ESC.kicad_pcb (KiCad board)
At the start: 2 copper layers, 10 x 40 mm, 5 parts

Commit message: CAN hub-ENC 変更
Routing:
- net CANH: track 16.1 -> 0.00 mm
- net CANL: track 16.1 -> 0.01 mm
- added copper zone on F.Cu, net CANH
- added copper zone on B.Cu, net CANL
Changed lines of the file:
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@@
-	)
-	(segment
-		(start 120.3 81.9012)
-		(end 120.3 97.9968)
-		(width 0.2)
-		(layer "F.Cu")
-		(net "CANL")
 	)
 	(segment
@@
 	)
 	(segment
+		(start 120.3 97.9968)
+		(end 120.2968 98)
+		(width 0.2)
+		(layer "B.Cu")
+		(net "CANL")
+	)
+	(segment
 		(start 117.5032 97.9968)
 		(end 117.5 98)
@@
 		(net "CANH")
 	)
-	(segment
-		(start 117.8 81.9012)
-		(end 117.8 97.9968)
-		(width 0.2)
+	(zone
+		(net "CANH")
 		(layer "F.Cu")
-		(net "CANH")
+		(hatch edge 0.5)
+		(connect_pads
+			(clearance 0)
+		)
+		(min_thickness 0.25)
+		(fill
+			(thermal_gap 0.5)
+			(thermal_bridge_width 0.5)
+			(island_removal_mode 0)
+		)
+		(polygon
+			(pts
+				(xy 114.5 79) (xy 123.5 79) (xy 123.5 102) (xy 114.5 102)
+			)
+		)
+	)
+	(zone
+		(net "CANL")
+		(layer "B.Cu")
+		(hatch edge 0.5)
+		(priority 1)
+		(connect_pads
+			(clearance 0)
+		)
+		(min_thickness 0.25)
+		(fill
+			(thermal_gap 0.5)
+			(thermal_bridge_width 0.5)
+			(island_removal_mode 0)
+		)
+		(polygon
+			(pts
+				(xy 114.5 79) (xy 123.5 79) (xy 123.5 102) (xy 114.5 102)
+			)
+		)
 	)
 	(embedded_fonts no)

Commit message: 一旦ここまで
Changed lines of the file:
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@@
 		)
 		(min_thickness 0.25)
-		(fill
+		(fill yes
 			(thermal_gap 0.5)
 			(thermal_bridge_width 0.5)
@@
 		(polygon
 			(pts
-				(xy 114.5 79) (xy 123.5 79) (xy 123.5 102) (xy 114.5 102)
+				(xy 115 79.5) (xy 123 79.5) (xy 123 101.5) (xy 115 101.5)
 			)
 		)
@@
 		)
 		(min_thickness 0.25)
-		(fill
+		(fill yes
 			(thermal_gap 0.5)
 			(thermal_bridge_width 0.5)
@@
 		(polygon
 			(pts
-				(xy 114.5 79) (xy 123.5 79) (xy 123.5 102) (xy 114.5 102)
+				(xy 115 79.5) (xy 123 79.5) (xy 123 101.5) (xy 115 101.5)
 			)
 		)
