File: XIAO-ESP32-S3-VAR/XIAO-ESP32-S3-VAR.kicad_sch (KiCad schematic)
At the start: 12 parts, among them J1 Conn_01x04_Socket, J2 Conn_01x03_Socket, J3 Conn_01x04_Socket, J4 Conn_01x03_Socket, J5 Conn_01x03_Socket, J6 Conn_01x02_Pin, U2 XIAO-ESP32-S3-SMD

Commit message: 一旦ここまで
Parts:
- renumbered J3 to J2, J2 to J3
Changed lines of the file:
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@@
 		(in_pos_files yes)
 		(dnp no)
-		(property "Reference" "J2"
+		(property "Reference" "J3"
 			(at 139.7 29.2099 0)
 			(show_name no)
@@
 			(project "XIAO-ESP32-S3-VAR"
 				(path "/f176684b-fd0e-445e-a6e8-0bba85d607c3"
-					(reference "J2")
+					(reference "J3")
 					(unit 1)
 				)
@@
 		(in_pos_files yes)
 		(dnp no)
-		(property "Reference" "J3"
+		(property "Reference" "J2"
 			(at 149.86 126.9999 0)
 			(show_name no)
@@
 			(project "XIAO-ESP32-S3-VAR"
 				(path "/f176684b-fd0e-445e-a6e8-0bba85d607c3"
-					(reference "J3")
-					(unit 1)
-				)
+					(reference "J2")
+					(unit 1)
+				)
